File: avionics/kicad/Lyra_flight_computer/Lyra v2/Lyra V2/Lyra V2.kicad_sch (KiCad schematic)
At the start: 90 parts, among them J1 USB_B_Micro, J10 Conn_01x04, J11 Conn_01x04, J12 Conn_01x03, J2 Screw_Terminal_01x04, J3 Screw_Terminal_01x04, J4 Conn_02x03_Odd_Even, J5 Screw_Terminal_01x04, J6 Screw_Terminal_01x04, J7 Conn_02x03_Odd_Even, J8 Conn_02x03_Odd_Even, J9 Conn_02x03_Odd_Even, J9 MEM2067-02-180-00-A, Q1 AO3401A, Q2 BSS138, Q3 BSS138, SW1 SW_Push_DPDT, U1 AZ1117-3.3, U2 AZ1117-5.0, U3 LIS3MDL, U4 BMP390L, U5 W25Q128JVS, U6 RP2040, U7 BMI088, X1 ECS-2520MV-xxx-xx

Commit message: lyra v3 work
Connections:
- no-connect marks 14 -> 15
Changed lines of the file:
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@@
   (no_connect (at 340.995 50.8))
   (no_connect (at 41.275 209.55))
+  (no_connect (at 343.535 118.745))
   (no_connect (at 322.58 97.155))
   (no_connect (at 322.58 94.615))
