File: avionics/kicad/Lyra_flight_computer/lyra V3/Lyrav3og.kicad_pcb (KiCad board)
At the start: 4 copper layers, 50 x 60 mm, 133 parts, among them J1 Conn_01x04, J10 TSW-104-08-T-T-RA, J11 Screw_Terminal_01x10, J12 Conn_01x02, J13 Conn_01x14, J15 USB_B_Micro, J16 Conn_01x02, J17 Conn_01x03, J18 Screw_Terminal_01x10, J2 Conn_01x02, J3 Conn_01x04, J4 Conn_01x03, J5 Conn_01x04, J6 USB_B_Micro, J7 Conn_02x03_Odd_Even, J8 Conn_01x14, J9 Conn_01x02, Q1 AO3401A, Q2 KY6802, Q3 KY6802, U1 AMS1117-5.0, U10 RP2040, U12 W25Q64JVXGIQ, U2 AMS1117-3.3, U3 W25Q64JVXGIQ, U4 BMI088, U5 MPL3115A2, U6 ADXL375BCCZ-RL7, U7 LIS3MDL, U8 RP2040, X1 S3D12.288000B20F30T, X2 S3D12.288000B20F30T

Commit message: bunch of stuff, new rouiting
Parts:
- removed U12: W25Q64JVXGIQ, easyeda2kicad:XSON-8_L4.0-W4.0-P0.80-TL-EP
- added C1: 100n, Capacitor_SMD:C_0402_1005Metric, B.Cu at (171.6, 90.6)
- added U11: W25Q16JVUXIQ, easyeda2kicad:USON-8_L3.0-W2.0-P0.50-BL-EP, B.Cu at (165.8, 86.2)
- added U9: W25Q16JVUXIQ, easyeda2kicad:USON-8_L3.0-W2.0-P0.50-BL-EP, B.Cu at (190.6, 87.1)
- C2, C3, C4, C46, C5, R32, U1, U2: moved to F.Cu
- JP4, R2, R26, R3: moved to B.Cu
- U3: value W25Q64JVXGIQ -> W25Q32JVZP; footprint easyeda2kicad:XSON-8_L4.0-W4.0-P0.80-TL-EP -> Package_SON:WSON-8-1EP_6x5mm_P1.27mm_EP3.4x4.3mm; moved to F.Cu
- moved J7 53.3 mm to (170.7, 62.1), turned to 180 degrees
- moved JP4 48.8 mm to (173.3, 61.8), turned to 180 degrees
- moved D1 17.3 mm to (170.8, 109.0)
- moved U3 17.2 mm to (174.0, 92.3)
- moved JP5 12.7 mm to (165.0, 74.2)
- moved C33 9.22 mm to (164.3, 72.4)
- moved C4 7.71 mm to (167.0, 110.7), turned to 180 degrees
- moved C5 7.27 mm to (175.2, 112.3), turned to 0 degrees
- moved U2 6.27 mm to (174.3, 115.9)
- moved R3 6.16 mm to (177.2, 106.9), turned to 180 degrees
- moved R2 5.95 mm to (177.2, 107.9), turned to 0 degrees
- moved R26 5.73 mm to (193.2, 86.9)
- moved J12 5.55 mm to (167.3, 90.3), turned to 0 degrees
- moved C46 4.84 mm to (190.6, 86.9), turned to 0 degrees
- moved U1 4.76 mm to (168.5, 115.9)
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Connections:
- JP5 pad 3: +12VA -> +BATT
- U10 pad 15: /INT12 BOT -> /INT21 BOT
- U10 pad 16: /INT21 BOT -> /INT12 BOT
- U3 pad 1: /QSPI_SS -> /FLASH CS BOT
- U3 pad 2: /QSPI_SD1 -> /SPI1 MISO BOT
- U3 pad 3: /QSPI_SD2 -> +3V3
- U3 pad 5: /QSPI_SDO -> /SPI1 MOSI BOT
- U3 pad 6: /QSPI_SCLK -> /SPI1 SCLK BOT
- U3 pad 7: /QSPI_SD3 -> +3V3
- U8 pad 17: /INT12 -> /INT21
- U8 pad 18: /INT21 -> /INT12
Routing:
- net /I2C1 SDA: track 0.00 -> 100.3 mm, vias 0 -> 1
- net /I2C1 SCL: track 0.00 -> 96.8 mm, vias 0 -> 6
- net GND: track 43.4 -> 109.9 mm, vias 37 -> 67
- net /GPIO26 BOT: track 0.00 -> 63.4 mm, vias 0 -> 2
- net /GPIO27 BOT: track 0.00 -> 57.2 mm, vias 0 -> 2
- net +BATT: track 6.58 -> 60.8 mm, vias 0 -> 2
- net VBUS: track 0.00 -> 50.7 mm
- net /BATT SENSE BOT: track 0.97 -> 51.5 mm, vias 0 -> 4
- net /P1 CONT BOT: track 1.17 -> 49.1 mm, vias 0 -> 3
- net +3V3: track 35.2 -> 76.2 mm, vias 28 -> 50
- net /P2 CONT BOT: track 1.03 -> 41.5 mm, vias 0 -> 4
- net /GPIO28 BOT: track 0.00 -> 33.6 mm, vias 0 -> 2
- net /PYRO PWR: track 24.1 -> 56.6 mm, vias 0 -> 2
- net /P3 CONT BOT: track 1.07 -> 32.9 mm, vias 0 -> 2
- net +5V: track 0.00 -> 27.8 mm, vias 0 -> 1
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- removed copper zone on B.Cu, net +3V3
- removed copper zone on F.Cu, net +3V3
- removed copper zone on F.Cu, net GND
