File: avionics/kicad/Lyra_flight_computer/lyra V3/Lyrav3.kicad_sch (KiCad schematic)
At the start: 133 parts, among them J1 Conn_01x04, J10 TSW-104-08-T-T-RA, J11 Screw_Terminal_01x10, J12 Conn_01x02, J13 Conn_01x14, J15 USB_B_Micro, J16 Conn_01x02, J17 Conn_01x03, J18 Screw_Terminal_01x10, J2 Conn_01x02, J3 Conn_01x04, J4 Conn_01x03, J5 Conn_01x04, J6 USB_B_Micro, J7 Conn_02x03_Odd_Even, J8 Conn_01x14, J9 Conn_01x02, Q1 AO3401A, Q2 KY6802, Q3 KY6802, U1 AMS1117-5.0, U10 RP2040, U12 W25Q64JVXGIQ, U2 AMS1117-3.3, U3 W25Q64JVXGIQ, U4 BMI088, U5 MPL3115A2, U6 ADXL375BCCZ-RL7, U7 LIS3MDL, U8 RP2040, X1 S3D12.288000B20F30T, X2 S3D12.288000B20F30T

Commit message: more lyrav3 work as well as more work on new text file and DMA
Parts:
- added TP1: TestPoint, TestPoint:TestPoint_Pad_1.0x1.0mm, symbol Connector:TestPoint
Connections:
- net +3V3: now also J11.1 (Pin_1)
- net GND: now also J11.2 (Pin_2)
- net GPIO26 BOT: no longer J11.2 (Pin_2)
- net GPIO27 BOT: now also TP1.1; no longer J11.1 (Pin_1)
- net INT12: now also U8.18 (GPIO15); no longer U8.17 (GPIO14)
- net INT21: now also U8.17 (GPIO14); no longer U8.18 (GPIO15)
Changed lines of the file:
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@@
   (junction (at 526.415 341.63) (diameter 0) (color 0 0 0 0)
   )
+  (junction (at 416.56 204.47) (diameter 0) (color 0 0 0 0)
+  )
   (junction (at 373.38 55.88) (diameter 0) (color 0 0 0 0)
   )
@@
   (junction (at 323.85 33.655) (diameter 0) (color 0 0 0 0)
   )
+  (junction (at 408.94 207.01) (diameter 0) (color 0 0 0 0)
+  )
   (junction (at 241.935 160.02) (diameter 0) (color 0 0 0 0)
   )
@@
     (stroke (width 0) (type default))
   )
-  (wire (pts (xy 413.385 204.47) (xy 426.085 204.47))
-    (stroke (width 0) (type default))
-  )
   (wire (pts (xy 32.385 353.695) (xy 38.735 353.695))
     (stroke (width 0) (type default))
@@
     (stroke (width 0) (type default))
   )
+  (wire (pts (xy 415.925 204.47) (xy 416.56 204.47))
+    (stroke (width 0) (type default))
+  )
   (wire (pts (xy 358.775 40.64) (xy 367.665 40.64))
     (stroke (width 0) (type default))
@@
     (stroke (width 0) (type default))
   )
+  (wire (pts (xy 416.56 204.47) (xy 426.085 204.47))
+    (stroke (width 0) (type default))
+  )
   (wire (pts (xy 282.716 196.8587) (xy 281.446 196.8587))
     (stroke (width 0) (type default))
@@
     (stroke (width 0) (type default))
   )
-  (wire (pts (xy 408.94 203.835) (xy 408.94 224.155))
+  (wire (pts (xy 408.94 203.835) (xy 408.94 207.01))
     (stroke (width 0) (type default))
   )
@@
     (stroke (width 0) (type default))
   )
+  (wire (pts (xy 408.94 207.01) (xy 408.94 224.155))
+    (stroke (width 0) (type default))
+  )
   (wire (pts (xy 574.675 310.515) (xy 574.675 311.15))
     (stroke (width 0) (type default))
@@
     (stroke (width 0) (type default))
   )
-  (wire (pts (xy 413.385 207.01) (xy 426.085 207.01))
-    (stroke (width 0) (type default))
-  )
   (wire (pts (xy 282.575 112.395) (xy 283.845 112.395))
     (stroke (width 0) (type default))
@@
     (stroke (width 0) (type default))
   )
+  (wire (pts (xy 399.415 181.61) (xy 418.465 181.61))
+    (stroke (width 0) (type default))
+  )
   (wire (pts (xy 361.315 207.645) (xy 371.475 207.645))
     (stroke (width 0) (type default))
@@
     (stroke (width 0) (type default))
   )
+  (wire (pts (xy 408.94 207.01) (xy 426.085 207.01))
+    (stroke (width 0) (type default))
+  )
   (wire (pts (xy 325.755 259.715) (xy 335.915 259.715))
     (stroke (width 0) (type default))
@@
     (effects (font (size 1.27 1.27)) (justify left bottom))
   )
+  (label "GPIO27 BOT" (at 418.465 181.61 180) (fields_autoplaced)
+    (effects (font (size 1.27 1.27)) (justify right bottom))
+  )
   (label "GPIO27" (at 294.005 349.25 180) (fields_autoplaced)
     (effects (font (size 1.27 1.27)) (justify right bottom))
@@
     (effects (font (size 1.27 1.27)) (justify left bottom))
   )
-  (label "INT21" (at 294.005 316.23 180) (fields_autoplaced)
-    (effects (font (size 1.27 1.27)) (justify right bottom))
-  )
   (label "LEDGREEN" (at 294.005 303.53 180) (fields_autoplaced)
     (effects (font (size 1.27 1.27)) (justify right bottom))
@@
     (effects (font (size 1.27 1.27)) (justify left bottom))
   )
-  (label "GPIO26 BOT" (at 413.385 207.01 0) (fields_autoplaced)
-    (effects (font (size 1.27 1.27)) (justify left bottom))
-  )
   (label "RUN" (at 177.8 295.275 180) (fields_autoplaced)
     (effects (font (size 1.27 1.27)) (justify right bottom))
@@
     (effects (font (size 1.27 1.27)) (justify right bottom))
   )
+  (label "INT12" (at 294.005 316.23 180) (fields_autoplaced)
+    (effects (font (size 1.27 1.27)) (justify right bottom))
+  )
   (label "RUN BOT" (at 339.09 295.275 0) (fields_autoplaced)
     (effects (font (size 1.27 1.27)) (justify left bottom))
@@
     (effects (font (size 1.27 1.27)) (justify right bottom))
   )
-  (label "GPIO27 BOT" (at 413.385 204.47 0) (fields_autoplaced)
-    (effects (font (size 1.27 1.27)) (justify left bottom))
-  )
   (label "P2 CONT BOT" (at 469.9 349.25 180) (fields_autoplaced)
     (effects (font (size 1.27 1.27)) (justify right bottom))
@@
     (effects (font (size 1.27 1.27)) (justify right bottom))
   )
-  (label "INT12" (at 294.005 313.69 180) (fields_autoplaced)
-    (effects (font (size 1.27 1.27)) (justify right bottom))
-  )
   (label "XIN" (at 189.23 328.295 180) (fields_autoplaced)
     (effects (font (size 1.27 1.27)) (justify right bottom))
@@
     (effects (font (size 1.27 1.27)) (justify left bottom))
   )
+  (label "INT21" (at 294.005 313.69 180) (fields_autoplaced)
+    (effects (font (size 1.27 1.27)) (justify right bottom))
+  )
   (label "XIN" (at 226.695 323.85 0) (fields_autoplaced)
     (effects (font (size 1.27 1.27)) (justify left bottom))
@@
     )
   )
+  (symbol (lib_id "power:+3V3") (at 416.56 204.47 0) (unit 1)
+    (in_bom yes) (on_board yes) (dnp no) (fields_autoplaced)
+    (property "Reference" "#PWR07" (at 416.56 208.28 0)
+      (effects (font (size 1.27 1.27)) hide)
+    )
+    (property "Value" "+3V3" (at 416.56 200.66 0)
+      (effects (font (size 1.27 1.27)))
+    )
+    (property "Footprint" "" (at 416.56 204.47 0)
+      (effects (font (size 1.27 1.27)) hide)
+    )
+    (property "Datasheet" "" (at 416.56 204.47 0)
+      (effects (font (size 1.27 1.27)) hide)
+    )
+    (pin "1")
+    (instances
+      (project "Lyrav3"
+        (path "/12cc3c39-e34e-4801-bd3f-38f875d59424"
+          (reference "#PWR07") (unit 1)
+        )
+      )
+      (project "Lyra V2"
+        (path "/63622aab-8dfa-4523-a589-40aebeb23162"
+          (reference "#PWR056") (unit 1)
+        )
+      )
+    )
+  )
   (symbol (lib_id "power:+3V3") (at 326.39 58.42 0) (unit 1)
     (in_bom yes) (on_board yes) (dnp no) (fields_autoplaced)
@@
         )
       )
+    )
+  )
+  (symbol (lib_id "Connector:TestPoint") (at 399.415 181.61 90) (unit 1)
+    (in_bom yes) (on_board yes) (dnp no) (fields_autoplaced)
+    (property "Reference" "TP1" (at 396.113 176.53 90)
+      (effects (font (size 1.27 1.27)))
+    )
+    (property "Value" "TestPoint" (at 396.113 179.07 90)
+      (effects (font (size 1.27 1.27)))
+    )
+    (property "Footprint" "TestPoint:TestPoint_Pad_1.0x1.0mm" (at 399.415 176.53 0)
+      (effects (font (size 1.27 1.27)) hide)
+    )
+    (property "Datasheet" "~" (at 399.415 176.53 0)
+      (effects (font (size 1.27 1.27)) hide)
+    )
+    (pin "1")
+    (instances
+      (project "Lyrav3"
+        (path "/12cc3c39-e34e-4801-bd3f-38f875d59424"
+          (reference "TP1") (unit 1)
+        )
+      )

Commit message: more lyrv v3 work
Parts:
- R13, R14: LCSC Part (none) -> C163447
- R21, R22, R29, R30: LCSC Part (none) -> C2909343
- R25, R31: LCSC Part (none) -> C375970
Changed lines of the file:
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@@
       (effects (font (size 1.27 1.27)) hide)
     )
-    (property "LCSC Part" "" (at 167.64 271.78 0)
+    (property "LCSC Part" " C163447 " (at 167.64 271.78 0)
       (effects (font (size 1.27 1.27)) hide)
     )
@@
       (effects (font (size 1.27 1.27)) hide)
     )
-    (property "LCSC Part" "" (at 382.27 285.75 0)
+    (property "LCSC Part" "C2909343" (at 382.27 285.75 0)
       (effects (font (size 1.27 1.27)) hide)
     )
@@
       (effects (font (size 1.27 1.27)) hide)
     )
-    (property "LCSC Part" "" (at 216.535 285.75 0)
+    (property "LCSC Part" "C2909343" (at 216.535 285.75 0)
       (effects (font (size 1.27 1.27)) hide)
     )
@@
       (effects (font (size 1.27 1.27)) hide)
     )
-    (property "LCSC Part" "" (at 349.885 292.1 0)
+    (property "LCSC Part" "C375970" (at 349.885 292.1 0)
       (effects (font (size 1.27 1.27)) hide)
     )
@@
       (effects (font (size 1.27 1.27)) hide)
     )
-    (property "LCSC Part" "" (at 163.83 271.78 0)
+    (property "LCSC Part" " C163447 " (at 163.83 271.78 0)
       (effects (font (size 1.27 1.27)) hide)
     )
@@
       (effects (font (size 1.27 1.27)) hide)
     )
-    (property "LCSC Part" "" (at 382.27 288.29 0)
+    (property "LCSC Part" "C2909343" (at 382.27 288.29 0)
       (effects (font (size 1.27 1.27)) hide)
     )
@@
       (effects (font (size 1.27 1.27)) hide)
     )
-    (property "LCSC Part" "" (at 166.37 292.1 0)
+    (property "LCSC Part" "C375970" (at 166.37 292.1 0)
       (effects (font (size 1.27 1.27)) hide)
     )
@@
       (effects (font (size 1.27 1.27)) hide)
     )
-    (property "LCSC Part" "" (at 216.535 288.29 0)
+    (property "LCSC Part" "C2909343" (at 216.535 288.29 0)
       (effects (font (size 1.27 1.27)) hide)
     )

Commit message: more lyra v3 work
got rid of the second MCU, just going to use I/O expanders and an ADC
Parts:
- removed C35, C38, C39, C40, C41, C42, C43, C44, C46, C6: 100n, Capacitor_SMD:C_0402_1005Metric, symbol Device:C_Small
- removed C36, C37: 1u, Capacitor_SMD:C_0402_1005Metric, symbol Device:C_Small
- removed C45: 2u2, Capacitor_SMD:C_0402_1005Metric, symbol Device:C_Small
- removed J1: Conn_01x04, Connector_JST:JST_SH_SM04B-SRSS-TB_1x04-1MP_P1.00mm_Horizontal, symbol Connector_Generic:Conn_01x04
- removed J11, J18: Screw_Terminal_01x10, TerminalBlock_Phoenix:TerminalBlock_Phoenix_MPT-0,5-10-2.54_1x10_P2.54mm_Horizontal, symbol Connector:Screw_Terminal_01x10
- removed J12: Conn_01x02, Jumper:SolderJumper-2_P1.3mm_Open_RoundedPad1.0x1.5mm, symbol Connector_Generic:Conn_01x02
- removed J15: USB_B_Micro, easyeda2kicad:MICRO-USB-SMD_U254-051T-4BHJ25-F2S, symbol Connector:USB_B_Micro
- removed J16: Conn_01x02, Jumper:SolderJumper-2_P1.3mm_Open_Pad1.0x1.5mm, symbol Connector_Generic:Conn_01x02
- removed J17: Conn_01x03, Connector_JST:JST_SH_SM03B-SRSS-TB_1x03-1MP_P1.00mm_Horizontal, symbol Connector_Generic:Conn_01x03
- removed R29, R30: 27R, Resistor_SMD:R_0402_1005Metric, symbol Device:R_Small
- removed R31: 10k, Resistor_SMD:R_0402_1005Metric, symbol Device:R_Small
- removed R32: 1k, Resistor_SMD:R_0402_1005Metric, symbol Device:R_Small
- removed U10: RP2040, Package_DFN_QFN:QFN-56-1EP_7x7mm_P0.4mm_EP3.2x3.2mm, symbol MCU_RaspberryPi:RP2040
- removed U12: W25Q64JVXGIQ, easyeda2kicad:XSON-8_L4.0-W4.0-P0.80-TL-EP, symbol easyeda2kicad:W25Q64JVXGIQ
- removed X2: S3D12.288000B20F30T, easyeda2kicad:OSC-SMD_4P-L3.2-W2.5-BL_SIT8008BI, symbol easyeda2kicad:S3D12.288000B20F30T
- added J11, J12: Screw_Terminal_01x12, TerminalBlock_Phoenix:TerminalBlock_Phoenix_MPT-0,5-12-2.54_1x12_P2.54mm_Horizontal, symbol Connector:Screw_Terminal_01x12
- added U10: ADS1015IDGS, easyeda2kicad:X2QFN-10_L2.0-W1.5-P0.50-BL, symbol Analog_ADC:ADS1015IDGS
Connections:
- net SPI0 CSn BOT is gone; now on net I2C1 SCL: J13.3 (Pin_3)
- net SPI0 MOSI BOT is gone; now on net I2C1 SDA: J13.4 (Pin_4)
- net +12P: now also J11.8 (Pin_8)
- net +12V: now also J11.9 (Pin_9)
- net +12VA: now also J12.1 (Pin_1)
- net +3V3: now also J12.3 (Pin_3)
- net +5V: now also J12.2 (Pin_2)
- net +BATT: now also J11.10 (Pin_10), J11.12 (Pin_12)
- net BATT SENSE BOT: no longer J13.7 (Pin_7)
- net BUZZER: now also U8.8 (GPIO6); no longer U8.7 (GPIO5)
- net GND: now also J11.11 (Pin_11), J11.5 (Pin_5), J12.4 (Pin_4)
- net GPIO26: no longer U8.38 (GPIO26_ADC0)
- net GPIO27: no longer U8.39 (GPIO27_ADC1)
- net GPIO27 BOT: no longer J13.10 (Pin_10)
- net GPIO28: no longer U8.40 (GPIO28_ADC2)
- net GPIO28 BOT: now also J11.6 (Pin_6); no longer J13.9 (Pin_9)
- net I2C1 SCL: no longer U4.8 (SCL/SCK), U5.8 (SCL), U6.14 (SCL/SCLK), U7.1 (SCL/SPC)
- net I2C1 SDA: no longer U4.9 (SDA/SDI), U5.7 (SDL), U6.13 (SDA/SDI/SDIO), U7.11 (SDA/SDI/SDO)
- net INT12: no longer U8.18 (GPIO15)
- net INT21: no longer U8.17 (GPIO14)
- net P1-: now also J12.11 (Pin_11)
- net P2-: now also J12.9 (Pin_9)
- net P3-: now also J12.7 (Pin_7)
- net P4-: now also J12.5 (Pin_5)
- net PYRO PWR: now also J11.7 (Pin_7), J12.10 (Pin_10), J12.12 (Pin_12), J12.6 (Pin_6), J12.8 (Pin_8)
- net I2C0 SDA: now reaches U8.6 (GPIO4)
- net I2C0 SDA: now also U4.9 (SDA/SDI), U5.7 (SDL), U6.13 (SDA/SDI/SDIO), U7.11 (SDA/SDI/SDO)
- net GPIO26 BOT: no longer names the net of J13.11 (Pin_11)
- net INT12 BOT: no longer names the net of J13.12 (Pin_12)
- net INT21 BOT: no longer names the net of J13.13 (Pin_13)
- net SPI0 MISO BOT: no longer names the net of J13.5 (Pin_5)
- net SPI0 SCK BOT: no longer names the net of J13.6 (Pin_6)
- new net I2C0 SCL: U4.8 (SCL/SCK), U5.8 (SCL), U6.14 (SCL/SCLK), U7.1 (SCL/SPC), U8.7 (GPIO5)
- no-connect marks 41 -> 36
Other:
- note added: "CONTROL"
- note added: "SD CARD"
- note removed: "DATALOGGING"
- note removed: "MCU 2"
- moved on the sheet: C12, Card2, H10, H9

Commit message: more lyrav3 work
Parts:
- removed J13, J8: Conn_01x14, Connector_JST:JST_SUR_SM14B-SURS-TF_1x14-1MP_P0.80mm_Horizontal, symbol Connector_Generic:Conn_01x14
- added J1, J13: Conn_01x10, Connector_JST:JST_SUR_SM10B-SURS-TF_1x10-1MP_P0.80mm_Horizontal, symbol Connector_Generic:Conn_01x10
- added J8: Conn_01x12, Connector_JST:JST_SUR_SM12B-SURS-TF_1x12-1MP_P0.80mm_Horizontal, symbol Connector_Generic:Conn_01x12
- added U9: ADS1015IDGS, easyeda2kicad:X2QFN-10_L2.0-W1.5-P0.50-BL, symbol Analog_ADC:ADS1015IDGS
Connections:
- net +3V3: now also U10.8 (VDD), J1.9 (Pin_9), J13.2 (Pin_2), U9.1 (ADDR), U9.8 (VDD)
- net +5VD: now also J1.8 (Pin_8), J13.3 (Pin_3)
- net BATT SENSE BOT: now also U9.4 (AIN0)
- net GND: now also U10.1 (ADDR), U10.3 (GND), J1.1 (Pin_1), J1.10 (Pin_10), J13.1 (Pin_1), J13.10 (Pin_10), U9.3 (GND)
- net I2C1 SCL: now also J13.4 (Pin_4)
- net I2C1 SDA: now also J13.5 (Pin_5)
- net P1 CONT BOT: now also U10.4 (AIN0)
- net P2 CONT BOT: now also U10.5 (AIN1)
- net P3 CONT BOT: now also U10.6 (AIN2)
- net P4 CONT BOT: now also U10.7 (AIN3)
- net SERVO1: now also U8.15 (GPIO12), J13.6 (Pin_6); no longer J10.1
- net SERVO2: now also U8.16 (GPIO13), J13.7 (Pin_7); no longer J10.4
- net SERVO3: now also U8.17 (GPIO14), J13.8 (Pin_8); no longer J10.7
- net SERVO4: now also U8.18 (GPIO15), J13.9 (Pin_9); no longer J10.10
- net I2C1 SCL BOT: now reaches U10.10 (SCL)
- net I2C1 SCL BOT: now also J1.7 (Pin_7), U9.10 (SCL)
- net I2C1 SDA BOT: now reaches U10.9 (SDA)
- net I2C1 SDA BOT: now also J1.6 (Pin_6), U9.9 (SDA)
- net BATT SENSE: no longer names the net of U8.41 (GPIO29_ADC3)
- new net SERVO1 BOT: J1.5 (Pin_5), J10.1
- new net SERVO2 BOT: J1.4 (Pin_4), J10.4
- new net SERVO3 BOT: J1.3 (Pin_3), J10.7
- new net SERVO4 BOT: J1.2 (Pin_2), J10.10
- no-connect marks 36 -> 41

Commit message: aghjkl
Parts:
- added U11: PCF8574, Package_DFN_QFN:WQFN-16-1EP_3x3mm_P0.5mm_EP1.6x1.6mm, symbol Interface_Expansion:PCF8574
Connections:
- net BATT SENSE BOT: now also U10.6 (AIN2); no longer U9.4 (AIN0)
- net P3 CONT BOT: now also U9.4 (AIN0); no longer U10.6 (AIN2)
- net P4 CONT BOT: now also U9.5 (AIN1); no longer U10.7 (AIN3)
Changed lines of the file:
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@@
   )
   (no_connect (at 170.815 205.74))
-  (no_connect (at 368.3 276.86))
   (no_connect (at 282.575 102.235))
   (no_connect (at 232.41 334.01))
@@
   (no_connect (at 368.3 279.4))
   (no_connect (at 368.3 281.94))
+  (no_connect (at 425.45 283.845))
   (no_connect (at 88.9 396.875))
   (no_connect (at 283.21 298.45))
@@
     (stroke (width 0) (type default))
   )
+  (wire (pts (xy 352.425 276.86) (xy 368.3 276.86))
+    (stroke (width 0) (type default))
+  )
   (wire (pts (xy 282.575 201.9387) (xy 282.575 201.93))
     (stroke (width 0) (type default))
@@
     (stroke (width 0) (type default))
   )
+  (wire (pts (xy 425.45 281.305) (xy 409.575 281.305))
+    (stroke (width 0) (type default))
+  )
   (wire (pts (xy 253.365 250.825) (xy 261.62 250.825))
     (stroke (width 0) (type default))
@@
     (stroke (width 0) (type default))
   )
-  (wire (pts (xy 368.3 274.32) (xy 346.71 274.32))
-    (stroke (width 0) (type default))
-  )
   (wire (pts (xy 157.48 140.335) (xy 157.48 140.97))
     (stroke (width 0) (type default))
@@
     (stroke (width 0) (type default))
   )
+  (wire (pts (xy 352.425 274.32) (xy 368.3 274.32))
+    (stroke (width 0) (type default))
+  )
   (wire (pts (xy 163.83 267.97) (xy 165.735 267.97))
     (stroke (width 0) (type default))
@@
     (stroke (width 0) (type default))
   )
-  (wire (pts (xy 409.575 281.305) (xy 425.45 281.305))
-    (stroke (width 0) (type default))
-  )
   (wire (pts (xy 423.545 73.66) (xy 414.655 73.66))
     (stroke (width 0) (type default))
@@
     (stroke (width 0) (type default))
   )
-  (wire (pts (xy 409.575 283.845) (xy 425.45 283.845))
-    (stroke (width 0) (type default))
-  )
   (wire (pts (xy 374.015 40.64) (xy 367.665 40.64))
     (stroke (width 0) (type default))
@@
     (effects (font (size 1.27 1.27)) (justify left bottom))
   )
-  (label "P4 CONT BOT" (at 409.575 283.845 0) (fields_autoplaced)
-    (effects (font (size 1.27 1.27)) (justify left bottom))
-  )
   (label "LEDBLUE" (at 262.255 207.01 0) (fields_autoplaced)
     (effects (font (size 1.27 1.27)) (justify left bottom))
@@
     (effects (font (size 1.27 1.27)) (justify left bottom))
   )
-  (label "P3 CONT BOT" (at 409.575 281.305 0) (fields_autoplaced)
-    (effects (font (size 1.27 1.27)) (justify left bottom))
-  )
   (label "P3-" (at 496.57 305.435 0) (fields_autoplaced)
     (effects (font (size 1.27 1.27)) (justify left bottom))
@@
     (effects (font (size 1.27 1.27)) (justify left bottom))
   )
+  (label "P4 CONT BOT" (at 352.425 276.86 0) (fields_autoplaced)
+    (effects (font (size 1.27 1.27)) (justify left bottom))
+  )
   (label "I2C0 SCL" (at 172.085 100.33 0) (fields_autoplaced)
     (effects (font (size 1.27 1.27)) (justify left bottom))
@@
     (effects (font (size 1.27 1.27)) (justify left bottom))
   )
+  (label "BATT SENSE BOT" (at 409.575 281.305 0) (fields_autoplaced)
+    (effects (font (size 1.27 1.27)) (justify left bottom))
+  )
   (label "SERVO1" (at 292.1 308.61 180) (fields_autoplaced)
     (effects (font (size 1.27 1.27)) (justify right bottom))
   )
-  (label "BATT SENSE BOT" (at 346.71 274.32 0) (fields_autoplaced)
-    (effects (font (size 1.27 1.27)) (justify left bottom))
-  )
   (label "I2C1 SCL BOT" (at 530.225 267.97 180) (fields_autoplaced)
     (effects (font (size 1.27 1.27)) (justify right bottom))
@@
     (effects (font (size 1.27 1.27)) (justify right bottom))
   )
+  (label "P3 CONT BOT" (at 352.425 274.32 0) (fields_autoplaced)
+    (effects (font (size 1.27 1.27)) (justify left bottom))
+  )
   (label "SERVO2" (at 292.1 311.15 180) (fields_autoplaced)
     (effects (font (size 1.27 1.27)) (justify right bottom))
@@
         )
       )
+    )
+  )
+  (symbol (lib_id "Interface_Expansion:PCF8574") (at 403.86 327.025 0) (unit 1)
+    (in_bom yes) (on_board yes) (dnp no) (fields_autoplaced)
+    (property "Reference" "U11" (at 405.8159 307.34 0)
+      (effects (font (size 1.27 1.27)) (justify left))
+    )
+    (property "Value" "PCF8574" (at 405.8159 309.88 0)
+      (effects (font (size 1.27 1.27)) (justify left))
+    )
+    (property "Footprint" "Package_DFN_QFN:WQFN-16-1EP_3x3mm_P0.5mm_EP1.6x1.6mm" (at 403.86 327.025 0)
+      (effects (font (size 1.27 1.27)) hide)
+    )
+    (property "Datasheet" "http://www.nxp.com/documents/data_sheet/PCF8574_PCF8574A.pdf" (at 403.86 327.025 0)
+      (effects (font (size 1.27 1.27)) hide)
+    )
+    (pin "1")
+    (pin "10")
+    (pin "11")
+    (pin "12")
+    (pin "13")
+    (pin "14")
+    (pin "15")
+    (pin "16")
+    (pin "2")
+    (pin "3")
+    (pin "4")
+    (pin "5")
+    (pin "6")
+    (pin "7")
+    (pin "8")
+    (pin "9")
+    (instances
+      (project "Lyrav3"
+        (path "/12cc3c39-e34e-4801-bd3f-38f875d59424"
+          (reference "U11") (unit 1)
+        )
+      )
