File: avionics/kicad/Lyra_flight_computer/lyra V3/Lyrav3.kicad_sch (KiCad schematic)
At the start: 113 parts, among them J1 Conn_01x10, J10 TSW-104-08-T-T-RA, J11 Screw_Terminal_01x12, J12 Screw_Terminal_01x12, J13 Conn_01x10, J2 Conn_01x02, J3 Conn_01x04, J4 Conn_01x03, J5 Conn_01x04, J6 USB_B_Micro, J7 Conn_02x03_Odd_Even, J8 Conn_01x12, J9 Conn_01x02, Q1 AO3401A, Q2 KY6802, Q3 KY6802, U1 AMS1117-5.0, U10 ADS1015IDGS, U11 PCF8574, U2 AMS1117-3.3, U3 W25Q64JVXGIQ, U4 BMI088, U5 MPL3115A2, U6 ADXL375BCCZ-RL7, U7 LIS3MDL, U8 RP2040, U9 ADS1015IDGS, X1 S3D12.288000B20F30T

Commit message: more lyrav3 work
Parts:
- removed D1: D_Small, Diode_SMD:D_SOD-123, symbol Device:D_Small
- removed D4: LED, LED_SMD:LED_0805_2012Metric, symbol Device:LED
- removed J3, J5: Conn_01x04, Connector_JST:JST_SH_SM04B-SRSS-TB_1x04-1MP_P1.00mm_Horizontal, symbol Connector_Generic:Conn_01x04
- removed J7: Conn_02x03_Odd_Even, Connector_JST:JST_SH_SM06B-SRSS-TB_1x06-1MP_P1.00mm_Horizontal, symbol Connector_Generic:Conn_02x03_Odd_Even
- removed J8: Conn_01x12, Connector_JST:JST_SUR_SM12B-SURS-TF_1x12-1MP_P0.80mm_Horizontal, symbol Connector_Generic:Conn_01x12
- removed JP4: SolderJumper_3_Open, Jumper:SolderJumper-3_P1.3mm_Open_Pad1.0x1.5mm, symbol Jumper:SolderJumper_3_Open
- removed R28: 1k, Resistor_SMD:R_0402_1005Metric, symbol Device:R_Small
- removed TP1: TestPoint, TestPoint:TestPoint_Pad_1.0x1.0mm, symbol Connector:TestPoint
- added C1, C6: 100n, Capacitor_SMD:C_0402_1005Metric, symbol Device:C_Small
- added D4: D, Diode_SMD:D_0402_1005Metric, symbol Device:D
- added J3: Conn_01x07, Connector_JST:JST_SH_SM07B-SRSS-TB_1x07-1MP_P1.00mm_Horizontal, symbol Connector_Generic:Conn_01x07
- added J5, J8: Conn_01x05, Connector_JST:JST_SH_SM05B-SRSS-TB_1x05-1MP_P1.00mm_Horizontal, symbol Connector_Generic:Conn_01x05
- J2: footprint Jumper:SolderJumper-2_P1.3mm_Open_Pad1.0x1.5mm -> Jumper:SolderJumper-2_P1.3mm_Open_RoundedPad1.0x1.5mm
Connections:
- net GPIO28 BOT is gone; now on net +5VD: J11.6 (Pin_6)
- net SD CS BOT is gone; now on net SD CS: Card2.2 (CD/DAT3)
- net SPI1 MISO BOT is gone; now on net SPI0 MISO: Card2.7 (DAT0)
- net SPI1 MOSI BOT is gone; now on net SPI0 MOSI: Card2.3 (CMD)
- net SPI1 SCLK BOT is gone; now on net SPI0 SCK: Card2.5 (CLX)
- net UART PWR BOT is gone; now on net I2C PWR: JP1.2 (C)
- net +3V3: now also U11.16 (VDD), C1.1, C6.1
- net +5V: now also J13.3 (Pin_3), JP1.1 (A), D4.1 (K); no longer J12.2 (Pin_2)
- net +5VD: no longer J13.3 (Pin_3), JP1.1 (A)
- net GND: now also J12.2 (Pin_2), U11.1 (A0), U11.2 (A1), U11.3 (A2), U11.8 (VSS), C1.2, C6.2, J3.7 (Pin_7), J5.5 (Pin_5), J8.5 (Pin_5)
- net I2C PWR: now also J5.2 (Pin_2); no longer JP2.2 (C)
- net I2C1 SCL BOT: now also U11.14 (SCL), J5.3 (Pin_3)
- net I2C1 SDA BOT: now also U11.15 (SDA), J5.4 (Pin_4)
- net P1 EN BOT: now also U11.4 (P0)
- net P2 EN BOT: now also U11.5 (P1)
- net P3 EN BOT: now also U11.6 (P2)
- net P4 EN BOT: now also U11.7 (P3)
- net SPI0 CSn: now also J3.4 (Pin_4)
- net SPI0 MISO: now also J3.2 (Pin_2)
- net SPI0 MOSI: now also J3.3 (Pin_3)
- net SPI0 SCK: now also J3.5 (Pin_5)
- net UART PWR: now also J8.2 (Pin_2)
- net UART0 RX: now also J8.3 (Pin_3)
- net UART0 TX: now also J8.4 (Pin_4)
- net at J6.1 (VBUS): now also D4.2 (A)
- net ADC GPIO: now reaches U9.6 (AIN2)
- net ADC GPIO: now also J11.1 (Pin_1)
- net ADC2 GPIO: now reaches U9.7 (AIN3)
- net ADC2 GPIO: now also J11.2 (Pin_2)
- net GPIOUT1: now reaches U11.11 (P6)
- net GPIOUT1: now also J11.3 (Pin_3)
- net GPIOUT2: now reaches U11.12 (P7)
- net GPIOUT2: now also J11.4 (Pin_4)
- net I2C GPIO: now reaches U11.9 (P4)
- net I2C GPIO: now also J5.1 (Pin_1)
- net SPI0 GPIO: now reaches U8.2 (GPIO0)
- net SPI0 GPIO: now also J3.1 (Pin_1)
- net UART GPIO: now reaches U8.36 (GPIO24)
- net UART GPIO: now also J8.1 (Pin_1)
- net SD CS: now reaches U8.4 (GPIO2)
- new net SPI PWR: J3.6 (Pin_6), JP2.2 (C)
- no-connect marks 41 -> 37
Other:
- moved on the sheet: R2, R3

Commit message: simplified lyrav3
Parts:
- removed C12 (x2), C33: 1u, Capacitor_SMD:C_0402_1005Metric, symbol Device:C_Small
- removed C30, C32: 100n, Capacitor_SMD:C_0402_1005Metric, symbol Device:C_Small
- removed C31: 2u2, Capacitor_SMD:C_0402_1005Metric, symbol Device:C_Small
- removed Card2: TF-002-H18, easyeda2kicad:SIM-SMD_TF-002-H18, symbol easyeda2kicad:TF-002-H18
- removed D3: LED, LED_SMD:LED_0805_2012Metric, symbol Device:LED
- removed D4: D, Diode_SMD:D_0402_1005Metric, symbol Device:D
- removed F2: 200ma, Fuse:Fuse_0805_2012Metric, symbol Device:Fuse_Small
- removed FB1: FerriteBead_Small, Diode_SMD:D_0603_1608Metric, symbol Device:FerriteBead_Small
- removed H10, H9: Access Hole, customfootprints:1x10 2.54mm pitch acess hole, symbol Mechanical:MountingHole
- removed H5, H6, H7, H8: MountingHole_Pad, MountingHole:MountingHole_3.2mm_M3_DIN965_Pad, symbol Mechanical:MountingHole_Pad
- removed J1, J13: Conn_01x10, Connector_JST:JST_SUR_SM10B-SURS-TF_1x10-1MP_P0.80mm_Horizontal, symbol Connector_Generic:Conn_01x10
- removed J10: TSW-104-08-T-T-RA, SamacSys_Parts:HDRRA12W64P254_3X4_1016X254X810P, symbol SamacSys_Parts:TSW-104-08-T-T-RA
- removed J11, J12: Screw_Terminal_01x12, TerminalBlock_Phoenix:TerminalBlock_Phoenix_MPT-0,5-12-2.54_1x12_P2.54mm_Horizontal, symbol Connector:Screw_Terminal_01x12
- removed J2, J9: Conn_01x02, Jumper:SolderJumper-2_P1.3mm_Open_RoundedPad1.0x1.5mm, symbol Connector_Generic:Conn_01x02
- removed J3: Conn_01x07, Connector_JST:JST_SH_SM07B-SRSS-TB_1x07-1MP_P1.00mm_Horizontal, symbol Connector_Generic:Conn_01x07
- removed J4: Conn_01x03, Connector_JST:JST_SH_SM03B-SRSS-TB_1x03-1MP_P1.00mm_Horizontal, symbol Connector_Generic:Conn_01x03
- removed J5, J8: Conn_01x05, Connector_JST:JST_SH_SM05B-SRSS-TB_1x05-1MP_P1.00mm_Horizontal, symbol Connector_Generic:Conn_01x05
- removed J6: USB_B_Micro, easyeda2kicad:MICRO-USB-SMD_U254-051T-4BHJ25-F2S, symbol Connector:USB_B_Micro
- removed JP1, JP2, JP3, JP5: SolderJumper_3_Open, Jumper:SolderJumper-3_P1.3mm_Open_Pad1.0x1.5mm, symbol Jumper:SolderJumper_3_Open
- removed U1: AMS1117-5.0, Package_TO_SOT_SMD:SOT-89-3, symbol Regulator_Linear:AMS1117-5.0
- removed U10, U9: ADS1015IDGS, easyeda2kicad:X2QFN-10_L2.0-W1.5-P0.50-BL, symbol Analog_ADC:ADS1015IDGS
- removed U11: PCF8574, Package_DFN_QFN:WQFN-16-1EP_3x3mm_P0.5mm_EP1.6x1.6mm, symbol Interface_Expansion:PCF8574
- removed U2: AMS1117-3.3, Package_TO_SOT_SMD:SOT-89-3, symbol Regulator_Linear:AMS1117-3.3
- removed U3: W25Q64JVXGIQ, easyeda2kicad:XSON-8_L4.0-W4.0-P0.80-TL-EP, symbol easyeda2kicad:W25Q64JVXGIQ
- removed U4: BMI088, SnapEDA Library:PQFN50P450X300X100-16N, symbol BMI088:BMI088
- removed U5: MPL3115A2, Package_LGA:NXP_LGA-8_3x5mm_P1.25mm_H1.1mm, symbol Sensor_Pressure:MPL3115A2
- removed U6: ADXL375BCCZ-RL7, easyeda2kicad:LGA-14_L5.0-W3.0-P0.80-BL, symbol easyeda2kicad:ADXL375BCCZ-RL7
- removed U7: LIS3MDL, Package_LGA:LGA-12_2x2mm_P0.5mm, symbol Sensor_Magnetic:LIS3MDL
- added C12, C18: 1u, Capacitor_SMD:C_0402_1005Metric, symbol Device:C_Small
- added D1: LED, LED_SMD:LED_0805_2012Metric, symbol Device:LED
- added D3: D, Diode_SMD:D_0402_1005Metric, symbol Device:D
- added J1: Screw_Terminal_01x08, TerminalBlock_Phoenix:TerminalBlock_Phoenix_MPT-0,5-8-2.54_1x08_P2.54mm_Horizontal, symbol Connector:Screw_Terminal_01x08
- added J2: Screw_Terminal_01x06, TerminalBlock_Phoenix:TerminalBlock_Phoenix_MPT-0,5-6-2.54_1x06_P2.54mm_Horizontal, symbol Connector:Screw_Terminal_01x06
- added J3, J4: Conn_01x02, Jumper:SolderJumper-2_P1.3mm_Open_RoundedPad1.0x1.5mm, symbol Connector_Generic:Conn_01x02
- added J5: Conn_01x03, Connector_JST:JST_SH_SM03B-SRSS-TB_1x03-1MP_P1.00mm_Horizontal, symbol Connector_Generic:Conn_01x03
- added J6: Conn_01x06, Connector_PinHeader_2.54mm:PinHeader_1x06_P2.54mm_Vertical, symbol Connector_Generic:Conn_01x06
- added J7: USB_B_Micro, easyeda2kicad:MICRO-USB-SMD_U254-051T-4BHJ25-F2S, symbol Connector:USB_B_Micro
- added J8: Conn_01x04, Connector_PinHeader_2.54mm:PinHeader_1x04_P2.54mm_Vertical, symbol Connector_Generic:Conn_01x04
- added U2: BMI088, easyeda2kicad:LGA-16_L4.5-W3.0-P0.50-BL, symbol BMI088:BMI088
- added U3: MPL3115A2, Package_LGA:NXP_LGA-8_3x5mm_P1.25mm_H1.1mm, symbol Sensor_Pressure:MPL3115A2
- added U4: ADXL375BCCZ-RL7, easyeda2kicad:LGA-14_L5.0-W3.0-P0.80-BL, symbol easyeda2kicad:ADXL375BCCZ-RL7
- added U5: LIS3MDL, Package_LGA:LGA-12_2x2mm_P0.5mm, symbol Sensor_Magnetic:LIS3MDL
- added U6: ADS1015IDGS, easyeda2kicad:X2QFN-10_L2.0-W1.5-P0.50-BL, symbol Analog_ADC:ADS1015IDGS
- added U7: W25Q64JVXGIQ, easyeda2kicad:XSON-8_L4.0-W4.0-P0.80-TL-EP, symbol easyeda2kicad:W25Q64JVXGIQ
- added U9: LDK130-33_SOT23_SOT353, easyeda2kicad:SOT-23-5_L3.0-W1.6-P0.95-LS2.8-BL, symbol Regulator_Linear:LDK130-33_SOT23_SOT353
- C10: value 10u -> 1u; footprint Capacitor_SMD:C_0603_1608Metric -> Capacitor_SMD:C_0402_1005Metric
- C11: value 10u -> 100n; footprint Capacitor_SMD:C_0603_1608Metric -> Capacitor_SMD:C_0402_1005Metric
- C14, C16, C22, C23: value 1u -> 100n
- C19, C6, C8: value 100n -> 1u
- C2, C3: value 22u -> 100n; footprint Capacitor_SMD:C_0603_1608Metric -> Capacitor_SMD:C_0402_1005Metric
- C27: value 100n -> 2u2
- C4: value 22u -> 10u
- C5: value 22u -> 1u; footprint Capacitor_SMD:C_0603_1608Metric -> Capacitor_SMD:C_0402_1005Metric
- C7: value 100n -> 10u; footprint Capacitor_SMD:C_0402_1005Metric -> Capacitor_SMD:C_0603_1608Metric
- F1: value 2a -> 200ma; footprint Fuse:Fuse_1812_4532Metric -> Fuse:Fuse_0805_2012Metric; LCSC Part (none) -> C883104
- R10: value 6k -> 20k
- R11, R23: value 470R -> 20k
- R12, R24: value 470R -> 6k
- R13: value 2k2 -> 6k; LCSC Part C163447 -> (none)
- R14: value 2k2 -> 10k; LCSC Part C163447 -> C375970
- R15: value 10R -> 27R; LCSC Part (none) -> C2909343
- R16: value 10R -> 470R
- R17: value 20k -> 470R
- R18: value 20k -> 27R; LCSC Part (none) -> C2909343
- R19, R20, R9: value 6k -> 10R
- R2: value 20k -> 1k
- R21: value 27R -> 20k; LCSC Part C2909343 -> (none)
- R22: value 27R -> 1k; LCSC Part C2909343 -> (none)
- R25: value 10k -> 6k; LCSC Part C375970 -> (none)
- R26, R27: value 1k -> 470R
- R3: value 6k -> 1k
- R4: value 1k -> 20k
- R5: value 10R -> 6k
- R6: value 10R -> 2k2; LCSC Part (none) -> C163447
- R7: value 20k -> 2k2; LCSC Part (none) -> C163447
- R8: value 20k -> 10R
Connections:
- net +5VD is gone; now on net +3V3: C3.1
- net UART GPIO is gone; now on net LEDGREEN: U8.36 (GPIO24)
- net +12P: now also F1.1, Q1.2 (S), J2.2 (Pin_2); no longer F1.2
- net +12V: now also R4.1, D3.1 (K), J2.3 (Pin_3); no longer R2.1
- net +12VA: now also C5.1, C7.1, C8.1, F1.2, J6.4 (Pin_4), U9.1 (IN), U9.3 (EN); no longer C11.1, C2.1, C4.1
- net +1V1: now also C16.1, C17.1, C18.1; no longer C20.1, C21.1, C22.1
- net +3V3: now also C11.1, C13.1, C19.1, C2.1, C20.1, C21.1, C22.1, C4.1, R2.2, R3.2, R6.1, R7.1, C12.1, J6.5 (Pin_5), U2.11 (VDDIO), U2.14 (CSB1), U2.3 (VDD), U2.7 (PS), U3.1 (VDD), U3.4 (VDDIO), U4.1 (VDDI/O), U4.3 (RESERVED), U4.6 (VS), U4.7 (~{CS}), U5.10 (~{CS}), U5.5 (Vdd), U5.6 (Vdd_IO), U6.1 (ADDR), U6.8 (VDD), U7.8 (VCC), U9.5 (OUT); no longer C14.1, C16.1, C17.1, C29.1, C5.1, C7.1, C8.1, C9.1, R13.1, R25.1, R27.2, R4.2
- net +BATT: now also J2.4 (Pin_4), J2.6 (Pin_6)
- net BOOTSEL: now also R22.2, J4.2 (Pin_2); no longer R26.2
- net GND: now also R12.2, R13.2, R16.1, R17.1, R24.2, R25.2, R26.1, R27.1, R5.2, C12.2, C18.2, D1.1 (K), J2.5 (Pin_5), J3.2 (Pin_2), J4.1 (Pin_1), J5.2 (Pin_2), J6.6 (Pin_6), J7.5 (GND), U2.10 (SDO2), U2.15 (SDO1), U2.4 (GNDA), U2.6 (GNDIO), U3.3 (GND), U4.11 (RESERVED), U4.12 (SDO/ALTADDRESS), U4.2 (GND), U4.4 (GND), U4.5 (GND), U5.12 (GND), U5.2 (GND), U5.3 (GND), U5.9 (SDO/SA1), U6.3 (GND), U7.4 (GND); no longer C29.2, C5.2, C6.2, R10.2, R11.1, R12.1, R19.2, R20.2, R23.1, R24.1, R3.2, R9.2
- net I2C0 SCL: now also U2.8 (SCL/SCK), U3.8 (SCL), U4.14 (SCL/SCLK), U5.1 (SCL/SPC)
- net I2C0 SDA: now also U2.9 (SDA/SDI), U3.7 (SDL), U4.13 (SDA/SDI/SDIO), U5.11 (SDA/SDI/SDO)
- net I2C1 SCL: now also R6.2, U6.10 (SCL); no longer R13.2, U8.35 (GPIO23)
- net I2C1 SDA: now also R7.2, U6.9 (SDA); no longer R14.2, U8.34 (GPIO22)
- net LEDBLUE: now also U8.37 (GPIO25); no longer U8.14 (GPIO11)
- net LEDGREEN: no longer U8.13 (GPIO10)
- net LEDRED: now also U8.35 (GPIO23); no longer U8.12 (GPIO9)
- net P1-: now also R8.1, J1.7 (Pin_7); no longer R5.1
- net P2-: now also R19.1, J1.5 (Pin_5); no longer R15.1
- net P3-: now also R9.1, J1.3 (Pin_3); no longer R6.1
- net P4-: now also R20.1, J1.1 (Pin_1); no longer R16.1
- net PYRO PWR: now also J1.2 (Pin_2), J1.4 (Pin_4), J1.6 (Pin_6), J1.8 (Pin_8), J2.1 (Pin_1)
- net QSPI_SCLK: now also U7.6 (CLK)
- net QSPI_SD1: now also U7.2 (DO(IO1))
- net QSPI_SD2: now also U7.3 (IO2)
- net QSPI_SD3: now also U7.7 (IO3)
- net QSPI_SDO: now also U7.5 (DI(IO0))
- net QSPI_SS: now also R22.1, U7.1 (~{CS}); no longer R26.1
- net RP USB_D+: now also R15.2; no longer R21.2
- net RP USB_D-: now also R18.1; no longer R22.1
- net RUN: now also R14.2, J3.1 (Pin_1); no longer R25.2
- net SWCLK: now also J5.1 (Pin_1)
- net SWD: now also J5.3 (Pin_3)
- net USB_D+: now also R15.1, J7.3 (D+); no longer R21.1
- net USB_D-: now also R18.2, J7.2 (D-); no longer R22.2
- net at LED1.4 (+), LED1.5 (+), LED1.6 (+): now also R2.1; no longer R4.1
- net at D2.2 (A): now also R3.1; no longer R1.1
- net BRKOUT2: now reaches U8.3 (GPIO1)
- net BRKOUT2: now also J8.3 (Pin_3)
- net BATT SENSE : now reaches U8.40 (GPIO28_ADC2)
- net BATT SENSE : now also R4.2, R5.1
- net BRKOUT4: now reaches U8.5 (GPIO3)
- net BRKOUT4: now also J8.1 (Pin_1)
- removed net BATT SENSE BOT: R2.2, R3.1
- removed net P1 CONT BOT: R7.2, R9.1
- net P1 EN BOT renamed P1 EN 
- net P1 EN : now also R16.2; no longer R11.2
- net P2 CONT BOT renamed P3 EN 
- net P3 EN : now also Q3.1 (G); no longer R19.1
- net P2 EN BOT renamed P2 EN 
- net P2 EN : now also R26.2; no longer R23.2
- net P3 CONT BOT: no longer names the net of R10.1, R8.2
- net P3 CONT BOT: now also Q2.6 (D)
- removed net P3 EN BOT: Q3.1 (G), R12.2
- removed net P4 CONT BOT: R18.2, R20.1
- net P4 EN BOT renamed P4 EN 
- net P4 EN : now also R27.2; no longer R24.2
- net SD CS renamed BRKOUT3
- net BRKOUT3: now also J8.2 (Pin_2)
- net SERVO1: no longer names the net of U8.15 (GPIO12)
- net SERVO2 renamed BRKOUT5
- net BRKOUT5: now also J6.1 (Pin_1)
- net SERVO3 renamed BRKOUT6
- net BRKOUT6: now also J6.2 (Pin_2)
- net SERVO4 renamed BRKOUT7
- net BRKOUT7: now also J6.3 (Pin_3)
- net SPI0 CSn: no longer names the net of U8.32 (GPIO21)
- net SPI0 GPIO renamed BRKOUT1
- net BRKOUT1: now also J8.4 (Pin_4)
- net SPI0 MISO: no longer names the net of U8.30 (GPIO19)
- net SPI0 MOSI: no longer names the net of U8.31 (GPIO20)
- net SPI0 SCK: no longer names the net of U8.29 (GPIO18)
- net UART0 RX: no longer names the net of U8.28 (GPIO17)
- net UART0 TX: no longer names the net of U8.27 (GPIO16)
- new net: D3.2 (A), J7.1 (VBUS)
- new net: Q2.4 (D), R19.2, R21.1
- new net: Q3.6 (D), R11.1, R9.2
- new net: Q3.4 (D), R20.2, R23.1
- new net: C29.2, C5.2, C6.2, U9.2 (GND)
- new net: C14.1, U5.4 (C1)
- new net: C9.1, U3.2 (CAP)
- new net: D1.2 (A), R1.1
- new net: C29.1, U9.4 (BP)
- new net P1 CONT : R10.2, R12.1, U6.4 (AIN0)
- new net P2 CONT : R21.2, R24.1, U6.5 (AIN1)
- new net P3 CONT : R11.2, R13.1, U6.6 (AIN2)
- new net P4 CONT : R23.2, R25.1, U6.7 (AIN3)
- no-connect marks 37 -> 34
Other:
- note removed: "BOTTOM BOARD"
- note removed: "CONTROL"
- note removed: "INTERCONNECT"
- note removed: "SD CARD"
- note removed: "TOP BOARD"

Commit message: lyrav3 work
Parts:
- removed D1: LED, LED_SMD:LED_0805_2012Metric, symbol Device:LED
- removed R1: 1k, Resistor_SMD:R_0402_1005Metric, symbol Device:R_Small
Connections:
- net I2C1 SCL is gone; now on net I2C0 SCL: R6.2, U6.10 (SCL)
- net I2C1 SDA is gone; now on net I2C0 SDA: R7.2, U6.9 (SDA)
- net GND: now also C29.2, C5.2, C6.2, U9.2 (GND)
Changed lines of the file:
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@@
   (no_connect (at 175.895 215.265))
   (no_connect (at 175.895 238.125))
-  (no_connect (at 175.895 207.645))
   (no_connect (at 108.585 64.77))
   (no_connect (at 175.895 230.505))
@@
   (no_connect (at 217.17 267.335))
   (no_connect (at 108.585 52.07))
-  (no_connect (at 175.895 210.185))
   (no_connect (at 144.145 54.61))
   (no_connect (at 175.895 263.525))
@@
   (no_connect (at 125.095 243.205))
   (no_connect (at 175.895 235.585))
+  (no_connect (at 175.895 210.185))
   (no_connect (at 158.115 117.475))
   (no_connect (at 175.895 212.725))
@@
   (no_connect (at 144.145 62.23))
   (no_connect (at 158.115 114.935))
+  (no_connect (at 175.895 207.645))
   (wire (pts (xy 106.045 102.235) (xy 109.855 102.235))
     (stroke (width 0) (type default))
@@
     (stroke (width 0) (type default))
   )
-  (wire (pts (xy 215.9 21.59) (xy 215.9 22.86))
-    (stroke (width 0) (type default))
-  )
   (wire (pts (xy 352.425 186.69) (xy 352.425 187.325))
     (stroke (width 0) (type default))
@@
     (stroke (width 0) (type default))
   )
-  (wire (pts (xy 215.9 29.21) (xy 215.9 27.94))
-    (stroke (width 0) (type default))
-  )
   (wire (pts (xy 314.96 180.34) (xy 325.755 180.34))
     (stroke (width 0) (type default))
@@
     (stroke (width 0) (type default))
   )
-  (wire (pts (xy 215.9 36.83) (xy 215.9 38.1))
-    (stroke (width 0) (type default))
-  )
   (wire (pts (xy 207.645 203.835) (xy 212.725 203.835))
     (stroke (width 0) (type default))
@@
     (fill (type none))
   )
-  (rectangle (start 362.585 109.22) (end 407.67 159.385)
-    (stroke (width 0) (type default))
-    (fill (type none))
-  )
   (rectangle (start 222.885 12.7) (end 346.075 70.485)
     (stroke (width 0) (type default))
@@
     (effects (font (size 2.54 2.54)) (justify left bottom))
   )
-  (label "I2C1 SCL" (at 203.2 172.085 0) (fields_autoplaced)
+  (label "I2C0 SCL" (at 203.2 172.085 0) (fields_autoplaced)
     (effects (font (size 1.27 1.27)) (justify left bottom))
   )
@@
     (effects (font (size 1.27 1.27)) (justify left bottom))
   )
-  (label "I2C1 SDA" (at 231.14 169.545 180) (fields_autoplaced)
+  (label "I2C0 SDA" (at 231.14 169.545 180) (fields_autoplaced)
     (effects (font (size 1.27 1.27)) (justify right bottom))
   )
@@
     (effects (font (size 1.27 1.27)) (justify left bottom))
   )
-  (label "I2C1 SCL" (at 231.14 172.085 180) (fields_autoplaced)
+  (label "I2C0 SCL" (at 231.14 172.085 180) (fields_autoplaced)
     (effects (font (size 1.27 1.27)) (justify right bottom))
   )
@@
     (effects (font (size 1.27 1.27)) (justify left bottom))
   )
-  (label "I2C1 SDA" (at 356.235 141.605 180) (fields_autoplaced)
+  (label "I2C0 SDA" (at 356.235 141.605 180) (fields_autoplaced)
     (effects (font (size 1.27 1.27)) (justify right bottom))
   )
@@
     (effects (font (size 1.27 1.27)) (justify left bottom))
   )
-  (label "I2C1 SDA" (at 203.2 169.545 0) (fields_autoplaced)
+  (label "I2C0 SDA" (at 203.2 169.545 0) (fields_autoplaced)
     (effects (font (size 1.27 1.27)) (justify left bottom))
   )
@@
     (effects (font (size 1.27 1.27)) (justify left bottom))
   )
-  (label "I2C1 SCL" (at 356.235 139.065 180) (fields_autoplaced)
+  (label "I2C0 SCL" (at 356.235 139.065 180) (fields_autoplaced)
     (effects (font (size 1.27 1.27)) (justify right bottom))
   )
@@
     )
   )
-  (symbol (lib_id "power:GND") (at 215.9 38.1 0) (unit 1)
-    (in_bom yes) (on_board yes) (dnp no) (fields_autoplaced)
-    (property "Reference" "#PWR010" (at 215.9 44.45 0)
-      (effects (font (size 1.27 1.27)) hide)
-    )
-    (property "Value" "GND" (at 215.9 43.18 0)
-      (effects (font (size 1.27 1.27)))
-    )
-    (property "Footprint" "" (at 215.9 38.1 0)
-      (effects (font (size 1.27 1.27)) hide)
-    )
-    (property "Datasheet" "" (at 215.9 38.1 0)
-      (effects (font (size 1.27 1.27)) hide)
-    )
-    (pin "1")
-    (instances
-      (project "Lyrav3"
-        (path "/12cc3c39-e34e-4801-bd3f-38f875d59424"
-          (reference "#PWR010") (unit 1)
-        )
-      )
-      (project "Lyra V2"
-        (path "/63622aab-8dfa-4523-a589-40aebeb23162"
-          (reference "#PWR04") (unit 1)
-        )
-      )
-    )
-  )
   (symbol (lib_id "Device:R_Small") (at 351.79 220.345 0) (unit 1)
     (in_bom yes) (on_board yes) (dnp no) (fields_autoplaced)
@@
     )
   )
-  (symbol (lib_id "power:+3V3") (at 215.9 21.59 0) (unit 1)
-    (in_bom yes) (on_board yes) (dnp no) (fields_autoplaced)
-    (property "Reference" "#PWR01" (at 215.9 25.4 0)
-      (effects (font (size 1.27 1.27)) hide)
-    )
-    (property "Value" "+3V3" (at 215.9 17.78 0)
-      (effects (font (size 1.27 1.27)))
-    )
-    (property "Footprint" "" (at 215.9 21.59 0)
-      (effects (font (size 1.27 1.27)) hide)
-    )
-    (property "Datasheet" "" (at 215.9 21.59 0)
-      (effects (font (size 1.27 1.27)) hide)
-    )
-    (pin "1")
-    (instances
-      (project "Lyrav3"
-        (path "/12cc3c39-e34e-4801-bd3f-38f875d59424"
-          (reference "#PWR01") (unit 1)
-        )
-      )
-      (project "Lyra V2"
-        (path "/63622aab-8dfa-4523-a589-40aebeb23162"
-          (reference "#PWR03") (unit 1)
-        )
-      )
-    )
-  )
   (symbol (lib_id "Device:C_Small") (at 245.745 30.48 0) (unit 1)
     (in_bom yes) (on_board yes) (dnp no) (fields_autoplaced)
@@
     )
   )
+  (symbol (lib_id "power:GND") (at 266.7 34.925 0) (unit 1)
+    (in_bom yes) (on_board yes) (dnp no) (fields_autoplaced)
+    (property "Reference" "#PWR08" (at 266.7 41.275 0)
+      (effects (font (size 1.27 1.27)) hide)
+    )
+    (property "Value" "GND" (at 266.7 40.005 0)
+      (effects (font (size 1.27 1.27)))
+    )
+    (property "Footprint" "" (at 266.7 34.925 0)
+      (effects (font (size 1.27 1.27)) hide)
+    )
+    (property "Datasheet" "" (at 266.7 34.925 0)
+      (effects (font (size 1.27 1.27)) hide)
+    )
+    (pin "1")
+    (instances
+      (project "Lyrav3"
+        (path "/12cc3c39-e34e-4801-bd3f-38f875d59424"
+          (reference "#PWR08") (unit 1)
+        )
+      )
+      (project "Board2"
+        (path "/3ee99ce6-1aa5-40d1-bb2e-7887993edb74"
+          (reference "#PWR032") (unit 1)
+        )
+      )
+      (project "Lyra V2"
+        (path "/63622aab-8dfa-4523-a589-40aebeb23162"
+          (reference "#PWR09") (unit 1)
+        )
+      )
+    )
+  )
   (symbol (lib_id "power:GND") (at 158.75 48.26 0) (unit 1)
     (in_bom yes) (on_board yes) (dnp no) (fields_autoplaced)
@@
     )
   )
-  (symbol (lib_id "Device:R_Small") (at 215.9 25.4 180) (unit 1)
-    (in_bom yes) (on_board yes) (dnp no) (fields_autoplaced)
-    (property "Reference" "R1" (at 217.805 24.765 0)
-      (effects (font (size 1.27 1.27)) (justify right))
-    )
-    (property "Value" "1k" (at 217.805 27.305 0)
-      (effects (font (size 1.27 1.27)) (justify right))
-    )
-    (property "Footprint" "Resistor_SMD:R_0402_1005Metric" (at 215.9 25.4 0)
-      (effects (font (size 1.27 1.27)) hide)
-    )
-    (property "Datasheet" "~" (at 215.9 25.4 0)
-      (effects (font (size 1.27 1.27)) hide)
-    )
-    (property "LCSC Part" "" (at 215.9 25.4 0)
-      (effects (font (size 1.27 1.27)) hide)
-    )
-    (property "LCSC_Part" "" (at 215.9 25.4 0)
-      (effects (font (size 1.27 1.27)) hide)
-    )
-    (pin "1")
-    (pin "2")
-    (instances
-      (project "Lyrav3"
-        (path "/12cc3c39-e34e-4801-bd3f-38f875d59424"
-          (reference "R1") (unit 1)
-        )
-      )
-      (project "Lyra V2"
-        (path "/63622aab-8dfa-4523-a589-40aebeb23162"
-          (reference "R1") (unit 1)
-        )
-      )
-    )
-  )
   (symbol (lib_id "Transistor_FET:AO3401A") (at 283.845 57.15 90) (unit 1)
     (in_bom yes) (on_board yes) (dnp no) (fields_autoplaced)
@@
         )
       )
-    )
-  )
-  (symbol (lib_id "Device:LED") (at 215.9 33.02 90) (unit 1)
-    (in_bom yes) (on_board yes) (dnp no)
-    (property "Reference" "D1" (at 212.725 35.2425 90)
-      (effects (font (size 1.27 1.27)) (justify left))
-    )
-    (property "Value" "LED" (at 212.725 33.02 90)
-      (effects (font (size 1.27 1.27)) (justify left))
-    )
-    (property "Footprint" "LED_SMD:LED_0805_2012Metric" (at 215.9 33.02 0)
-      (effects (font (size 1.27 1.27)) hide)
-    )
-    (property "Datasheet" "~" (at 215.9 33.02 0)
-      (effects (font (size 1.27 1.27)) hide)
-    )
-    (property "LCSC Part" "" (at 215.9 33.02 90)
-      (effects (font (size 1.27 1.27)) hide)
-    )
-    (pin "1")
-    (pin "2")
-    (instances
-      (project "Lyrav3"
-        (path "/12cc3c39-e34e-4801-bd3f-38f875d59424"
-          (reference "D1") (unit 1)
-        )
-      )
-      (project "Lyra V2"
-        (path "/63622aab-8dfa-4523-a589-40aebeb23162"
-          (reference "D2") (unit 1)
-        )
-      )
