File: avionics/kicad/Lyra_flight_computer/lyra V3/Lyrav3.kicad_sch (KiCad schematic)
At the start: 84 parts, among them J1 Screw_Terminal_01x08, J2 Screw_Terminal_01x06, J3 Conn_01x02, J4 Conn_01x02, J5 Conn_01x03, J6 Conn_01x06, J7 USB_B_Micro, J8 Conn_01x04, Q1 AO3401A, Q2 AO3400A, Q3 AO3400A, Q4 AO3400A, Q5 AO3400A, U1 AZ1117-3.3, U2 BMI088, U3 MPL3115A2, U4 ADXL375BCCZ-RL7, U5 LIS3MDL, U6 ADS1015IDGS, U7 W25Q64JVXGIQ, U8 RP2040, X1 S3D12.288000B20F30T

Commit message: more lyrav3 work
Parts:
- removed J1: Screw_Terminal_01x08, TerminalBlock_Phoenix:TerminalBlock_Phoenix_MPT-0,5-8-2.54_1x08_P2.54mm_Horizontal, symbol Connector:Screw_Terminal_01x08
- added J9: Screw_Terminal_01x06, TerminalBlock_Phoenix:TerminalBlock_Phoenix_MPT-0,5-6-2.54_1x06_P2.54mm_Horizontal, symbol Connector:Screw_Terminal_01x06
- J5: footprint Connector_JST:JST_SH_SM03B-SRSS-TB_1x03-1MP_P1.00mm_Horizontal -> Connector_PinHeader_2.00mm:PinHeader_1x03_P2.00mm_Vertical
Connections:
- net +12P: no longer J2.2 (Pin_2)
- net P1-: now also J9.5 (Pin_5)
- net P2-: now also J9.3 (Pin_3)
- net P3-: now also J9.1 (Pin_1)
- net P4-: now also J2.1 (Pin_1)
- net PYRO PWR: now also J2.2 (Pin_2), J9.2 (Pin_2), J9.4 (Pin_4), J9.6 (Pin_6); no longer J2.1 (Pin_1)
Changed lines of the file:
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@@
     (stroke (width 0) (type default))
   )
-  (wire (pts (xy 217.805 88.265) (xy 227.965 88.265))
+  (wire (pts (xy 205.74 92.71) (xy 195.58 92.71))
     (stroke (width 0) (type default))
   )
@@
     (stroke (width 0) (type default))
   )
-  (wire (pts (xy 224.155 85.725) (xy 227.965 85.725))
+  (wire (pts (xy 199.39 90.17) (xy 195.58 90.17))
     (stroke (width 0) (type default))
   )
@@
     (stroke (width 0) (type default))
   )
-  (wire (pts (xy 217.805 103.505) (xy 227.965 103.505))
-    (stroke (width 0) (type default))
-  )
   (wire (pts (xy 175.26 38.1) (xy 184.785 38.1))
     (stroke (width 0) (type default))
@@
     (stroke (width 0) (type default))
   )
+  (wire (pts (xy 224.155 100.965) (xy 227.965 100.965))
+    (stroke (width 0) (type default))
+  )
   (wire (pts (xy 360.68 191.135) (xy 367.03 191.135))
     (stroke (width 0) (type default))
@@
     (stroke (width 0) (type default))
   )
+  (wire (pts (xy 217.805 103.505) (xy 227.965 103.505))
+    (stroke (width 0) (type default))
+  )
   (wire (pts (xy 342.9 144.145) (xy 342.9 149.225))
     (stroke (width 0) (type default))
@@
     (stroke (width 0) (type default))
   )
-  (wire (pts (xy 224.155 100.965) (xy 227.965 100.965))
-    (stroke (width 0) (type default))
-  )
   (wire (pts (xy 142.875 24.13) (xy 142.875 25.4))
     (stroke (width 0) (type default))
@@
     (stroke (width 0) (type default))
   )
-  (wire (pts (xy 195.58 92.71) (xy 201.93 92.71))
-    (stroke (width 0) (type default))
-  )
   (wire (pts (xy 182.245 197.485) (xy 175.895 197.485))
     (stroke (width 0) (type default))
@@
     (stroke (width 0) (type default))
   )
-  (wire (pts (xy 195.58 90.17) (xy 213.995 90.17))
-    (stroke (width 0) (type default))
-  )
   (wire (pts (xy 175.895 263.525) (xy 186.69 263.525))
     (stroke (width 0) (type default))
@@
     (effects (font (size 1.27 1.27)) (justify right bottom))
   )
-  (label "P1-" (at 224.155 100.965 0) (fields_autoplaced)
-    (effects (font (size 1.27 1.27)) (justify left bottom))
-  )
   (label "QSPI_SD1" (at 42.545 212.725 0) (fields_autoplaced)
     (effects (font (size 1.27 1.27)) (justify left bottom))
@@
     (effects (font (size 1.27 1.27)) (justify right bottom))
   )
-  (label "PYRO PWR" (at 217.805 103.505 0) (fields_autoplaced)
-    (effects (font (size 1.27 1.27)) (justify left bottom))
-  )
   (label "BUZZER" (at 186.69 240.665 180) (fields_autoplaced)
     (effects (font (size 1.27 1.27)) (justify right bottom))
@@
     (effects (font (size 1.27 1.27)) (justify right bottom))
   )
+  (label "P1-" (at 224.155 100.965 0) (fields_autoplaced)
+    (effects (font (size 1.27 1.27)) (justify left bottom))
+  )
   (label "BRKOUT6" (at 266.7 243.205 0) (fields_autoplaced)
     (effects (font (size 1.27 1.27)) (justify left bottom))
@@
     (effects (font (size 1.27 1.27)) (justify right bottom))
   )
-  (label "P4-" (at 224.155 85.725 0) (fields_autoplaced)
-    (effects (font (size 1.27 1.27)) (justify left bottom))
+  (label "P4-" (at 199.39 90.17 180) (fields_autoplaced)
+    (effects (font (size 1.27 1.27)) (justify right bottom))
   )
   (label "RP USB_D+" (at 113.665 194.945 0) (fields_autoplaced)
@@
     (effects (font (size 1.27 1.27)) (justify left bottom))
   )
+  (label "PYRO PWR" (at 217.805 103.505 0) (fields_autoplaced)
+    (effects (font (size 1.27 1.27)) (justify left bottom))
+  )
   (label "LEDGREEN" (at 175.26 38.1 0) (fields_autoplaced)
     (effects (font (size 1.27 1.27)) (justify left bottom))
@@
     (effects (font (size 1.27 1.27)) (justify left bottom))
   )
-  (label "PYRO PWR" (at 213.995 90.17 180) (fields_autoplaced)
-    (effects (font (size 1.27 1.27)) (justify right bottom))
-  )
   (label "LEDBLUE" (at 175.26 43.18 0) (fields_autoplaced)
     (effects (font (size 1.27 1.27)) (justify left bottom))
@@
     (effects (font (size 1.27 1.27)) (justify right bottom))
   )
-  (label "PYRO PWR" (at 217.805 88.265 0) (fields_autoplaced)
-    (effects (font (size 1.27 1.27)) (justify left bottom))
+  (label "PYRO PWR" (at 205.74 92.71 180) (fields_autoplaced)
+    (effects (font (size 1.27 1.27)) (justify right bottom))
   )
   (label "QSPI_SCLK" (at 90.805 215.265 180) (fields_autoplaced)
@@
     )
   )
-  (symbol (lib_id "Connector:Screw_Terminal_01x08") (at 233.045 93.345 0) (unit 1)
-    (in_bom no) (on_board yes) (dnp no) (fields_autoplaced)
-    (property "Reference" "J1" (at 236.22 93.345 0)
-      (effects (font (size 1.27 1.27)) (justify left))
-    )
-    (property "Value" "Screw_Terminal_01x08" (at 236.22 95.885 0)
-      (effects (font (size 1.27 1.27)) (justify left))
-    )
-    (property "Footprint" "TerminalBlock_Phoenix:TerminalBlock_Phoenix_MPT-0,5-8-2.54_1x08_P2.54mm_Horizontal" (at 233.045 93.345 0)
-      (effects (font (size 1.27 1.27)) hide)
-    )
-    (property "Datasheet" "~" (at 233.045 93.345 0)
-      (effects (font (size 1.27 1.27)) hide)
-    )
-    (pin "1")
-    (pin "2")
-    (pin "3")
-    (pin "4")
-    (pin "5")
-    (pin "6")
-    (pin "7")
-    (pin "8")
-    (instances
-      (project "Lyrav3"
-        (path "/12cc3c39-e34e-4801-bd3f-38f875d59424"
-          (reference "J1") (unit 1)
-        )
-      )
-    )
-  )
   (symbol (lib_id "power:+3V3") (at 55.88 98.425 0) (unit 1)
     (in_bom yes) (on_board yes) (dnp no) (fields_autoplaced)
@@
       (effects (font (size 1.27 1.27)))
     )
-    (property "Footprint" "Connector_JST:JST_SH_SM03B-SRSS-TB_1x03-1MP_P1.00mm_Horizontal" (at 210.185 241.3 0)
+    (property "Footprint" "Connector_PinHeader_2.00mm:PinHeader_1x03_P2.00mm_Vertical" (at 210.185 241.3 0)
       (effects (font (size 1.27 1.27)) hide)
     )
@@
     )
   )
+  (symbol (lib_id "Connector:Screw_Terminal_01x06") (at 233.045 95.885 0) (unit 1)
+    (in_bom no) (on_board yes) (dnp no)
+    (property "Reference" "J9" (at 233.045 85.09 0)
+      (effects (font (size 1.27 1.27)))
+    )
+    (property "Value" "Screw_Terminal_01x06" (at 233.045 87.63 0)
+      (effects (font (size 1.27 1.27)))
+    )
+    (property "Footprint" "TerminalBlock_Phoenix:TerminalBlock_Phoenix_MPT-0,5-6-2.54_1x06_P2.54mm_Horizontal" (at 233.045 95.885 0)
+      (effects (font (size 1.27 1.27)) hide)
+    )
+    (property "Datasheet" "~" (at 233.045 95.885 0)
+      (effects (font (size 1.27 1.27)) hide)
+    )
+    (pin "1")
+    (pin "2")
+    (pin "3")
+    (pin "4")
+    (pin "5")
+    (pin "6")
+    (instances
+      (project "Lyrav3"
+        (path "/12cc3c39-e34e-4801-bd3f-38f875d59424"
+          (reference "J9") (unit 1)
+        )
+      )
+    )
+  )
   (symbol (lib_id "Device:C_Small") (at 68.58 118.11 0) (unit 1)
     (in_bom yes) (on_board yes) (dnp no) (fields_autoplaced)
@@
         )
       )
-    )
-  )
-  (symbol (lib_id "power:+12P") (at 201.93 92.71 270) (unit 1)
-    (in_bom yes) (on_board yes) (dnp no)
-    (property "Reference" "#PWR030" (at 198.12 92.71 0)
-      (effects (font (size 1.27 1.27)) hide)
-    )
-    (property "Value" "+12P" (at 205.74 92.71 90)
-      (effects (font (size 1.27 1.27)) (justify left))
-    )
-    (property "Footprint" "" (at 201.93 92.71 0)
-      (effects (font (size 1.27 1.27)) hide)
-    )
-    (property "Datasheet" "" (at 201.93 92.71 0)
-      (effects (font (size 1.27 1.27)) hide)
-    )
-    (pin "1")
-    (instances
-      (project "Lyrav3"
-        (path "/12cc3c39-e34e-4801-bd3f-38f875d59424"
-          (reference "#PWR030") (unit 1)
-        )
-      )
-      (project "Lyra V2"
-        (path "/63622aab-8dfa-4523-a589-40aebeb23162"
-          (reference "#PWR023") (unit 1)
-        )
-      )

Commit message: move aruond
Connections:
- net P1-: now also J9.2 (Pin_2); no longer J9.5 (Pin_5)
- net P2-: now also J9.4 (Pin_4); no longer J9.3 (Pin_3)
- net P3-: now also J9.6 (Pin_6); no longer J9.1 (Pin_1)
- net PYRO PWR: now also J9.1 (Pin_1), J9.3 (Pin_3), J9.5 (Pin_5); no longer J9.2 (Pin_2), J9.4 (Pin_4), J9.6 (Pin_6)
Changed lines of the file:
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@@
     )
   )
-  (symbol (lib_id "Connector:Screw_Terminal_01x06") (at 233.045 95.885 0) (unit 1)
+  (symbol (lib_id "Connector:Screw_Terminal_01x06") (at 233.045 98.425 0) (mirror x) (unit 1)
     (in_bom no) (on_board yes) (dnp no)
-    (property "Reference" "J9" (at 233.045 85.09 0)
+    (property "Reference" "J9" (at 233.045 109.22 0)
       (effects (font (size 1.27 1.27)))
     )
-    (property "Value" "Screw_Terminal_01x06" (at 233.045 87.63 0)
+    (property "Value" "Screw_Terminal_01x06" (at 233.045 106.68 0)
       (effects (font (size 1.27 1.27)))
     )
-    (property "Footprint" "TerminalBlock_Phoenix:TerminalBlock_Phoenix_MPT-0,5-6-2.54_1x06_P2.54mm_Horizontal" (at 233.045 95.885 0)
+    (property "Footprint" "TerminalBlock_Phoenix:TerminalBlock_Phoenix_MPT-0,5-6-2.54_1x06_P2.54mm_Horizontal" (at 233.045 98.425 0)
       (effects (font (size 1.27 1.27)) hide)
     )
-    (property "Datasheet" "~" (at 233.045 95.885 0)
+    (property "Datasheet" "~" (at 233.045 98.425 0)
       (effects (font (size 1.27 1.27)) hide)
     )

Commit message: routing twioce
Connections:
- net PYRO PWR is gone; now on net +12P: J2.2 (Pin_2), J9.1 (Pin_1), J9.3 (Pin_3), J9.5 (Pin_5)
- net P1 CONT : now also U6.5 (AIN1); no longer U6.4 (AIN0)
- net P2 CONT : now also U6.4 (AIN0); no longer U6.5 (AIN1)
- net P3 CONT : now also U6.7 (AIN3); no longer U6.6 (AIN2)
- net P4 CONT : now also U6.6 (AIN2); no longer U6.7 (AIN3)
Changed lines of the file:
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@@
   (junction (at 32.385 41.275) (diameter 0) (color 0 0 0 0)
   )
+  (junction (at 222.25 93.345) (diameter 0) (color 0 0 0 0)
+  )
   (junction (at 28.575 95.885) (diameter 0) (color 0 0 0 0)
   )
@@
   (junction (at 320.294 191.008) (diameter 0) (color 0 0 0 0)
   )
+  (junction (at 222.25 98.425) (diameter 0) (color 0 0 0 0)
+  )
   (junction (at 333.629 178.943) (diameter 0) (color 0 0 0 0)
   )
@@
     (stroke (width 0) (type default))
   )
+  (wire (pts (xy 222.25 98.425) (xy 222.25 103.505))
+    (stroke (width 0) (type default))
+  )
   (wire (pts (xy 97.79 114.935) (xy 103.505 114.935))
     (stroke (width 0) (type default))
@@
     (stroke (width 0) (type default))
   )
-  (wire (pts (xy 306.705 139.065) (xy 322.58 139.065))
+  (wire (pts (xy 306.705 136.525) (xy 322.58 136.525))
     (stroke (width 0) (type default))
   )
@@
     (stroke (width 0) (type default))
   )
+  (wire (pts (xy 222.25 93.345) (xy 227.965 93.345))
+    (stroke (width 0) (type default))
+  )
   (wire (pts (xy 32.385 41.275) (xy 32.385 42.545))
     (stroke (width 0) (type default))
@@
     (stroke (width 0) (type default))
   )
+  (wire (pts (xy 222.25 93.345) (xy 222.25 98.425))
+    (stroke (width 0) (type default))
+  )
   (wire (pts (xy 361.95 209.55) (xy 371.475 209.55))
     (stroke (width 0) (type default))
@@
     (stroke (width 0) (type default))
   )
-  (wire (pts (xy 306.705 136.525) (xy 322.58 136.525))
+  (wire (pts (xy 306.705 139.065) (xy 322.58 139.065))
     (stroke (width 0) (type default))
   )
@@
     (stroke (width 0) (type default))
   )
-  (wire (pts (xy 205.74 92.71) (xy 195.58 92.71))
-    (stroke (width 0) (type default))
-  )
   (wire (pts (xy 67.31 114.3) (xy 68.58 114.3))
     (stroke (width 0) (type default))
@@
     (stroke (width 0) (type default))
   )
+  (wire (pts (xy 222.25 98.425) (xy 227.965 98.425))
+    (stroke (width 0) (type default))
+  )
   (wire (pts (xy 144.145 41.91) (xy 144.78 41.91))
     (stroke (width 0) (type default))
@@
     (stroke (width 0) (type default))
   )
-  (wire (pts (xy 217.805 93.345) (xy 227.965 93.345))
+  (wire (pts (xy 277.495 262.89) (xy 266.7 262.89))
     (stroke (width 0) (type default))
   )
-  (wire (pts (xy 277.495 262.89) (xy 266.7 262.89))
+  (wire (pts (xy 222.25 103.505) (xy 227.965 103.505))
     (stroke (width 0) (type default))
   )
@@
     (stroke (width 0) (type default))
   )
-  (wire (pts (xy 306.705 141.605) (xy 322.58 141.605))
+  (wire (pts (xy 306.705 144.145) (xy 322.58 144.145))
     (stroke (width 0) (type default))
   )
@@
     (stroke (width 0) (type default))
   )
-  (wire (pts (xy 217.805 103.505) (xy 227.965 103.505))
-    (stroke (width 0) (type default))
-  )
   (wire (pts (xy 342.9 144.145) (xy 342.9 149.225))
     (stroke (width 0) (type default))
@@
     (stroke (width 0) (type default))
   )
-  (wire (pts (xy 217.805 98.425) (xy 227.965 98.425))
-    (stroke (width 0) (type default))
-  )
   (wire (pts (xy 217.805 165.735) (xy 217.805 169.545))
     (stroke (width 0) (type default))
@@
     (stroke (width 0) (type default))
   )
-  (wire (pts (xy 306.705 144.145) (xy 322.58 144.145))
+  (wire (pts (xy 306.705 141.605) (xy 322.58 141.605))
     (stroke (width 0) (type default))
   )
@@
     (effects (font (size 1.27 1.27)) (justify right bottom))
   )
-  (label "P2 CONT " (at 306.705 139.065 0) (fields_autoplaced)
+  (label "P2 CONT " (at 306.705 136.525 0) (fields_autoplaced)
     (effects (font (size 1.27 1.27)) (justify left bottom))
   )
@@
     (effects (font (size 1.27 1.27)) (justify left bottom))
   )
-  (label "P1 CONT " (at 306.705 136.525 0) (fields_autoplaced)
+  (label "P1 CONT " (at 306.705 139.065 0) (fields_autoplaced)
     (effects (font (size 1.27 1.27)) (justify left bottom))
   )
@@
     (effects (font (size 1.27 1.27)) (justify left bottom))
   )
-  (label "P4 CONT " (at 306.705 144.145 0) (fields_autoplaced)
+  (label "P4 CONT " (at 306.705 141.605 0) (fields_autoplaced)
     (effects (font (size 1.27 1.27)) (justify left bottom))
   )
@@
     (effects (font (size 1.27 1.27)) (justify left bottom))
   )
-  (label "PYRO PWR" (at 217.805 103.505 0) (fields_autoplaced)
-    (effects (font (size 1.27 1.27)) (justify left bottom))
-  )
   (label "LEDGREEN" (at 175.26 38.1 0) (fields_autoplaced)
     (effects (font (size 1.27 1.27)) (justify left bottom))
@@
     (effects (font (size 1.27 1.27)) (justify left bottom))
   )
-  (label "PYRO PWR" (at 217.805 93.345 0) (fields_autoplaced)
-    (effects (font (size 1.27 1.27)) (justify left bottom))
-  )
   (label "I2C1 SDA" (at 186.69 243.205 180) (fields_autoplaced)
     (effects (font (size 1.27 1.27)) (justify right bottom))
@@
     (effects (font (size 1.27 1.27)) (justify right bottom))
   )
-  (label "PYRO PWR" (at 205.74 92.71 180) (fields_autoplaced)
-    (effects (font (size 1.27 1.27)) (justify right bottom))
-  )
   (label "QSPI_SCLK" (at 90.805 215.265 180) (fields_autoplaced)
     (effects (font (size 1.27 1.27)) (justify right bottom))
   )
-  (label "P3 CONT " (at 306.705 141.605 0) (fields_autoplaced)
-    (effects (font (size 1.27 1.27)) (justify left bottom))
-  )
-  (label "PYRO PWR" (at 217.805 98.425 0) (fields_autoplaced)
+  (label "P3 CONT " (at 306.705 144.145 0) (fields_autoplaced)
     (effects (font (size 1.27 1.27)) (justify left bottom))
   )
@@
     )
   )
+  (symbol (lib_id "power:+12P") (at 222.25 93.345 90) (unit 1)
+    (in_bom yes) (on_board yes) (dnp no) (fields_autoplaced)
+    (property "Reference" "#PWR030" (at 226.06 93.345 0)
+      (effects (font (size 1.27 1.27)) hide)
+    )
+    (property "Value" "+12P" (at 219.075 93.345 90)
+      (effects (font (size 1.27 1.27)) (justify left))
+    )
+    (property "Footprint" "" (at 222.25 93.345 0)
+      (effects (font (size 1.27 1.27)) hide)
+    )
+    (property "Datasheet" "" (at 222.25 93.345 0)
+      (effects (font (size 1.27 1.27)) hide)
+    )
+    (pin "1")
+    (instances
+      (project "Lyrav3"
+        (path "/12cc3c39-e34e-4801-bd3f-38f875d59424"
+          (reference "#PWR030") (unit 1)
+        )
+      )
+      (project "Board2"
+        (path "/3ee99ce6-1aa5-40d1-bb2e-7887993edb74"
+          (reference "#PWR016") (unit 1)
+        )
+      )
+      (project "Lyra V2"
+        (path "/63622aab-8dfa-4523-a589-40aebeb23162"
+          (reference "#PWR010") (unit 1)
+        )
+      )
+    )
+  )
   (symbol (lib_id "Device:R_Small") (at 352.044 181.483 0) (unit 1)
     (in_bom yes) (on_board yes) (dnp no) (fields_autoplaced)
@@
         )
       )
+    )
+  )
+  (symbol (lib_id "power:+12P") (at 195.58 92.71 270) (unit 1)
+    (in_bom yes) (on_board yes) (dnp no) (fields_autoplaced)
+    (property "Reference" "#PWR010" (at 191.77 92.71 0)
+      (effects (font (size 1.27 1.27)) hide)
+    )
+    (property "Value" "+12P" (at 199.39 92.71 90)
+      (effects (font (size 1.27 1.27)) (justify left))
+    )
+    (property "Footprint" "" (at 195.58 92.71 0)
+      (effects (font (size 1.27 1.27)) hide)
+    )
+    (property "Datasheet" "" (at 195.58 92.71 0)
+      (effects (font (size 1.27 1.27)) hide)
+    )
+    (pin "1")
+    (instances
+      (project "Lyrav3"
+        (path "/12cc3c39-e34e-4801-bd3f-38f875d59424"
+          (reference "#PWR010") (unit 1)
+        )
+      )
+      (project "Board2"
+        (path "/3ee99ce6-1aa5-40d1-bb2e-7887993edb74"
+          (reference "#PWR016") (unit 1)
+        )
+      )
+      (project "Lyra V2"
+        (path "/63622aab-8dfa-4523-a589-40aebeb23162"
+          (reference "#PWR010") (unit 1)
+        )
+      )

Commit message: rout lyrav3 fully
Connections:
- net P1 EN : now also U8.9 (GPIO7); no longer U8.6 (GPIO4)
- net P2 EN : now also U8.8 (GPIO6); no longer U8.7 (GPIO5)
- net P3 EN : now also U8.7 (GPIO5); no longer U8.8 (GPIO6)
- net P4 EN : now also U8.6 (GPIO4); no longer U8.9 (GPIO7)
