File: avionics/kicad/Lyra_flight_computer/lyra V3/Lyrav3.kicad_sch (KiCad schematic)
At the start: 83 parts, among them J2 Screw_Terminal_01x06, J3 Conn_01x02, J4 Conn_01x02, J5 Conn_01x03, J6 Conn_01x06, J7 USB_B_Micro, J8 Conn_01x04, J9 Screw_Terminal_01x06, Q1 AO3401A, Q2 AO3400A, Q3 AO3400A, Q4 AO3400A, Q5 AO3400A, U1 AZ1117-3.3, U2 BMI088, U4 ADXL375BCCZ-RL7, U5 LIS3MDL, U6 ADS1015IDGS, U7 DPS310XTSA1, U8 RP2040, U9 W25Q128JVS, X1 S3D12.288000B20F30T

Commit message: new routing and other stuff
add brownout cap
Parts:
- removed C13, C14, C3: 100n, Capacitor_SMD:C_0603_1608Metric, symbol Device:C_Small
- removed F1: 200ma, Fuse:Fuse_0805_2012Metric, symbol Device:Fuse_Small
- removed U5: LIS3MDL, Package_LGA:LGA-12_2x2mm_P0.5mm, symbol Sensor_Magnetic:LIS3MDL
- removed U7: DPS310XTSA1, easyeda2kicad:LGA-8_DPS310XTSA1, symbol easyeda2kicad:DPS310XTSA1
- added R22, R28: 1k, Resistor_SMD:R_0402_1005Metric, symbol Device:R_Small
- added U3: BMP388, easyeda2kicad:SENSORM-SMD_BMP388, symbol easyeda2kicad:BMP388
- C1, C11, C15, C16, C17, C2, C21, C22, C23, C24, C25, C26, C27: footprint Capacitor_SMD:C_0603_1608Metric -> Capacitor_SMD:C_0402_1005Metric; LCSC Part C14663 -> C1525
- C10, C18, C19, C8: footprint Capacitor_SMD:C_0603_1608Metric -> Capacitor_SMD:C_0402_1005Metric; LCSC Part C15849 -> C52923
- C12: value 1u -> 100n; footprint Capacitor_SMD:C_0603_1608Metric -> Capacitor_SMD:C_0402_1005Metric; LCSC Part C15849 -> C1525
- C4: value 10u -> 100n; footprint Capacitor_SMD:C_0603_1608Metric -> Capacitor_SMD:C_0402_1005Metric; LCSC Part C19702 -> C1525
- C5, C6, C7: footprint Capacitor_SMD:C_0603_1608Metric -> Capacitor_SMD:C_0402_1005Metric; LCSC Part C19702 -> C15525
- C9: value 1000uf -> 680uf; footprint Capacitor_THT:CP_Radial_D8.0mm_P3.80mm -> Capacitor_THT:CP_Radial_D6.3mm_P2.50mm; LCSC Part C19702 -> (none)
- R1, R12, R13, R24, R25, R5: value 6k -> 5.1k; footprint Resistor_SMD:R_0603_1608Metric -> Resistor_SMD:R_0402_1005Metric; LCSC Part C4260 -> C25905
- R10, R11, R21, R23, R4: value 20k -> 15k; footprint Resistor_SMD:R_0603_1608Metric -> Resistor_SMD:R_0402_1005Metric; LCSC Part C25804 -> C25756
- R14, R16, R17, R2, R26, R27, R3: footprint Resistor_SMD:R_0603_1608Metric -> Resistor_SMD:R_0402_1005Metric; LCSC Part C21190 -> C11702
- R15, R18: value 27R -> 22R; footprint Resistor_SMD:R_0603_1608Metric -> Resistor_SMD:R_0402_1005Metric; LCSC Part C25190 -> C25091
- R19, R20, R8, R9: value 10R -> 1R; LCSC Part C22859 -> C22936
- R6, R7: footprint Resistor_SMD:R_0603_1608Metric -> Resistor_SMD:R_0402_1005Metric; LCSC Part C4190 -> C25879
Connections:
- net +12VA is gone; now on net +12P: C5.1, C7.1, C8.1, C9.1, J6.4 (Pin_4), R4.1, U1.3 (VI)
- net +3V3: now also D4.1 (A), U3.1 (VDDIO), U3.10 (VDD), U3.6 (CSB); no longer R2.2
- net GND: now also U3.3 (VSS), U3.5 (SDO), U3.8 (VSS), U3.9 (VSS)
- net I2C1 SCL: now also U3.2 (SCK)
- net I2C1 SDA: now also U3.4 (SDI)
- net LEDBLUE: now also R28.1; no longer D4.4 (BK)
- net LEDGREEN: now also R22.1; no longer D4.3 (GK)
- net LEDRED: now also R2.1; no longer D4.2 (RK)
- new net: D4.4 (BK), R28.2
- new net: D4.2 (RK), R2.2
- new net: D4.3 (GK), R22.2
- no-connect marks 27 -> 26
Other:
- note removed: "MAGNETOMETER"
- moved on the sheet: C1, C10, C11, C2, C5, C6, C7, C8, C9, D1, D2, D4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
