File: avionics/kicad/Lyra_flight_computer/lyra V3/Lyrav3.kicad_pcb (KiCad board)
At the start: 4 copper layers, 50 x 60 mm, 111 parts, among them J1 Conn_01x04, J10 TSW-104-08-T-T-RA, J11 Screw_Terminal_01x12, J12 Screw_Terminal_01x12, J13 Conn_01x14, J2 Conn_01x02, J3 Conn_01x04, J4 Conn_01x03, J5 Conn_01x04, J6 USB_B_Micro, J7 Conn_02x03_Odd_Even, J8 Conn_01x14, J9 Conn_01x02, Q1 AO3401A, Q2 KY6802, Q3 KY6802, U1 AMS1117-5.0, U10 ADS1015IDGS, U2 AMS1117-3.3, U3 W25Q64JVXGIQ, U4 BMI088, U5 MPL3115A2, U6 ADXL375BCCZ-RL7, U7 LIS3MDL, U8 RP2040, X1 S3D12.288000B20F30T

Commit message: more lyrav3 work
Parts:
- J1: value Conn_01x04 -> Conn_01x10; footprint Connector_JST:JST_SH_SM04B-SRSS-TB_1x04-1MP_P1.00mm_Horizontal -> Connector_JST:JST_SUR_SM10B-SURS-TF_1x10-1MP_P0.80mm_Horizontal; moved to B.Cu
- J13: value Conn_01x14 -> Conn_01x10; footprint Connector_JST:JST_SUR_SM14B-SURS-TF_1x14-1MP_P0.80mm_Horizontal -> Connector_JST:JST_SUR_SM10B-SURS-TF_1x10-1MP_P0.80mm_Horizontal; moved to F.Cu
- J8: value Conn_01x14 -> Conn_01x12; footprint Connector_JST:JST_SUR_SM14B-SURS-TF_1x14-1MP_P0.80mm_Horizontal -> Connector_JST:JST_SUR_SM12B-SURS-TF_1x12-1MP_P0.80mm_Horizontal
- moved TP1 39.0 mm to (221.1, 78.7), turned to 90 degrees
- moved J13 22.9 mm to (206.3, 71.2), turned to 90 degrees
- moved Card2 21.3 mm to (196.3, 104.3), turned to 180 degrees
- moved J1 14.0 mm to (181.7, 71.4), turned to -90 degrees
- moved J8 6.72 mm to (215.1, 70.2)
- moved R25 2.21 mm to (203.2, 84.8)
- moved X1 2.18 mm to (203.3, 79.6), turned to 90 degrees
- moved C21 0.49 mm to (200.7, 77.0)
- moved C23 0.49 mm to (194.4, 75.5)
- moved C24 0.49 mm to (193.7, 73.5)
- moved C26 0.49 mm to (200.7, 78.0)
- moved C27 0.49 mm to (194.7, 81.1)
- moved C30 0.49 mm to (195.7, 77.8)
- moved J4 0.49 mm to (205.1, 77.2)
- moved R21 0.49 mm to (191.8, 77.2)
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Connections:
- J1 pad 1: /UART PWR BOT -> GND
- J1 pad 2: /UART0 TX BOT -> /SERVO4 BOT
- J1 pad 3: /UART0 RX BOT -> /SERVO3 BOT
- J1 pad 4: GND -> /SERVO2 BOT
- J10 pad 1: /SERVO1 -> /SERVO1 BOT
- J10 pad 10: /SERVO4 -> /SERVO4 BOT
- J10 pad 4: /SERVO2 -> /SERVO2 BOT
- J10 pad 7: /SERVO3 -> /SERVO3 BOT
- J11 pad 1: /GPIO 112 BOT -> unconnected-(J11-Pin_1-Pad1)
- J11 pad 2: /GPIO 102 BOT -> unconnected-(J11-Pin_2-Pad2)
- J13 pad 10: unconnected-(J13-Pin_10-Pad10) -> GND
- J13 pad 3: /I2C1 SCL -> +5VD
- J13 pad 4: /I2C1 SDA -> /I2C1 SCL
- J13 pad 5: unconnected-(J13-Pin_5-Pad5) -> /I2C1 SDA
- J13 pad 6: unconnected-(J13-Pin_6-Pad6) -> /SERVO1
- J13 pad 7: unconnected-(J13-Pin_7-Pad7) -> /SERVO2
- J13 pad 8: GND -> /SERVO3
- J13 pad 9: unconnected-(J13-Pin_9-Pad9) -> /SERVO4
- J8 pad 1: +5V -> unconnected-(J8-Pin_1-Pad1)
- J8 pad 10: /SPI0 MISO -> unconnected-(J8-Pin_10-Pad10)
- J8 pad 11: /SPI0 MOSI -> unconnected-(J8-Pin_11-Pad11)
- J8 pad 12: /SPI0 CSn -> unconnected-(J8-Pin_12-Pad12)
- J8 pad 2: /INT21 -> unconnected-(J8-Pin_2-Pad2)
- J8 pad 3: /INT12 -> unconnected-(J8-Pin_3-Pad3)
- J8 pad 4: /GPIO26 -> unconnected-(J8-Pin_4-Pad4)
- J8 pad 5: /GPIO27 -> unconnected-(J8-Pin_5-Pad5)
- J8 pad 6: /GPIO28 -> unconnected-(J8-Pin_6-Pad6)
- J8 pad 7: GND -> unconnected-(J8-Pin_7-Pad7)
- J8 pad 8: /BATT SENSE -> unconnected-(J8-Pin_8-Pad8)
- J8 pad 9: /SPI0 SCK -> unconnected-(J8-Pin_9-Pad9)
- U10 pad 1: unconnected-(U10-ADDR-Pad1) -> GND
- U10 pad 10: unconnected-(U10-SCL-Pad10) -> /I2C1 SCL BOT
- U10 pad 3: unconnected-(U10-GND-Pad3) -> GND
- U10 pad 8: unconnected-(U10-VDD-Pad8) -> +3V3
- U10 pad 9: unconnected-(U10-SDA-Pad9) -> /I2C1 SDA BOT
- U8 pad 15: unconnected-(U8-GPIO12-Pad15) -> /SERVO1
- U8 pad 16: unconnected-(U8-GPIO13-Pad16) -> /SERVO2
- U8 pad 17: unconnected-(U8-GPIO14-Pad17) -> /SERVO3
- U8 pad 18: unconnected-(U8-GPIO15-Pad18) -> /SERVO4

Commit message: aghjkl
Parts:
- added U11: PCF8574, Package_DFN_QFN:WQFN-16-1EP_3x3mm_P0.5mm_EP1.6x1.6mm, F.Cu at (143.6, 69.4)
- added U9: ADS1015IDGS, easyeda2kicad:X2QFN-10_L2.0-W1.5-P0.50-BL, F.Cu at (142.8, 73.4)
Connections:
- U10 pad 4: unconnected-(U10-AIN0-Pad4) -> /P1 CONT BOT
- U10 pad 5: unconnected-(U10-AIN1-Pad5) -> /P2 CONT BOT
- U10 pad 6: unconnected-(U10-AIN2-Pad6) -> /P3 CONT BOT
- U10 pad 7: unconnected-(U10-AIN3-Pad7) -> /P4 CONT BOT
- U8 pad 41: /BATT SENSE -> unconnected-(U8-GPIO29_ADC3-Pad41)

Commit message: Update Lyrav3.kicad_pcb
Connections:
- U10 pad 6: /P3 CONT BOT -> /BATT SENSE BOT
- U10 pad 7: /P4 CONT BOT -> unconnected-(U10-AIN3-Pad7)
- U9 pad 4: /BATT SENSE BOT -> /P3 CONT BOT
- U9 pad 5: unconnected-(U9-AIN1-Pad5) -> /P4 CONT BOT
Changed lines of the file:
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@@
   (net 143 "unconnected-(U9-AIN2-Pad6)")
   (net 144 "unconnected-(U9-AIN3-Pad7)")
-  (net 145 "unconnected-(U9-AIN1-Pad5)")
-  (net 146 "unconnected-(U11-A0-Pad1)")
-  (net 147 "unconnected-(U11-A1-Pad2)")
-  (net 148 "unconnected-(U11-A2-Pad3)")
-  (net 149 "unconnected-(U11-P0-Pad4)")
-  (net 150 "unconnected-(U11-P1-Pad5)")
-  (net 151 "unconnected-(U11-P2-Pad6)")
-  (net 152 "unconnected-(U11-P3-Pad7)")
-  (net 153 "unconnected-(U11-VSS-Pad8)")
-  (net 154 "unconnected-(U11-P4-Pad9)")
-  (net 155 "unconnected-(U11-P5-Pad10)")
-  (net 156 "unconnected-(U11-P6-Pad11)")
-  (net 157 "unconnected-(U11-P7-Pad12)")
-  (net 158 "unconnected-(U11-~{INT}-Pad13)")
-  (net 159 "unconnected-(U11-SCL-Pad14)")
-  (net 160 "unconnected-(U11-SDA-Pad15)")
-  (net 161 "unconnected-(U11-VDD-Pad16)")
+  (net 145 "unconnected-(U11-A0-Pad1)")
+  (net 146 "unconnected-(U11-A1-Pad2)")
+  (net 147 "unconnected-(U11-A2-Pad3)")
+  (net 148 "unconnected-(U11-P0-Pad4)")
+  (net 149 "unconnected-(U11-P1-Pad5)")
+  (net 150 "unconnected-(U11-P2-Pad6)")
+  (net 151 "unconnected-(U11-P3-Pad7)")
+  (net 152 "unconnected-(U11-VSS-Pad8)")
+  (net 153 "unconnected-(U11-P4-Pad9)")
+  (net 154 "unconnected-(U11-P5-Pad10)")
+  (net 155 "unconnected-(U11-P6-Pad11)")
+  (net 156 "unconnected-(U11-P7-Pad12)")
+  (net 157 "unconnected-(U11-~{INT}-Pad13)")
+  (net 158 "unconnected-(U11-SCL-Pad14)")
+  (net 159 "unconnected-(U11-SDA-Pad15)")
+  (net 160 "unconnected-(U11-VDD-Pad16)")
+  (net 161 "unconnected-(U10-AIN3-Pad7)")
   (footprint "Diode_SMD:D_SOD-123" (layer "F.Cu")
     (at 174.498 92.1004 90)
@@
     (pad "" smd roundrect (at 0.4 0.4) (size 0.64 0.64) (layers "F.Paste") (roundrect_rratio 0.25))
     (pad "1" smd roundrect (at -1.4375 -0.75) (size 0.875 0.25) (layers "F.Cu" "F.Paste" "F.Mask") (roundrect_rratio 0.25)
-      (net 146 "unconnected-(U11-A0-Pad1)") (pinfunction "A0") (pintype "input"))
+      (net 145 "unconnected-(U11-A0-Pad1)") (pinfunction "A0") (pintype "input"))
     (pad "2" smd roundrect (at -1.4375 -0.25) (size 0.875 0.25) (layers "F.Cu" "F.Paste" "F.Mask") (roundrect_rratio 0.25)
-      (net 147 "unconnected-(U11-A1-Pad2)") (pinfunction "A1") (pintype "input"))
+      (net 146 "unconnected-(U11-A1-Pad2)") (pinfunction "A1") (pintype "input"))
     (pad "3" smd roundrect (at -1.4375 0.25) (size 0.875 0.25) (layers "F.Cu" "F.Paste" "F.Mask") (roundrect_rratio 0.25)
-      (net 148 "unconnected-(U11-A2-Pad3)") (pinfunction "A2") (pintype "input"))
+      (net 147 "unconnected-(U11-A2-Pad3)") (pinfunction "A2") (pintype "input"))
     (pad "4" smd roundrect (at -1.4375 0.75) (size 0.875 0.25) (layers "F.Cu" "F.Paste" "F.Mask") (roundrect_rratio 0.25)
-      (net 149 "unconnected-(U11-P0-Pad4)") (pinfunction "P0") (pintype "bidirectional"))
+      (net 148 "unconnected-(U11-P0-Pad4)") (pinfunction "P0") (pintype "bidirectional"))
     (pad "5" smd roundrect (at -0.75 1.4375) (size 0.25 0.875) (layers "F.Cu" "F.Paste" "F.Mask") (roundrect_rratio 0.25)
-      (net 150 "unconnected-(U11-P1-Pad5)") (pinfunction "P1") (pintype "bidirectional"))
+      (net 149 "unconnected-(U11-P1-Pad5)") (pinfunction "P1") (pintype "bidirectional"))
     (pad "6" smd roundrect (at -0.25 1.4375) (size 0.25 0.875) (layers "F.Cu" "F.Paste" "F.Mask") (roundrect_rratio 0.25)
-      (net 151 "unconnected-(U11-P2-Pad6)") (pinfunction "P2") (pintype "bidirectional"))
+      (net 150 "unconnected-(U11-P2-Pad6)") (pinfunction "P2") (pintype "bidirectional"))
     (pad "7" smd roundrect (at 0.25 1.4375) (size 0.25 0.875) (layers "F.Cu" "F.Paste" "F.Mask") (roundrect_rratio 0.25)
-      (net 152 "unconnected-(U11-P3-Pad7)") (pinfunction "P3") (pintype "bidirectional"))
+      (net 151 "unconnected-(U11-P3-Pad7)") (pinfunction "P3") (pintype "bidirectional"))
     (pad "8" smd roundrect (at 0.75 1.4375) (size 0.25 0.875) (layers "F.Cu" "F.Paste" "F.Mask") (roundrect_rratio 0.25)
-      (net 153 "unconnected-(U11-VSS-Pad8)") (pinfunction "VSS") (pintype "power_in"))
+      (net 152 "unconnected-(U11-VSS-Pad8)") (pinfunction "VSS") (pintype "power_in"))
     (pad "9" smd roundrect (at 1.4375 0.75) (size 0.875 0.25) (layers "F.Cu" "F.Paste" "F.Mask") (roundrect_rratio 0.25)
-      (net 154 "unconnected-(U11-P4-Pad9)") (pinfunction "P4") (pintype "bidirectional"))
+      (net 153 "unconnected-(U11-P4-Pad9)") (pinfunction "P4") (pintype "bidirectional"))
     (pad "10" smd roundrect (at 1.4375 0.25) (size 0.875 0.25) (layers "F.Cu" "F.Paste" "F.Mask") (roundrect_rratio 0.25)
-      (net 155 "unconnected-(U11-P5-Pad10)") (pinfunction "P5") (pintype "bidirectional"))
+      (net 154 "unconnected-(U11-P5-Pad10)") (pinfunction "P5") (pintype "bidirectional"))
     (pad "11" smd roundrect (at 1.4375 -0.25) (size 0.875 0.25) (layers "F.Cu" "F.Paste" "F.Mask") (roundrect_rratio 0.25)
-      (net 156 "unconnected-(U11-P6-Pad11)") (pinfunction "P6") (pintype "bidirectional"))
+      (net 155 "unconnected-(U11-P6-Pad11)") (pinfunction "P6") (pintype "bidirectional"))
     (pad "12" smd roundrect (at 1.4375 -0.75) (size 0.875 0.25) (layers "F.Cu" "F.Paste" "F.Mask") (roundrect_rratio 0.25)
-      (net 157 "unconnected-(U11-P7-Pad12)") (pinfunction "P7") (pintype "bidirectional"))
+      (net 156 "unconnected-(U11-P7-Pad12)") (pinfunction "P7") (pintype "bidirectional"))
     (pad "13" smd roundrect (at 0.75 -1.4375) (size 0.25 0.875) (layers "F.Cu" "F.Paste" "F.Mask") (roundrect_rratio 0.25)
-      (net 158 "unconnected-(U11-~{INT}-Pad13)") (pinfunction "~{INT}") (pintype "open_collector"))
+      (net 157 "unconnected-(U11-~{INT}-Pad13)") (pinfunction "~{INT}") (pintype "open_collector"))
     (pad "14" smd roundrect (at 0.25 -1.4375) (size 0.25 0.875) (layers "F.Cu" "F.Paste" "F.Mask") (roundrect_rratio 0.25)
-      (net 159 "unconnected-(U11-SCL-Pad14)") (pinfunction "SCL") (pintype "input"))
+      (net 158 "unconnected-(U11-SCL-Pad14)") (pinfunction "SCL") (pintype "input"))
     (pad "15" smd roundrect (at -0.25 -1.4375) (size 0.25 0.875) (layers "F.Cu" "F.Paste" "F.Mask") (roundrect_rratio 0.25)
-      (net 160 "unconnected-(U11-SDA-Pad15)") (pinfunction "SDA") (pintype "bidirectional"))
+      (net 159 "unconnected-(U11-SDA-Pad15)") (pinfunction "SDA") (pintype "bidirectional"))
     (pad "16" smd roundrect (at -0.75 -1.4375) (size 0.25 0.875) (layers "F.Cu" "F.Paste" "F.Mask") (roundrect_rratio 0.25)
-      (net 161 "unconnected-(U11-VDD-Pad16)") (pinfunction "VDD") (pintype "power_in"))
+      (net 160 "unconnected-(U11-VDD-Pad16)") (pinfunction "VDD") (pintype "power_in"))
     (pad "17" smd rect (at 0 0) (size 1.6 1.6) (layers "F.Cu" "F.Mask"))
     (model "${KICAD6_3DMODEL_DIR}/Package_DFN_QFN.3dshapes/WQFN-16-1EP_3x3mm_P0.5mm_EP1.6x1.6mm.wrl"
@@
       (net 2 "GND") (pinfunction "GND") (pintype "power_in"))
     (pad "4" smd rect (at 0.75 0.63) (size 0.3 0.58) (layers "F.Cu" "F.Paste" "F.Mask")
-      (net 74 "/BATT SENSE BOT") (pinfunction "AIN0") (pintype "input"))
+      (net 68 "/P3 CONT BOT") (pinfunction "AIN0") (pintype "input"))
     (pad "5" smd rect (at 0.86 0 90) (size 0.35 0.63) (layers "F.Cu" "F.Paste" "F.Mask")
-      (net 145 "unconnected-(U9-AIN1-Pad5)") (pinfunction "AIN1") (pintype "input+no_connect"))
+      (net 66 "/P4 CONT BOT") (pinfunction "AIN1") (pintype "input"))
     (pad "6" smd rect (at 0.75 -0.63) (size 0.3 0.58) (layers "F.Cu" "F.Paste" "F.Mask")
       (net 143 "unconnected-(U9-AIN2-Pad6)") (pinfunction "AIN2") (pintype "input+no_connect"))
@@
       (net 70 "/P2 CONT BOT") (pinfunction "AIN1") (pintype "input"))
     (pad "6" smd rect (at 0.75 -0.63) (size 0.3 0.58) (layers "F.Cu" "F.Paste" "F.Mask")
-      (net 68 "/P3 CONT BOT") (pinfunction "AIN2") (pintype "input"))
+      (net 74 "/BATT SENSE BOT") (pinfunction "AIN2") (pintype "input"))
     (pad "7" smd rect (at 0.25 -0.63) (size 0.25 0.58) (layers "F.Cu" "F.Paste" "F.Mask")
-      (net 66 "/P4 CONT BOT") (pinfunction "AIN3") (pintype "input"))
+      (net 161 "unconnected-(U10-AIN3-Pad7)") (pinfunction "AIN3") (pintype "input+no_connect"))
     (pad "8" smd rect (at -0.25 -0.63) (size 0.25 0.58) (layers "F.Cu" "F.Paste" "F.Mask")
       (net 3 "+3V3") (pinfunction "VDD") (pintype "power_in"))

Commit message: more lyrav3 work
Parts:
- removed D1: D_Small, Diode_SMD:D_SOD-123
- removed J7: Conn_02x03_Odd_Even, Connector_JST:JST_SH_SM06B-SRSS-TB_1x06-1MP_P1.00mm_Horizontal
- removed JP4: SolderJumper_3_Open, Jumper:SolderJumper-3_P1.3mm_Open_Pad1.0x1.5mm
- removed R28: 1k, Resistor_SMD:R_0402_1005Metric
- removed TP1: TestPoint, TestPoint:TestPoint_Pad_1.0x1.0mm
- added C1: 100n, Capacitor_SMD:C_0402_1005Metric, B.Cu at (172.2, 93.3)
- added C6: 100n, Capacitor_SMD:C_0402_1005Metric, B.Cu at (170.7, 108.5)
- C16, C17, C19, D2, JP2, R27: moved to F.Cu
- D4: value LED -> D; footprint LED_SMD:LED_0805_2012Metric -> Diode_SMD:D_0402_1005Metric
- F1, Q1, R10, R16, R18, R20, R6, R8: moved to B.Cu
- J2: footprint Jumper:SolderJumper-2_P1.3mm_Open_Pad1.0x1.5mm -> Jumper:SolderJumper-2_P1.3mm_Open_RoundedPad1.0x1.5mm
- J3: value Conn_01x04 -> Conn_01x07; footprint Connector_JST:JST_SH_SM04B-SRSS-TB_1x04-1MP_P1.00mm_Horizontal -> Connector_JST:JST_SH_SM07B-SRSS-TB_1x07-1MP_P1.00mm_Horizontal
- J5: value Conn_01x04 -> Conn_01x05; footprint Connector_JST:JST_SH_SM04B-SRSS-TB_1x04-1MP_P1.00mm_Horizontal -> Connector_JST:JST_SH_SM05B-SRSS-TB_1x05-1MP_P1.00mm_Horizontal; moved to F.Cu
- J8: value Conn_01x12 -> Conn_01x05; footprint Connector_JST:JST_SUR_SM12B-SURS-TF_1x12-1MP_P0.80mm_Horizontal -> Connector_JST:JST_SH_SM05B-SRSS-TB_1x05-1MP_P1.00mm_Horizontal; moved to B.Cu
- moved U11 41.0 mm to (170.9, 100.1), turned to -90 degrees
- moved U10 40.4 mm to (170.7, 108.5), turned to -90 degrees
- moved U9 33.3 mm to (171.2, 90.7), turned to -90 degrees
- moved J5 24.3 mm to (171.1, 62.2), turned to 180 degrees
- moved C34 22.9 mm to (194.9, 104.2), turned to 0 degrees
- moved J8 20.6 mm to (196.1, 62.3), turned to 0 degrees
- moved D4 16.3 mm to (191.0, 71.9), turned to -90 degrees
- moved D2 4.66 mm to (160.8, 77.5), turned to 180 degrees
- moved C31 4.48 mm to (192.9, 85.0)
- moved C32 4.48 mm to (193.0, 83.0)
- moved U3 4.48 mm to (190.4, 83.7)
- moved R3 3.43 mm to (175.2, 103.8), turned to 90 degrees
- moved J2 3.31 mm to (202.9, 83.7)
- moved R25 3.22 mm to (203.5, 81.6)
- moved R10 2.67 mm to (169.0, 98.2)
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Connections:
- Card2 pad 2: /SD CS BOT -> /SD CS
- Card2 pad 3: /SPI1 MOSI BOT -> /SPI0 MOSI
- Card2 pad 5: /SPI1 SCLK BOT -> /SPI0 SCK
- Card2 pad 7: /SPI1 MISO BOT -> /SPI0 MISO
- D4 pad 1: GND -> +5V
- J11 pad 1: unconnected-(J11-Pin_1-Pad1) -> /ADC GPIO
- J11 pad 2: unconnected-(J11-Pin_2-Pad2) -> /ADC2 GPIO
- J11 pad 3: unconnected-(J11-Pin_3-Pad3) -> /GPIOUT1
- J11 pad 4: unconnected-(J11-Pin_4-Pad4) -> /GPIOUT2
- J11 pad 6: /GPIO28 BOT -> +5V
- J12 pad 2: +5V -> GND
- J13 pad 3: +5VD -> +5V
- J3 pad 1: /I2C PWR -> /SPI0 GPIO
- J3 pad 2: /I2C1 SCL -> /SPI0 MISO
- J3 pad 3: /I2C1 SDA -> /SPI0 MOSI
- J3 pad 4: GND -> /SPI0 CSn
- J5 pad 1: /UART PWR -> /I2C GPIO
- J5 pad 2: /UART0 RX -> /I2C PWR
- J5 pad 3: /UART0 TX -> /I2C1 SCL BOT
- J5 pad 4: GND -> /I2C1 SDA BOT
- J6 pad 1: unconnected-(J6-VBUS-Pad1) -> Net-(D4-A)
- J8 pad 1: unconnected-(J8-Pin_1-Pad1) -> /UART GPIO
- J8 pad 2: unconnected-(J8-Pin_2-Pad2) -> /UART PWR
- J8 pad 3: unconnected-(J8-Pin_3-Pad3) -> /UART0 RX
- J8 pad 4: unconnected-(J8-Pin_4-Pad4) -> /UART0 TX
- J8 pad 5: unconnected-(J8-Pin_5-Pad5) -> GND
- JP1 pad 1: +5VD -> +5V
- JP1 pad 2: /UART PWR BOT -> /I2C PWR
- JP2 pad 2: /I2C PWR -> /SPI PWR
- U11 pad 1: unconnected-(U11-A0-Pad1) -> GND
- U11 pad 11: unconnected-(U11-P6-Pad11) -> /GPIOUT1
- U11 pad 12: unconnected-(U11-P7-Pad12) -> /GPIOUT2
- U11 pad 14: unconnected-(U11-SCL-Pad14) -> /I2C1 SCL BOT
- U11 pad 15: unconnected-(U11-SDA-Pad15) -> /I2C1 SDA BOT
- U11 pad 16: unconnected-(U11-VDD-Pad16) -> +3V3
- U11 pad 2: unconnected-(U11-A1-Pad2) -> GND
- U11 pad 3: unconnected-(U11-A2-Pad3) -> GND
- U11 pad 4: unconnected-(U11-P0-Pad4) -> /P1 EN BOT
- U11 pad 5: unconnected-(U11-P1-Pad5) -> /P2 EN BOT
- U11 pad 6: unconnected-(U11-P2-Pad6) -> /P3 EN BOT
- U11 pad 7: unconnected-(U11-P3-Pad7) -> /P4 EN BOT
- U11 pad 8: unconnected-(U11-VSS-Pad8) -> GND
- U11 pad 9: unconnected-(U11-P4-Pad9) -> /I2C GPIO
- U8 pad 2: unconnected-(U8-GPIO0-Pad2) -> /SPI0 GPIO
- U8 pad 36: unconnected-(U8-GPIO24-Pad36) -> /UART GPIO
- U8 pad 4: unconnected-(U8-GPIO2-Pad4) -> /SD CS
- U9 pad 6: unconnected-(U9-AIN2-Pad6) -> /ADC GPIO
- U9 pad 7: unconnected-(U9-AIN3-Pad7) -> /ADC2 GPIO
Other:
- board text removed: "IO101"
- board text removed: "IO112"
- board text removed: "IO271"
- board text removed: "IO281"
- board text removed: "IO282"

Commit message: simplified lyrav3
Parts:
- removed C30, C32: 100n, Capacitor_SMD:C_0402_1005Metric
- removed C31: 2u2, Capacitor_SMD:C_0402_1005Metric
- removed C33, C34: 1u, Capacitor_SMD:C_0402_1005Metric
- removed Card2: TF-002-H18, easyeda2kicad:SIM-SMD_TF-002-H18
- removed D4: D, Diode_SMD:D_0402_1005Metric
- removed F2: 200ma, Fuse:Fuse_0805_2012Metric
- removed FB1: FerriteBead_Small, Diode_SMD:D_0603_1608Metric
- removed H10, H9: Access Hole, customfootprints:1x10 2.54mm pitch acess hole
- removed H5, H6, H7, H8: MountingHole_Pad, MountingHole:MountingHole_3.2mm_M3_DIN965_Pad
- removed J10: TSW-104-08-T-T-RA, SamacSys_Parts:HDRRA12W64P254_3X4_1016X254X810P
- removed J11, J12: Screw_Terminal_01x12, TerminalBlock_Phoenix:TerminalBlock_Phoenix_MPT-0,5-12-2.54_1x12_P2.54mm_Horizontal
- removed J13: Conn_01x10, Connector_JST:JST_SUR_SM10B-SURS-TF_1x10-1MP_P0.80mm_Horizontal
- removed J9: Conn_01x02, Jumper:SolderJumper-2_P1.3mm_Open_RoundedPad1.0x1.5mm
- removed JP1, JP2, JP3, JP5: SolderJumper_3_Open, Jumper:SolderJumper-3_P1.3mm_Open_Pad1.0x1.5mm
- removed U1: AMS1117-5.0, Package_TO_SOT_SMD:SOT-89-3
- removed U10: ADS1015IDGS, easyeda2kicad:X2QFN-10_L2.0-W1.5-P0.50-BL
- removed U11: PCF8574, Package_DFN_QFN:WQFN-16-1EP_3x3mm_P0.5mm_EP1.6x1.6mm
- added C18: 1u, Capacitor_SMD:C_0402_1005Metric, F.Cu at (126.1, 88.6)
- added D1: LED, LED_SMD:LED_0805_2012Metric, F.Cu at (139.6, 60.8)
- added J7: USB_B_Micro, easyeda2kicad:MICRO-USB-SMD_U254-051T-4BHJ25-F2S, F.Cu at (203.8, 83.4)
- C1, C13, C15, C20, C21, C24, C25, C26, C28, C29, C9, Q1, R1: moved to F.Cu
- C10: value 10u -> 1u; footprint Capacitor_SMD:C_0603_1608Metric -> Capacitor_SMD:C_0402_1005Metric; moved to F.Cu
- C11: value 10u -> 100n; footprint Capacitor_SMD:C_0603_1608Metric -> Capacitor_SMD:C_0402_1005Metric
- C14, C22, C23: value 1u -> 100n; moved to F.Cu
- C16: value 1u -> 100n
- C19: value 100n -> 1u
- C2, C3: value 22u -> 100n; footprint Capacitor_SMD:C_0603_1608Metric -> Capacitor_SMD:C_0402_1005Metric; moved to F.Cu
- C27: value 100n -> 2u2; moved to F.Cu
- C4: value 22u -> 10u; moved to F.Cu
- C5: value 22u -> 1u; footprint Capacitor_SMD:C_0603_1608Metric -> Capacitor_SMD:C_0402_1005Metric; moved to F.Cu
- C6, C8: value 100n -> 1u; moved to F.Cu
- C7: value 100n -> 10u; footprint Capacitor_SMD:C_0402_1005Metric -> Capacitor_SMD:C_0603_1608Metric; moved to F.Cu
- D3: value LED -> D; footprint LED_SMD:LED_0805_2012Metric -> Diode_SMD:D_0402_1005Metric
- F1: value 2a -> 200ma; footprint Fuse:Fuse_1812_4532Metric -> Fuse:Fuse_0805_2012Metric; moved to F.Cu
- J1: value Conn_01x10 -> Screw_Terminal_01x08; footprint Connector_JST:JST_SUR_SM10B-SURS-TF_1x10-1MP_P0.80mm_Horizontal -> TerminalBlock_Phoenix:TerminalBlock_Phoenix_MPT-0,5-8-2.54_1x08_P2.54mm_Horizontal; moved to F.Cu
- J2: value Conn_01x02 -> Screw_Terminal_01x06; footprint Jumper:SolderJumper-2_P1.3mm_Open_RoundedPad1.0x1.5mm -> TerminalBlock_Phoenix:TerminalBlock_Phoenix_MPT-0,5-6-2.54_1x06_P2.54mm_Horizontal; moved to F.Cu
- J3: value Conn_01x07 -> Conn_01x02; footprint Connector_JST:JST_SH_SM07B-SRSS-TB_1x07-1MP_P1.00mm_Horizontal -> Jumper:SolderJumper-2_P1.3mm_Open_RoundedPad1.0x1.5mm; moved to F.Cu
- J4: value Conn_01x03 -> Conn_01x02; footprint Connector_JST:JST_SH_SM03B-SRSS-TB_1x03-1MP_P1.00mm_Horizontal -> Jumper:SolderJumper-2_P1.3mm_Open_RoundedPad1.0x1.5mm; moved to F.Cu
- J5: value Conn_01x05 -> Conn_01x03; footprint Connector_JST:JST_SH_SM05B-SRSS-TB_1x05-1MP_P1.00mm_Horizontal -> Connector_JST:JST_SH_SM03B-SRSS-TB_1x03-1MP_P1.00mm_Horizontal
- J6: value USB_B_Micro -> Conn_01x06; footprint easyeda2kicad:MICRO-USB-SMD_U254-051T-4BHJ25-F2S -> Connector_PinHeader_2.54mm:PinHeader_1x06_P2.54mm_Vertical
- J8: value Conn_01x05 -> Conn_01x04; footprint Connector_JST:JST_SH_SM05B-SRSS-TB_1x05-1MP_P1.00mm_Horizontal -> Connector_PinHeader_2.54mm:PinHeader_1x04_P2.54mm_Vertical; moved to F.Cu
- R10: value 6k -> 20k; moved to F.Cu
- R11, R23: value 470R -> 20k
- R12, R24: value 470R -> 6k
- R13: value 2k2 -> 6k
- R14: value 2k2 -> 10k
- R15: value 10R -> 27R; moved to F.Cu
- R16: value 10R -> 470R; moved to F.Cu
- R17: value 20k -> 470R
- R18: value 20k -> 27R; moved to F.Cu
- R19: value 6k -> 10R
- R2: value 20k -> 1k
- R20, R9: value 6k -> 10R; moved to F.Cu
- R21: value 27R -> 20k
- R22: value 27R -> 1k
- R25: value 10k -> 6k; moved to F.Cu
- R26, R27: value 1k -> 470R
- R3: value 6k -> 1k
- R4: value 1k -> 20k; moved to F.Cu
- R5: value 10R -> 6k; moved to F.Cu
- R6: value 10R -> 2k2; moved to F.Cu
- R7: value 20k -> 2k2; moved to F.Cu
- R8: value 20k -> 10R; moved to F.Cu
- U2: value AMS1117-3.3 -> BMI088; footprint Package_TO_SOT_SMD:SOT-89-3 -> easyeda2kicad:LGA-16_L4.5-W3.0-P0.50-BL; moved to F.Cu
- U3: value W25Q64JVXGIQ -> MPL3115A2; footprint easyeda2kicad:XSON-8_L4.0-W4.0-P0.80-TL-EP -> Package_LGA:NXP_LGA-8_3x5mm_P1.25mm_H1.1mm; moved to F.Cu
- U4: value BMI088 -> ADXL375BCCZ-RL7; footprint SnapEDA Library:PQFN50P450X300X100-16N -> easyeda2kicad:LGA-14_L5.0-W3.0-P0.80-BL
- U5: value MPL3115A2 -> LIS3MDL; footprint Package_LGA:NXP_LGA-8_3x5mm_P1.25mm_H1.1mm -> Package_LGA:LGA-12_2x2mm_P0.5mm
- U6: value ADXL375BCCZ-RL7 -> ADS1015IDGS; footprint easyeda2kicad:LGA-14_L5.0-W3.0-P0.80-BL -> easyeda2kicad:X2QFN-10_L2.0-W1.5-P0.50-BL
- U7: value LIS3MDL -> W25Q64JVXGIQ; footprint Package_LGA:LGA-12_2x2mm_P0.5mm -> easyeda2kicad:XSON-8_L4.0-W4.0-P0.80-TL-EP; moved to B.Cu
- U9: value ADS1015IDGS -> LDK130-33_SOT23_SOT353; footprint easyeda2kicad:X2QFN-10_L2.0-W1.5-P0.50-BL -> easyeda2kicad:SOT-23-5_L3.0-W1.6-P0.95-LS2.8-BL
- moved R4 86.0 mm to (111.6, 82.8)
- moved R25 83.2 mm to (120.4, 82.8), turned to 0 degrees
- moved R14 83.1 mm to (114.5, 88.8)
- moved R13 82.9 mm to (114.5, 86.8)
- moved J3 81.9 mm to (135.2, 61.1), turned to 0 degrees
- moved C8 80.0 mm to (123.3, 82.7)
- moved C17 77.2 mm to (126.1, 86.7), turned to 0 degrees
- moved R27 76.9 mm to (120.4, 86.8), turned to 0 degrees
- moved C16 76.4 mm to (126.1, 84.7), turned to 0 degrees
- moved R21 75.2 mm to (117.5, 88.8)
- moved C19 74.7 mm to (129.0, 76.8), turned to 0 degrees
- moved R26 72.5 mm to (120.4, 84.8), turned to 0 degrees
- moved U6 72.5 mm to (123.6, 100.3), turned to 0 degrees
- moved C21 71.8 mm to (129.0, 80.8)
- moved R22 71.4 mm to (120.4, 76.8), turned to 0 degrees
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Connections:
- C11 pad 1: +12VA -> +3V3
- C12 pad 1: +12VA -> +3V3
- C13 pad 1: Net-(U5-CAP) -> +3V3
- C14 pad 1: +3V3 -> Net-(U5-C1)
- C16 pad 1: +3V3 -> +1V1
- C17 pad 1: +3V3 -> +1V1
- C19 pad 1: Net-(U7-C1) -> +3V3
- C2 pad 1: +12VA -> +3V3
- C20 pad 1: +1V1 -> +3V3
- C21 pad 1: +1V1 -> +3V3
- C22 pad 1: +1V1 -> +3V3
- C29 pad 1: +3V3 -> Net-(U9-BP)
- C29 pad 2: GND -> Net-(U9-GND)
- C3 pad 1: +5VD -> +3V3
- C4 pad 1: +12VA -> +3V3
- C5 pad 1: +3V3 -> +12VA
- C5 pad 2: GND -> Net-(U9-GND)
- C6 pad 2: GND -> Net-(U9-GND)
- C7 pad 1: +3V3 -> +12VA
- C8 pad 1: +3V3 -> +12VA
- C9 pad 1: +3V3 -> Net-(U3-CAP)
- D3 pad 1: GND -> +12V
- F1 pad 1: Net-(Q1-S) -> +12P
- F1 pad 2: +12P -> +12VA
- J1 pad 1: GND -> /P4-
- J1 pad 2: /SERVO4 BOT -> /PYRO PWR
- J1 pad 3: /SERVO3 BOT -> /P3-
- J1 pad 4: /SERVO2 BOT -> /PYRO PWR
- J1 pad 5: /SERVO1 BOT -> /P2-
- J1 pad 6: /I2C1 SDA BOT -> /PYRO PWR
- J1 pad 7: /I2C1 SCL BOT -> /P1-
- J1 pad 8: +5VD -> /PYRO PWR
- J2 pad 1: /RUN -> /PYRO PWR
- J2 pad 2: GND -> +12P
- J3 pad 1: /SPI0 GPIO -> /RUN
- J3 pad 2: /SPI0 MISO -> GND
- J4 pad 1: /SWCLK -> GND
- J4 pad 2: GND -> /BOOTSEL
- J5 pad 1: /I2C GPIO -> /SWCLK
- J5 pad 2: /I2C PWR -> GND
- J5 pad 3: /I2C1 SCL BOT -> /SWD
- J6 pad 1: Net-(D4-A) -> /BRKOUT5
- J6 pad 2: /USB_D- -> /BRKOUT6
- J6 pad 3: /USB_D+ -> /BRKOUT7
- J6 pad 4: unconnected-(J6-ID-Pad4) -> +12VA
- J6 pad 5: GND -> +3V3
- J6 pad 6: unconnected-(J6-Shield-Pad6) -> GND
- J8 pad 1: /UART GPIO -> /BRKOUT4
- J8 pad 2: /UART PWR -> /BRKOUT3
- J8 pad 3: /UART0 RX -> /BRKOUT2
- J8 pad 4: /UART0 TX -> /BRKOUT1
- Q1 pad 2: Net-(Q1-S) -> +12P
- Q2 pad 1: /P1 EN BOT -> /P1 EN 
- Q2 pad 3: /P2 EN BOT -> /P2 EN 
- Q3 pad 1: /P3 EN BOT -> /P3 EN 
- Q3 pad 3: /P4 EN BOT -> /P4 EN 
- R1 pad 1: Net-(D2-A) -> Net-(D1-A)
- R10 pad 1: /P3 CONT BOT -> Net-(Q2A-D)
- R10 pad 2: GND -> /P1 CONT 
- R11 pad 1: GND -> Net-(Q3A-D)
- R11 pad 2: /P1 EN BOT -> /P3 CONT 
- R12 pad 1: GND -> /P1 CONT 
- R12 pad 2: /P3 EN BOT -> GND
- R13 pad 1: +3V3 -> /P3 CONT 
- R13 pad 2: /I2C1 SCL -> GND
- R14 pad 2: /I2C1 SDA -> /RUN
- R15 pad 1: /P2- -> /USB_D+
- R15 pad 2: Net-(Q2B-D) -> /RP USB_D+
- R16 pad 1: /P4- -> GND
- R16 pad 2: Net-(Q3B-D) -> /P1 EN 
- R17 pad 1: Net-(Q2B-D) -> GND
- R17 pad 2: /P2 CONT BOT -> /P3 EN 
- R18 pad 1: Net-(Q3B-D) -> /RP USB_D-
- R18 pad 2: /P4 CONT BOT -> /USB_D-
- R19 pad 1: /P2 CONT BOT -> /P2-
- R19 pad 2: GND -> Net-(Q2B-D)
- R2 pad 1: +12V -> Net-(LED1-+-Pad4)
- R2 pad 2: /BATT SENSE BOT -> +3V3
- R20 pad 1: /P4 CONT BOT -> /P4-
- R20 pad 2: GND -> Net-(Q3B-D)
- R21 pad 1: /USB_D+ -> Net-(Q2B-D)
- R21 pad 2: /RP USB_D+ -> /P2 CONT 
- R22 pad 1: /RP USB_D- -> /QSPI_SS
- R22 pad 2: /USB_D- -> /BOOTSEL
- R23 pad 1: GND -> Net-(Q3B-D)
- R23 pad 2: /P2 EN BOT -> /P4 CONT 
- R24 pad 1: GND -> /P2 CONT 
- R24 pad 2: /P4 EN BOT -> GND
- R25 pad 1: +3V3 -> /P4 CONT 
- R25 pad 2: /RUN -> GND
- R26 pad 1: /QSPI_SS -> GND
- R26 pad 2: /BOOTSEL -> /P2 EN 
- R27 pad 1: Net-(D3-A) -> GND
- R27 pad 2: +3V3 -> /P4 EN 
- R3 pad 1: /BATT SENSE BOT -> Net-(D2-A)
- R3 pad 2: GND -> +3V3
- R4 pad 1: Net-(LED1-+-Pad4) -> +12V
- R4 pad 2: +3V3 -> /BATT SENSE 
- R5 pad 1: /P1- -> /BATT SENSE 
- R5 pad 2: Net-(Q2A-D) -> GND
- R6 pad 1: /P3- -> +3V3
- R6 pad 2: Net-(Q3A-D) -> /I2C1 SCL
- R7 pad 1: Net-(Q2A-D) -> +3V3
- R7 pad 2: /P1 CONT BOT -> /I2C1 SDA
- R8 pad 1: Net-(Q3A-D) -> /P1-
- R8 pad 2: /P3 CONT BOT -> Net-(Q2A-D)
- R9 pad 1: /P1 CONT BOT -> /P3-
- R9 pad 2: GND -> Net-(Q3A-D)
- U2 pad 1: GND -> unconnected-(U2-INT2-Pad1)
- U2 pad 2: +3V3 -> unconnected-(U2-NC-Pad2)
- U2 pad 3: +12VA -> +3V3
- U3 pad 1: /QSPI_SS -> +3V3
- U3 pad 2: /QSPI_SD1 -> Net-(U3-CAP)
- U3 pad 3: /QSPI_SD2 -> GND
- U3 pad 4: GND -> +3V3
- U3 pad 5: /QSPI_SDO -> unconnected-(U3-INT2-Pad5)
- U3 pad 6: /QSPI_SCLK -> unconnected-(U3-INT1-Pad6)
- U3 pad 7: /QSPI_SD3 -> /I2C0 SDA
- U3 pad 8: +3V3 -> /I2C0 SCL
- U4 pad 1: unconnected-(U4-INT2-Pad1) -> +3V3
- U4 pad 10: GND -> unconnected-(U4-NC-Pad10)
- U4 pad 11: +3V3 -> GND
- U4 pad 12: unconnected-(U4-INT3-Pad12) -> GND
- U4 pad 13: unconnected-(U4-INT4-Pad13) -> /I2C0 SDA
- U4 pad 14: +3V3 -> /I2C0 SCL
- U4 pad 2: unconnected-(U4-NC-Pad2) -> GND
- U4 pad 5: unconnected-(U4-CSB2-Pad5) -> GND
- U4 pad 6: GND -> +3V3
- U4 pad 8: /I2C0 SCL -> unconnected-(U4-INT1-Pad8)
- U4 pad 9: /I2C0 SDA -> unconnected-(U4-INT2-Pad9)
- U5 pad 1: +3V3 -> /I2C0 SCL
- U5 pad 2: Net-(U5-CAP) -> GND
- U5 pad 4: +3V3 -> Net-(U5-C1)
- U5 pad 5: unconnected-(U5-INT2-Pad5) -> +3V3
- U5 pad 6: unconnected-(U5-INT1-Pad6) -> +3V3
- U5 pad 7: /I2C0 SDA -> unconnected-(U5-INT-Pad7)
- U5 pad 8: /I2C0 SCL -> unconnected-(U5-DRDY-Pad8)
- U6 pad 10: unconnected-(U6-NC-Pad10) -> /I2C1 SCL
- U6 pad 2: GND -> unconnected-(U6-ALERT/RDY-Pad2)
- U6 pad 3: +3V3 -> GND
- U6 pad 4: GND -> /P1 CONT 
- U6 pad 5: GND -> /P2 CONT 
- U6 pad 6: +3V3 -> /P3 CONT 
- U6 pad 7: +3V3 -> /P4 CONT 
- U6 pad 8: unconnected-(U6-INT1-Pad8) -> +3V3
- U6 pad 9: unconnected-(U6-INT2-Pad9) -> /I2C1 SDA
- U7 pad 1: /I2C0 SCL -> /QSPI_SS
- U7 pad 2: GND -> /QSPI_SD1
- U7 pad 3: GND -> /QSPI_SD2
- U7 pad 4: Net-(U7-C1) -> GND
- U7 pad 5: +3V3 -> /QSPI_SDO
- U7 pad 6: +3V3 -> /QSPI_SCLK
- U7 pad 7: unconnected-(U7-INT-Pad7) -> /QSPI_SD3
- U7 pad 8: unconnected-(U7-DRDY-Pad8) -> +3V3
- U7 pad 9: GND -> unconnected-(U7-EP-Pad9)
- U8 pad 12: /LEDRED -> unconnected-(U8-GPIO9-Pad12)
- U8 pad 13: /LEDGREEN -> unconnected-(U8-GPIO10-Pad13)
- U8 pad 14: /LEDBLUE -> unconnected-(U8-GPIO11-Pad14)
- U8 pad 15: /SERVO1 -> unconnected-(U8-GPIO12-Pad15)
- U8 pad 16: /SERVO2 -> /BRKOUT5
- U8 pad 17: /SERVO3 -> /BRKOUT6
- U8 pad 18: /SERVO4 -> /BRKOUT7
- U8 pad 2: /SPI0 GPIO -> /BRKOUT1
- U8 pad 27: /UART0 TX -> unconnected-(U8-GPIO16-Pad27)
- U8 pad 28: /UART0 RX -> unconnected-(U8-GPIO17-Pad28)
- U8 pad 29: /SPI0 SCK -> unconnected-(U8-GPIO18-Pad29)
- U8 pad 3: unconnected-(U8-GPIO1-Pad3) -> /BRKOUT2
- U8 pad 30: /SPI0 MISO -> unconnected-(U8-GPIO19-Pad30)
- U8 pad 31: /SPI0 MOSI -> unconnected-(U8-GPIO20-Pad31)
- U8 pad 32: /SPI0 CSn -> unconnected-(U8-GPIO21-Pad32)
- U8 pad 34: /I2C1 SDA -> unconnected-(U8-GPIO22-Pad34)
- U8 pad 35: /I2C1 SCL -> /LEDRED
- U8 pad 36: /UART GPIO -> /LEDGREEN
- U8 pad 37: unconnected-(U8-GPIO25-Pad37) -> /LEDBLUE
- U8 pad 4: /SD CS -> /BRKOUT3
- U8 pad 40: unconnected-(U8-GPIO28_ADC2-Pad40) -> /BATT SENSE 
- U8 pad 5: unconnected-(U8-GPIO3-Pad5) -> /BRKOUT4
- U9 pad 1: +3V3 -> +12VA
- U9 pad 2: unconnected-(U9-ALERT/RDY-Pad2) -> Net-(U9-GND)
- U9 pad 3: GND -> +12VA
- U9 pad 4: /P3 CONT BOT -> Net-(U9-BP)
- U9 pad 5: /P4 CONT BOT -> +3V3
Routing:
- removed copper zone on B.Cu, net +3V3
- removed copper zone on F.Cu, net +3V3
- removed copper zone on B.Cu, net GND
- removed copper zone on F.Cu, net GND
Other:
- board size 50 x 60 mm -> 25 x 60 mm
- board text removed: "GND"
- board text removed: "LYRA V3"
- board text removed: "P1+"
- board text removed: "P1-"
- board text removed: "P2+"
- board text removed: "P2-"
- board text removed: "P3+"
- board text removed: "P3-"
- board text removed: "P4+"
- board text removed: "P4-"
- board text removed: "PRS"
