File: Hardware/kicad/Lyra_flight_computer/lyragps/lyragps/lyragps.kicad_pcb (KiCad board)
At the start: 2 copper layers, 25 x 38.4 mm, 8 parts, among them IC1 TESEO-LIV4FTR, J2 Conn_01x06, J3 Conn_01x04

Commit message: cui
Parts:
- moved IC1 6.41 mm to (162.4, 81.9)
- moved ANT1 5.49 mm to (161.8, 74.1)
Changed lines of the file:
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@@
   (net 29 "unconnected-(ANT1-FEED-Pad1)")
   (footprint "SamacSys_Parts.3dshapes:GP1575124A02" (layer "F.Cu")
-    (at 161.925 79.629)
+    (at 161.8234 74.1426)
     (descr "GP.1575.12.4.A.02-1")
     (tags "Antenna")
@@
   )
   (footprint "SamacSys_Parts.3dshapes:TESEOLIV4FTR" (layer "B.Cu")
-    (at 166.116 87.094 180)
+    (at 162.4076 81.8642 180)
     (descr "TESEO-LIV4FTR-1")
     (tags "Integrated Circuit")
