File: Hardware/kicad/Lyra_flight_computer/lyrav3r1/lyrav3r1/_autosave-lyrav3r1.kicad_pcb (KiCad board)
At the start: 4 copper layers, 25 x 55 mm, 106 parts, among them IC1 TESEO-LIV3F, J1 Conn_01x02, J2 Screw_Terminal_01x06, J3 Conn_Coaxial, J4 Conn_01x02, J7 USB_B_Micro, J9 Screw_Terminal_01x06, Q1 AO3401A, Q2 AO3400A, Q3 AO3400A, Q4 AO3400A, Q5 AO3400A, U1 SX1262, U2 BMI088, U3 BMP388, U4 ADXL375BCCZ-RL7, U5 M3406, U6 SKY13453-385LF, U7 WS7916S-6/TR, U8 RP2040, U9 W25Q128JVS, X2 SX1M12.000M10F30TNN, Y1 CF4032M00012001

Commit message: stufffff
Parts:
- moved IC1 4.96 mm to (202.6, 76.1)
- moved J3 0.11 mm to (195.7, 66.1)
Changed lines of the file:
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@@
 	(footprint "Connector_Coaxial:SMA_Samtec_SMA-J-P-X-ST-EM1_EdgeMount"
 		(layer "B.Cu")
-		(at 195.707 66.0035)
+		(at 195.707 66.113)
 		(descr "Connector SMA, 0Hz to 20GHz, 50Ohm, Edge Mount (http://suddendocs.samtec.com/prints/sma-j-p-x-st-em1-mkt.pdf)")
 		(tags "SMA Straight Samtec Edge Mount")
@@
 	(footprint "SamacSys_Parts:SON110P970X1010X230-18N"
 		(layer "B.Cu")
-		(at 202.311 81.026 180)
+		(at 202.565 76.073 180)
 		(descr "TESEO-LIV3F")
 		(tags "Integrated Circuit")
