File: Hardware/kicad/Lyra_flight_computer/lyrav3r1/lyrav3r1/lyrav3r1.kicad_sch (KiCad schematic)
At the start: 119 parts, among them IC1 TESEO-LIV3F, J1 Conn_01x02, J2 Screw_Terminal_01x06, J3 Conn_Coaxial, J4 Conn_01x02, J5 Conn_01x05, J7 USB_B_Micro, J9 Screw_Terminal_01x06, Q1 AO3401A, Q2 AO3400A, Q3 AO3400A, Q4 AO3400A, Q5 AO3400A, Q6 NPN, U1 SX1262, U2 BMI088, U3 BMP388, U4 ADXL375BCCZ-RL7, U5 M3406, U6 SKY13453-385LF, U7 WS7916S-6/TR, U8 RP2040, U9 W25Q128JVS, X2 SX1M12.000M10F30TNN, Y1 CF4032M00012001

Commit message: w45dytfv
Parts:
- removed R13, R24, R25: 5.1k, Resistor_SMD:R_0402_1005Metric, symbol Device:R_Small
- removed R16, R26, R27: 1k, Resistor_SMD:R_0402_1005Metric, symbol Device:R_Small
- removed R21, R23: 15k, Resistor_SMD:R_0402_1005Metric, symbol Device:R_Small
- added Q10, Q7, Q8, Q9: AO3400A, Package_TO_SOT_SMD:SOT-23, symbol Transistor_FET:AO3400A
- AE1: footprint (none) -> APAE1575R1820ABDC1_T:XDCR_APAE1575R1820ABDC1-T
- J5: footprint (none) -> .pretty:Pad_01x_05
- R10, R11: value 15k -> 1k; LCSC Part C25756 -> C11702
- R12: value 5.1k -> 1k; LCSC Part C25905 -> C11702
- TP1: footprint TestPoint:TestPoint_Keystone_5019_Minature -> TestPoint:TestPoint_Pad_1.0x1.0mm
Connections:
- net GND: now also R10.1, R11.1, R12.1, Q10.2 (S), Q7.2 (S), Q8.2 (S), Q9.2 (S); no longer R12.2
- net P1 CONT : now also Q7.3 (D); no longer R10.2, R12.1
- net P1 EN : now also Q4.1 (G), R17.2; no longer Q3.1 (G)
- net P1-: now also Q4.3 (D), Q7.1 (G); no longer Q3.3 (D), R10.1
- net P2 CONT : now also Q3.3 (D)
- net P2 EN : now also R10.2
- net P2-: now also Q3.1 (G)
- net P3 CONT : now also Q8.3 (D); no longer R11.2
- net P3 EN : now also Q5.1 (G), R11.2; no longer Q4.1 (G), R17.2
- net P3-: now also Q5.3 (D), Q8.1 (G); no longer Q4.3 (D), R11.1
- net P4 CONT : now also Q10.3 (D)
- net P4 EN : now also R12.2, Q9.1 (G); no longer Q5.1 (G)
- net P4-: now also Q10.1 (G), Q9.3 (D); no longer Q5.3 (D)
Other:
- moved on the sheet: Q4, R17

Commit message: asd
Parts:
- removed Q6: NPN, symbol Simulation_SPICE:NPN
- added C32, C33: 120p, symbol Device:C_Small
- added FL1: SAFEA1G58KA0F00R15, .pretty:FILTER-SMD_5P-L1.4-W1.1-L, symbol .kicad_sym:SAFEA1G58KA0F00R15
- added Q6: Q_NPN_BCE, symbol Device:Q_NPN_BCE
Connections:
- net +12P is gone; now on net +BATT: C5.1, C7.1, C8.1, C9.1, J2.2 (Pin_2), J9.1 (Pin_1), J9.3 (Pin_3), J9.5 (Pin_5), Q1.2 (S), R4.1, U5.1 (RUN), U5.4 (VIN)
- net +BATT: now also Q6.3 (E); no longer J2.4 (Pin_4), J2.6 (Pin_6)
- net ANT: now also C32.2; no longer U7.6 (RFOUT)
- net ANT IN: now also C33.1; no longer L3.1
- net BUZZER: now also Q6.1 (B)
- net GND: now also FL1.2 (GND), FL1.3 (GND), FL1.5 (GND)
- net at BZ1.1 (+): now also Q6.2 (C)
- net +12V renamed BATT POSTSW
- new net: C33.2, L3.1
- new net: C32.1, FL1.4 (OUT)
- new net: FL1.1 (IN), U7.6 (RFOUT)
- new net BATT RAW: J2.4 (Pin_4), J2.6 (Pin_6)
Other:
- moved on the sheet: C7, C8, C9, D1, D2, J2, Q1, R3

Commit message: work
Parts:
- removed C9: 680uf, Capacitor_THT:CP_Radial_D6.3mm_P2.50mm, symbol Device:C_Small
- added R13, R16: 5.1k, Resistor_SMD:R_0402_1005Metric, symbol Device:R_Small
- C32: footprint (none) -> Capacitor_SMD:C_0402_1005Metric
Connections:
- net +3V3: now also R13.1, R16.1; no longer U4.7 (~{CS})
- net +BATT: now also Q6.2 (C); no longer Q6.3 (E)
- net BRKOUT1: no longer U8.37 (GPIO25)
- net BUZZER: no longer U8.32 (GPIO21)
- net GND: no longer U4.12 (SDO/ALTADDRESS)
- net MISO: now also U2.15 (SDO1), U3.4 (SDI), U4.12 (SDO/ALTADDRESS), U8.36 (GPIO24)
- net MOSI: now also U2.9 (SDA/SDI), U3.5 (SDO), U4.13 (SDA/SDI/SDIO), U8.35 (GPIO23)
- net P1 CONT : now also U8.29 (GPIO18); no longer U8.6 (GPIO4)
- net P1 EN : now also U8.30 (GPIO19); no longer U8.7 (GPIO5)
- net P2 CONT : now also U8.27 (GPIO16); no longer U8.4 (GPIO2)
- net P2 EN : now also U8.28 (GPIO17); no longer U8.5 (GPIO3)
- net P3 CONT : now also U8.17 (GPIO14); no longer U8.2 (GPIO0)
- net P3 EN : now also U8.18 (GPIO15); no longer U8.3 (GPIO1)
- net P4 CONT : now also U8.31 (GPIO20); no longer U8.8 (GPIO6)
- net P4 EN : now also U8.32 (GPIO21); no longer U8.9 (GPIO7)
- net SCK: now also U2.8 (SCL/SCK), U3.2 (SCK), U4.14 (SCL/SCLK), U8.34 (GPIO22)
- net SCL: now also U8.3 (GPIO1), R16.2
- net SDA: now also U8.2 (GPIO0), R13.2
- net SX CS: now also U8.37 (GPIO25)
- net BMP CS: now reaches U3.6 (CSB)
- net BMIACCEL CS: now reaches U2.14 (CSB1)
- net BMIGYRO CS: now reaches U2.5 (CSB2)
- net at BZ1.1 (+): now also Q6.3 (E); no longer Q6.2 (C)
- new net ADXL CS: U4.7 (~{CS})
- no-connect marks 27 -> 20
Other:
- note added: "C45 and C46 not populated"
- note added: "Internal pullups on the RP2040"
- note added: "LNA and SAW filter"
- note removed: "C23 and C24 not populated"
- moved on the sheet: AE1, C1, C16, C17, C18, C19, C2, C21, C22, C23, C24, C25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

Commit message: asdfghj
Parts:
- removed U5: M3406, .pretty:SOT-23-5_L3.0-W1.7-P0.95-LS2.8-BR, symbol .kicad_sym:M3406
- added C9: 22u, Capacitor_SMD:C_0805_2012Metric, symbol Device:C_Small
- added U10: MT2492, .pretty:SOT-23-6_L2.9-W1.6-P0.95-LS2.8-BL, symbol .kicad_sym:MT2492
- BZ1: footprint (none) -> .pretty:Buzzer_12x9.5RM7.6; Part # (none) -> PKHPS0013E4000-A2
- C5: value 4u7 -> 22u; footprint Capacitor_SMD:C_0603_1608Metric -> Capacitor_SMD:C_0805_2012Metric; LCSC Part (none) -> C45783
- C6: value 10u -> 22nf; footprint Capacitor_SMD:C_0603_1608Metric -> Capacitor_SMD:C_0402_1005Metric; LCSC Part (none) -> C1532
- L2: value 2u2 -> 4.7u
- R4: value 15k -> 40k; LCSC Part C25756 -> (none)
- R5: value 5.1k -> 25k; LCSC Part C25905 -> (none)
- R7: value 15k -> 110k; footprint Resistor_SMD:R_0402_1005Metric -> Resistor_SMD:R_0603_1608Metric; LCSC Part (none) -> C25805
- R8: value 50k -> 20k; LCSC Part (none) -> C25765
Connections:
- net +3V3: now also R7.1, C9.1; no longer C6.1
- net +BATT: now also BZ1.1 (+), U10.4 (EN), U10.5 (IN); no longer Q6.2 (C)
- net GND: now also Q6.3 (E), C9.2, U10.2 (GND); no longer BZ1.2 (-), C6.2
- net at L2.1: now also C6.2, U10.6 (SW); no longer R7.1
- net at R7.2, R8.1: now also U10.3 (FB)
- new net: BZ1.2 (-), Q6.2 (C)
- new net: C6.1, U10.1 (BS)
Other:
- moved on the sheet: BZ1

Commit message: redoing stuff
Parts:
- removed C10: 1u, Capacitor_SMD:C_0402_1005Metric, symbol Device:C_Small
- removed C11: 100n, Capacitor_SMD:C_0402_1005Metric, symbol Device:C_Small
- removed D4: LED_ARGB, customfootprints:LED_Cree-PLCC4_2x2mm_CCW, symbol Device:LED_ARGB
- removed D7: LED, symbol Device:LED
- removed J2, J9: Screw_Terminal_01x06, TerminalBlock_Phoenix:TerminalBlock_Phoenix_MPT-0,5-6-2.54_1x06_P2.54mm_Horizontal, symbol Connector:Screw_Terminal_01x06
- removed R2, R22, R9: 1k, Resistor_SMD:R_0402_1005Metric, symbol Device:R_Small
- removed U4: ADXL375BCCZ-RL7, easyeda2kicad:LGA-14_L5.0-W3.0-P0.80-BL, symbol easyeda2kicad:ADXL375BCCZ-RL7
- added C34: 10u, Capacitor_SMD:C_0603_1608Metric, symbol Device:C_Small
- added C50: 100n, Capacitor_SMD:C_0402_1005Metric, symbol Device:C_Small
- added D3: LED, LED_SMD:LED_0805_2012Metric, symbol Device:LED
- added J2: Screw_Terminal_01x02, TerminalBlock_Phoenix:TerminalBlock_Phoenix_MPT-0,5-2-2.54_1x02_P2.54mm_Horizontal, symbol Connector:Screw_Terminal_01x02
- added J8: Screw_Terminal_01x07, TerminalBlock_Phoenix:TerminalBlock_Phoenix_MPT-0,5-7-2.54_1x07_P2.54mm_Horizontal, symbol Connector:Screw_Terminal_01x07
- added TP2, TP3: TestPoint, TestPoint:TestPoint_Pad_1.0x1.0mm, symbol Connector:TestPoint
- added U5: ADXL375BCCZ-RL7, easyeda2kicad:LGA-14_L5.0-W3.0-P0.80-BL, symbol easyeda2kicad:ADXL375BCCZ-RL7
- C14: footprint (none) -> Capacitor_SMD:C_0603_1608Metric; LCSC Part (none) -> C96446
- C15: value 10u -> 1n; footprint (none) -> Capacitor_SMD:C_0402_1005Metric; LCSC Part (none) -> C1523
- C20: footprint (none) -> Capacitor_SMD:C_0603_1608Metric; LCSC Part (none) -> C39148
- C28: footprint (none) -> Capacitor_SMD:C_0402_1005Metric; LCSC Part (none) -> C1523
- C32: value 120p -> 1u; LCSC Part (none) -> C52923
- C33: value 120p -> 1n; footprint (none) -> Capacitor_SMD:C_0402_1005Metric; LCSC Part (none) -> C1523
- L2: footprint (none) -> Inductor_SMD:L_Changjiang_FNR3015S; LCSC Part (none) -> C2762019
Connections:
- net BMIACCEL CS is gone; now on net +3V3: U2.14 (CSB1)
- net BMP CS is gone; now on net +3V3: U3.6 (CSB)
- net LEDRED is gone; now on net GPS_RST: U8.14 (GPIO11)
- net RF GND 1 is gone; now on net GND: IC1.10 (GND_RF_1)
- net RF GND 2 is gone; now on net GND: IC1.12 (GND_RF_2)
- net +3V3: now also C32.1, U2.7 (PS), C50.1, D3.1 (K), U5.1 (VDDI/O), U5.3 (RESERVED), U5.6 (VS), U5.7 (~{CS})
- net +BATT: now also J8.1 (Pin_1)
- net ANT: now also C33.2; no longer C32.2
- net ANT IN: now also C15.1; no longer C33.1
- net BATT POSTSW: now also J2.1 (Pin_1)
- net BATT RAW: now also J2.2 (Pin_2), J8.7 (Pin_7)
- net BRKOUT1: now also U8.18 (GPIO15)
- net BUSY: now also U8.9 (GPIO7)
- net BUZZER: now also U8.28 (GPIO17)
- net DIO1: now also U8.11 (GPIO8)
- net GND: now also C32.2, U2.10 (SDO2), U2.15 (SDO1), U3.5 (SDO), C34.2, C50.2, J8.6 (Pin_6), TP3.1, U5.11 (RESERVED), U5.12 (SDO/ALTADDRESS), U5.2 (GND), U5.4 (GND), U5.5 (GND); no longer C15.2
- net GPS 3v3: now also C34.1; no longer C15.1
- net MISO: now also U8.6 (GPIO4); no longer U2.15 (SDO1), U3.4 (SDI), U8.36 (GPIO24)
- net MOSI: now also U8.5 (GPIO3); no longer U2.9 (SDA/SDI), U3.5 (SDO), U8.35 (GPIO23)
- net P1 CONT : now also U8.30 (GPIO19); no longer U8.29 (GPIO18)
- net P1 EN : now also U8.29 (GPIO18); no longer U8.30 (GPIO19)
- net P1-: now also J8.5 (Pin_5)
- net P2 CONT : now also U8.32 (GPIO21); no longer U8.27 (GPIO16)
- net P2 EN : now also U8.31 (GPIO20); no longer U8.28 (GPIO17)
- net P2-: now also J8.4 (Pin_4)
- net P3 CONT : now also U8.35 (GPIO23); no longer U8.17 (GPIO14)
- net P3 EN : now also U8.34 (GPIO22); no longer U8.18 (GPIO15)
- net P3-: now also J8.3 (Pin_3)
- net P4 CONT : now also U8.37 (GPIO25); no longer U8.31 (GPIO20)
- net P4 EN : now also U8.36 (GPIO24); no longer U8.32 (GPIO21)
- net P4-: now also J8.2 (Pin_2)
- net SCK: now also U8.8 (GPIO6); no longer U2.8 (SCL/SCK), U3.2 (SCK), U8.34 (GPIO22)
- net SCL: now also U2.8 (SCL/SCK), U3.2 (SCK), U8.16 (GPIO13), U5.14 (SCL/SCLK); no longer U8.3 (GPIO1)
- net SDA: now also U2.9 (SDA/SDI), U3.4 (SDI), U8.15 (GPIO12), U5.13 (SDA/SDI/SDIO); no longer U8.2 (GPIO0)
- net SX CS: now also U8.7 (GPIO5); no longer U8.37 (GPIO25)
- net at L3.1: now also C15.2; no longer C33.2
- net at FL1.4 (OUT): now also C33.1; no longer C32.1
- net at R28.2: now also D3.2 (A)
- net BMIGYRO CS: no longer names the net of U2.5 (CSB2)
- net LEDBLUE: no longer names the net of U8.12 (GPIO9)
- net LEDBLUE: no longer R28.1
- net LEDGREEN: no longer names the net of U8.13 (GPIO10)
- net PPS: no longer names the net of C20.1, IC1.4 (1PPS)
- net PPS: now also TP2.1
- new net LEDINDICATION: R28.1
Other:
- moved on the sheet: C1, C2, J4, L2, Q10, Q2, Q3, Q4, Q5, Q7, Q8, Q9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

Commit message: found new gps chip and getting close t oend of schematic
Parts:
- removed C29: 470nF, Capacitor_SMD:C_0402_1005Metric, symbol Device:C
- removed C30, C40: 100pF, Capacitor_SMD:C_0402_1005Metric, symbol Device:C
- removed C31, C38: 3.3pF, Capacitor_SMD:C_0402_1005Metric, symbol Device:C
- removed C35: 22nF, Capacitor_SMD:C_0402_1005Metric, symbol Device:C
- removed C36: 4.7pF, Capacitor_SMD:C_0402_1005Metric, symbol Device:C
- removed C37: 1pF, Capacitor_SMD:C_0402_1005Metric, symbol Device:C
- removed C39: 18pF, Capacitor_SMD:C_0402_1005Metric, symbol Device:C
- removed C41: 15pF, Capacitor_SMD:C_0402_1005Metric, symbol Device:C
- removed C42, C43, C47, C48, C49: 100nF, Capacitor_SMD:C_0402_1005Metric, symbol Device:C
- removed C44: 33pF, Capacitor_SMD:C_0402_1005Metric, symbol Device:C
- removed C45, C46: TBD, Capacitor_SMD:C_0402_1005Metric, symbol Device:C
- removed FB2: 200mA, Inductor_SMD:L_0603_1608Metric, symbol Device:FerriteBead
- removed J3: Conn_Coaxial, Connector_Coaxial:SMA_Samtec_SMA-J-P-X-ST-EM1_EdgeMount, symbol Connector:Conn_Coaxial
- removed L3: 10n, symbol Device:L_Small
- removed L4: 15uH, Inductor_SMD:L_0603_1608Metric, symbol Device:L
- removed L5: 33nH, Inductor_SMD:L_0402_1005Metric, symbol Device:L
- removed L6: 68nH, Inductor_SMD:L_0402_1005Metric, symbol Device:L
- removed L7: 3.9nH, Inductor_SMD:L_0402_1005Metric, symbol Device:L
- removed L8: 15nH, Inductor_SMD:L_0402_1005Metric, symbol Device:L
- removed L9: 0R, Inductor_SMD:L_0402_1005Metric, symbol Device:L
- removed Q6: Q_NPN_BCE, symbol Device:Q_NPN_BCE
- removed R19: 100R, Resistor_SMD:R_0402_1005Metric, symbol Device:R
- removed R6: 5.1k, Resistor_SMD:R_0402_1005Metric, symbol Device:R_Small
- removed U1: SX1262, Package_DFN_QFN:QFN-24-1EP_4x4mm_P0.5mm_EP2.7x2.7mm, symbol stanley_misc:SX1262
- removed U6: SKY13453-385LF, .pretty:QFN-6_L1.0-W1.0-P0.50-LS1.0-BL, symbol stanley_misc:SKY13453-385LF
- removed Y1: CF4032M00012001, Crystal:Crystal_SMD_3225-4Pin_3.2x2.5mm, symbol Device:Crystal_GND24_Small
- added AE2: Antenna, .pretty:SMA-SMD_HJ-SMA086, symbol Device:Antenna
- added L4: 10n, Inductor_SMD:L_0402_1005Metric, symbol Device:L_Small
- added Q11: Q_NPN_BEC, Package_TO_SOT_SMD:SOT-23, symbol Device:Q_NPN_BEC
- added U4: VGDD79S868N0S1, .pretty:WIRELM-SMD_L11.5-W11.5-P1.50-BL, symbol .kicad_sym:VGDD79S868N0S1
- AE1: footprint APAE1575R1820ABDC1_T:XDCR_APAE1575R1820ABDC1-T -> .pretty:APAE1575R1240ABDD1-T
- C14: value 10u -> 10n; footprint Capacitor_SMD:C_0603_1608Metric -> Capacitor_SMD:C_0402_1005Metric; LCSC Part C96446 -> C15195
- C34: value 10u -> 56p; LCSC Part C96446 -> C39148
- L1: value 27n -> 10n; footprint (none) -> Inductor_SMD:L_0402_1005Metric; LCSC Part (none) -> C27147
Connections:
- net +3V3: now also U4.6 (VCC)
- net BUSY: now also U4.11 (BUSY)
- net BUZZER: now also Q11.1 (B)
- net DIO1: now also U4.10 (DIO1)
- net GND: now also Q11.2 (E), U4.12 (GND), U4.13 (GND), U4.7 (GND), U4.9 (GND)
- net LEDINDICATION: now also U8.17 (GPIO14)
- net MISO: now also U4.2 (MISO)
- net MOSI: now also U4.3 (MOSI)
- net SCK: now also U4.4 (SCK)
- net SX CS: now also U4.5 (NSS)
- net at C15.2: now also L4.1
- net at BZ1.2 (-): now also Q11.3 (C)
- net DIO3: now reaches U8.3 (GPIO1)
- net DIO3: now also U4.8 (DIO3)
- net SX RST: now reaches U8.4 (GPIO2)
- net SX RST: now also U4.1 (RST)
- net at U7.3 (RFIN): now also L4.2
- new net: AE2.1 (A), U4.14 (ANT)
- no-connect marks 20 -> 22
Other:
- note added: "Hardware guide says 27nh, but jlc only has 10nh but it should be fine?"
- note removed: "50 ohm"
- note removed: "C45 and C46 not populated"
- note removed: "From the datasheet: Load Capacitance = 12pf therefore needed capacitance = 15pf (assuming 4pf parasitic)"
- moved on the sheet: L1

Commit message: qwe
Parts:
- removed U4: VGDD79S868N0S1, .pretty:WIRELM-SMD_L11.5-W11.5-P1.50-BL, symbol .kicad_sym:VGDD79S868N0S1
- added U1: E22-400MM22S, .pretty:WIRELM-SMD_E22-400MM22S, symbol .kicad_sym:E22-400MM22S
Connections:
- net +3V3: now also U1.1 (VCC)
- net BUSY: now also U1.11 (BUSY)
- net GND: now also U1.16 (GND), U1.2 (GND), U1.7 (GND)
- net MISO: now also U1.12 (MISO)
- net MOSI: now also U1.13 (MOSI)
- net SCK: now also U1.15 (SCK)
- net SX CS: now also U1.14 (NSS)
- net SX RST: now also U1.3 (NRST)
- net at AE2.1 (A): now also U1.6 (ANT)
- no-connect marks 22 -> 31
Other:
- moved on the sheet: AE2

Commit message: first pass at routing
Parts:
- removed AE2: Antenna, .pretty:SMA-SMD_HJ-SMA086, symbol Device:Antenna
- removed C8: 1u, Capacitor_SMD:C_0402_1005Metric, symbol Device:C_Small
- removed C9: 22u, Capacitor_SMD:C_0805_2012Metric, symbol Device:C_Small
- removed L2: 4.7u, Inductor_SMD:L_Changjiang_FNR3015S, symbol Device:L_Small
- removed R5: 25k, Resistor_SMD:R_0402_1005Metric, symbol Device:R_Small
- removed R7: 110k, Resistor_SMD:R_0603_1608Metric, symbol Device:R_Small
- removed R8: 20k, Resistor_SMD:R_0402_1005Metric, symbol Device:R_Small
- removed TP3: TestPoint, TestPoint:TestPoint_Pad_1.0x1.0mm, symbol Connector:TestPoint
- removed U10: MT2492, .pretty:SOT-23-6_L2.9-W1.6-P0.95-LS2.8-BL, symbol .kicad_sym:MT2492
- added AE3: Antenna_Shield, .pretty:CONN-SMD_KH-SMA-KE8-G, symbol Device:Antenna_Shield
- added C10: 10n, Capacitor_SMD:C_0402_1005Metric, symbol Device:C_Small
- added C11: 10u, Capacitor_SMD:C_0603_1608Metric, symbol Device:C_Small
- added C29: 100n, Capacitor_SMD:C_0402_1005Metric, symbol Device:C_Small
- added R2: 20k, Resistor_SMD:R_0402_1005Metric, symbol Device:R_Small
- added U6: RT9013-33GB_C19268157, .pretty:SOT-23-5_L2.9-W1.6-P0.95-LS2.8-BR, symbol .kicad_sym:RT9013-33GB_C19268157
- AE1, BZ1, D2, D3, IC1, J2, J5, J8, TP1, TP2: now left out of the parts list
- C5: value 22u -> 1u; footprint Capacitor_SMD:C_0805_2012Metric -> Capacitor_SMD:C_0402_1005Metric; LCSC Part C45783 -> C52923
- C6: value 22nf -> 1u; LCSC Part C1532 -> C52923
- Q1: LCSC Part C15127 -> C15127
- R4: LCSC Part (none) -> C25086
- U1: value E22-400MM22S -> E22-900MM22S; LCSC Part C5333984 -> (none); now left out of the parts list
Connections:
- net DIO3 is gone; now on net TXEN: U8.3 (GPIO1)
- net +3V3: now also C5.1, C10.1, C11.1, U6.5 (VOUT)
- net +BATT: now also C6.1, U6.1 (VIN), U6.3 (CE); no longer C5.1
- net BATT SENSE : now also R2.1
- net BRKOUT1: now also U8.13 (GPIO10); no longer U8.18 (GPIO15)
- net BUZZER: now also U8.27 (GPIO16); no longer U8.28 (GPIO17)
- net GND: now also C6.2, AE3.2 (Shield), C10.2, C11.2, C29.2, R2.2, U6.2 (GND)
- net LEDINDICATION: now also U8.28 (GPIO17); no longer U8.17 (GPIO14)
- net P1 CONT : now also U8.29 (GPIO18); no longer U8.30 (GPIO19)
- net P1 EN : now also U8.30 (GPIO19); no longer U8.29 (GPIO18)
- net P2 CONT : now also U8.31 (GPIO20); no longer U8.32 (GPIO21)
- net P2 EN : now also U8.32 (GPIO21); no longer U8.31 (GPIO20)
- net P3 CONT : now also U8.34 (GPIO22); no longer U8.35 (GPIO23)
- net P3 EN : now also U8.35 (GPIO23); no longer U8.34 (GPIO22)
- net P4 CONT : now also U8.36 (GPIO24); no longer U8.37 (GPIO25)
- net P4 EN : now also U8.37 (GPIO25); no longer U8.36 (GPIO24)
- net SX RST: now also C29.1
- net RXEN: now reaches U1.10 (RXEN)
- net RXEN: now also U8.2 (GPIO0)
- net at U1.6 (ANT): now also AE3.1 (A)
- net TXEN: now reaches U1.9 (TXEN)
- net DIO1: no longer names the net of U8.11 (GPIO8)
- no-connect marks 31 -> 30
Other:
- moved on the sheet: C7
