File: Hardware/kicad/Lyra_flight_computer/lyrav3r1/recivier/recivier.kicad_sch (KiCad schematic)
At the start: 83 parts, among them J1 USB_B_Micro, J2 Conn_01x02, J3 Conn_01x02, J4 Screw_Terminal_01x02, J5 Screw_Terminal_01x02, Q1 AO3401A, SW1 K2-1102DP-L3SW-04, SW2 K2-1102DP-L3SW-04, SW3 K2-1102DP-L3SW-04, SW4 K2-1102DP-L3SW-04, SW5 K2-1102DP-L3SW-04, U1 E22-900MM22S, U2 W25Q128JVS, U3 RP2040, U4 TXB0104RGY, U5 PCM5102A, U6 ATGM336H-5N31, U7 LIS3MDLTR, U8 AMS1117-3.3, U9 AMS1117-5.0, X1 SX1M12.000M10F30TNN

Commit message: reciver work and finalized lyrav3r1
Parts:
- added R16: 1k, Resistor_SMD:R_0402_1005Metric, symbol Device:R_Small
- added R17: 40k, Resistor_SMD:R_0402_1005Metric, symbol Device:R_Small
- added SW6: SW_SPDT, .pretty:SW-TH_SK12D07VG4, symbol Switch:SW_SPDT
- D2: now in the parts list
- DS1: footprint Display:AG12864E -> .pretty:ST7920 AZ; now left out of the parts list
- J4, J5: footprint (none) -> TerminalBlock:TerminalBlock_bornier-2_P5.08mm; LCSC Part (none) -> C395882
- R9: footprint (none) -> Resistor_SMD:R_0402_1005Metric; LCSC Part (none) -> C25117
- RV1: footprint (none) -> .pretty:RES-ADJ-SMD_3314J
- SW1, SW2, SW3, SW4, SW5: footprint :SW-TH_4P-L6.0-W6.0-P4.50-LS6.5 -> .pretty:SW-TH_4P-L6.0-W6.0-P4.50-LS6.5
- U6: footprint :GPSM-SMD_ATGM336H-TR -> .pretty:GPSM-SMD_ATGM336H-TR
Connections:
- net +3.3VA: now also SW1.1, SW2.2, SW3.1, SW4.1, SW5.1; no longer SW2.1
- net +5V: now also RV1.3; no longer RV1.1
- net +BATT: now also R17.1, SW6.1 (A); no longer C35.1, Q1.2 (S)
- net BCK: now also U3.11 (GPIO8); no longer U3.28 (GPIO17)
- net BUSY: now also U3.31 (GPIO20); no longer U3.9 (GPIO7)
- net BUTTON1: now also U3.6 (GPIO4); no longer SW1.4, U3.30 (GPIO19)
- net BUTTON2: now also U3.2 (GPIO0); no longer SW2.4, U3.31 (GPIO20)
- net BUTTON3: now also U3.4 (GPIO2); no longer SW3.4, U3.32 (GPIO21)
- net BUTTON4: now also U3.5 (GPIO3); no longer SW4.4, U3.34 (GPIO22)
- net BUTTON5: now also U3.3 (GPIO1); no longer SW5.4, U3.35 (GPIO23)
- net DIN: now also U3.13 (GPIO10); no longer U3.27 (GPIO16)
- net GND: now also RV1.1, R16.1; no longer RV1.3
- net LCD CS: now also U3.17 (GPIO14), U4.2 (A1); no longer DS1.4 (RS), U3.11 (GPIO8), U4.12 (B2), U4.3 (A2)
- net LRCK: now also U3.14 (GPIO11); no longer U3.18 (GPIO15)
- net MISO: now also U3.36 (GPIO24); no longer U3.6 (GPIO4)
- net MOSI: now also U3.35 (GPIO23), U4.3 (A2); no longer U3.5 (GPIO3), U4.4 (A3)
- net MOSI 2 5V: now also U4.12 (B2); no longer U4.11 (B3)
- net RXEN: now also U3.40 (GPIO28_ADC2); no longer U3.2 (GPIO0)
- net SCK: now also U3.12 (GPIO9); no longer Card1.5 (CLK), U1.15 (SCK), U3.29 (GPIO18), U3.8 (GPIO6), U4.2 (A1)
- net SD_CS: now also U3.38 (GPIO26_ADC0); no longer U3.12 (GPIO9)
- net SX CS: now also U3.32 (GPIO21); no longer U3.7 (GPIO5)
- net SX RST: now also U3.30 (GPIO19); no longer U3.4 (GPIO2)
- net TXEN: now also U3.39 (GPIO27_ADC1); no longer U3.3 (GPIO1)
- net BATT SENSE: now reaches U3.41 (GPIO29_ADC3)
- net BATT SENSE: now also R16.2, R17.2
- net SCK 2 5V renamed LCD CS 5V
- net LCD CS 5V: now also DS1.4 (RS); no longer DS1.6 (E)
- new net: C35.1, Q1.2 (S), SW6.2 (B)
- new net SCLK: Card1.5 (CLK), U1.15 (SCK), U3.34 (GPIO22), U4.4 (A3)
- new net SCLK 2 5V: DS1.6 (E), U4.11 (B3)
- now unconnected: SW1.2, SW3.2, SW4.2, SW5.2
- no-connect marks 50 -> 60
Other:
- moved on the sheet: RV1

Commit message: work, lyra mostly final
Parts:
- added D4: LED, LED_SMD:LED_0805_2012Metric, symbol Device:LED
- added R15: 1k, Resistor_SMD:R_0402_1005Metric, symbol Device:R_Small
Connections:
- net +3.3VA: now also D4.2 (A)
- net LEDINDICATION: now reaches U3.18 (GPIO15)
- net LEDINDICATION: now also R15.1
- new net: D4.1 (K), R15.2
- no-connect marks 60 -> 59

Commit message: reciver rework
Parts:
- removed DS1: ST7920, .pretty:ST7920 AZ, symbol Display_Graphic:ERM19264
- removed RV1: R_Potentiometer, .pretty:RES-ADJ-SMD_3314J, symbol Device:R_Potentiometer
- removed U4: TXB0104RGY, Package_DFN_QFN:Texas_S-PVQFN-N14, symbol Logic_LevelTranslator:TXB0104RGY
- added D?: ER-TFT032A3-3, .pretty:FPC-SMD_40P-P0.50_AMPHENOL_62684-402100ALF, symbol .kicad_sym:ER-TFT032IPS_LCD
Connections:
- net +3.3VA: now also D?.38 (IM0), D?.40 (IM2), D?.6 (IOVCC)
- net GND: now also D?.16 (GND), D?.37 (GND), D?.39 (IM1), D?.5 (GND)
- new net RST: D?.15 (RESET)
- no-connect marks 59 -> 67

Commit message: stuffs
Parts:
- removed C31, C37, C38: 1u, Capacitor_SMD:C_0402_1005Metric, symbol Device:C_Small
- removed Card1: TF-115K, .pretty:TF-SMD_TF-115K, symbol .kicad_sym:TF-115K
- removed J4: Screw_Terminal_01x02, TerminalBlock:TerminalBlock_bornier-2_P5.08mm, symbol Connector:Screw_Terminal_01x02
- removed SW1, SW2, SW3, SW4, SW5: K2-1102DP-L3SW-04, .pretty:SW-TH_4P-L6.0-W6.0-P4.50-LS6.5, symbol .kicad_sym:K2-1102DP-L3SW-04
- removed U9: AMS1117-5.0, Package_TO_SOT_SMD:SOT-223-3_TabPin2, symbol Regulator_Linear:AMS1117-5.0
- added C16: 100n, Capacitor_SMD:C_0402_1005Metric, symbol Device:C_Small
- added C18: 10u, Capacitor_SMD:C_0603_1608Metric, symbol Device:C_Small
- added C19: 2u2, Capacitor_SMD:C_0603_1608Metric, symbol Device:C_Small
- added J6: Conn_01x08, Connector_PinSocket_2.54mm:PinSocket_1x08_P2.54mm_Vertical, symbol Connector_Generic:Conn_01x08
- added J8: AudioJack4, .pretty:AUDIO-SMD_PJ-320D, symbol Connector_Audio:AudioJack4
- added R18, R19: 5.1k, Resistor_SMD:R_0402_1005Metric, symbol Device:R_Small
- added R20: 470, Resistor_SMD:R_0402_1005Metric, symbol Device:R_Small
- D5: renamed from D?; footprint .pretty:FPC-SMD_40P-P0.50_AMPHENOL_62684-402100ALF -> .pretty:R-TFT032IPS-3.2; Vendor https://www.buydisplay.com/3-2-inch-240x320-ips-tft-lcd-dis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 -> https://www.buydisplay.com/3-2-inch-240x320-ips-tft-lcd-mod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
Connections:
- net +3.3VA: now also D5.2 (VDD), D5.29 (BL_ON/OFF), C16.2, C18.2, J6.1 (Pin_1); no longer D5.38 (IM0), D5.40 (IM2), D5.6 (IOVCC)
- net BCK: now also U3.9 (GPIO7); no longer U3.11 (GPIO8)
- net BUTTON1: now also U3.8 (GPIO6), J6.2 (Pin_2); no longer U3.6 (GPIO4)
- net BUTTON2: now also U3.7 (GPIO5), J6.3 (Pin_3); no longer U3.2 (GPIO0)
- net BUTTON3: now also U3.6 (GPIO4), J6.4 (Pin_4); no longer U3.4 (GPIO2)
- net BUTTON4: now also J6.5 (Pin_5)
- net BUTTON5: now also U3.4 (GPIO2), J6.6 (Pin_6); no longer U3.3 (GPIO1)
- net DIN: now also U3.12 (GPIO9); no longer U3.13 (GPIO10)
- net GND: now also D5.1 (GND), D5.40 (GND), C16.1, C18.1, C19.2, J8.R2, R18.2, R19.2; no longer D5.16 (GND), D5.37 (GND), D5.39 (IM1), D5.5 (GND)
- net LCD CS: now also D5.23 (LCD_/CS)
- net LEDINDICATION: now also U3.29 (GPIO18); no longer U3.18 (GPIO15)
- net LRCK: now also U3.13 (GPIO10); no longer U3.14 (GPIO11)
- net MISO: now also D5.28 (LCD_SDO), D5.32 (SDO)
- net MOSI: now also D5.27 (LCD_SDI), D5.34 (SDI)
- net SCK: now also U3.11 (GPIO8); no longer U3.12 (GPIO9)
- net SCLK: now also D5.33 (SCLK)
- net SD_CS: now also D5.35 (SD_/CS)
- net LCD /WR: now reaches U3.37 (GPIO25)
- net LCD /WR: now also D5.25 (/WR(D/C))
- net LCD RST: now reaches D5.21 (RESET)
- net LCD RST: now also U3.14 (GPIO11)
- net LCD D/C: now reaches D5.24 (D/C(SCL))
- net LCD D/C: now also U3.18 (GPIO15)
- net at U5.6 (OUTL): now also R20.1
- net AUDIOOUT renamed AUDIOOUT R
- net AUDIOOUT R: now also J8.R1
- net RST: no longer names the net of D5.15 (DB12)
- new net AUDIOOUT L: C19.1, J8.T, R20.2
- new net BUTTON6: J6.7 (Pin_7), R18.1, U3.3 (GPIO1)
- new net BUTTON7: J6.8 (Pin_8), R19.1, U3.2 (GPIO0)
- no-connect marks 67 -> 51
Other:
- note added: "COM UP DWN LET RHT MID SET RST"
- note removed: "SD CARD"
- moved on the sheet: C34, C35, C36, D2, D3, D5, J5, Q1, R10, R11, R12, R13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

Commit message: post order omcmit
Parts:
- removed J5: Screw_Terminal_01x02, TerminalBlock:TerminalBlock_bornier-2_P5.08mm, symbol Connector:Screw_Terminal_01x02
- removed J6: Conn_01x08, Connector_PinSocket_2.54mm:PinSocket_1x08_P2.54mm_Vertical, symbol Connector_Generic:Conn_01x08
- removed R18, R19: 5.1k, Resistor_SMD:R_0402_1005Metric, symbol Device:R_Small
- added BT1: Battery, SamacSys_Parts:12BH349GR, symbol Device:Battery
- added J10: Conn_01x05, Connector_PinHeader_2.54mm:PinHeader_1x05_P2.54mm_Horizontal, symbol Connector_Generic:Conn_01x05
- added J4, J7: Conn_01x04, Connector_PinHeader_2.54mm:PinHeader_1x04_P2.54mm_Horizontal, symbol Connector_Generic:Conn_01x04
- added SW1, SW2, SW3, SW4, SW5: K2-1102DP-L3SW-04, .pretty:SW-TH_4P-L6.0-W6.0-P4.50-LS6.5, symbol .kicad_sym:K2-1102DP-L3SW-04
- D4: now in the parts list
- D5: now left out of the parts list
- J8: LCSC Part (none) -> C521460
- R16: value 1k -> 15k
Connections:
- net +3.3VA: now also J10.1 (Pin_1), J4.1 (Pin_1), J7.1 (Pin_1), SW1.1, SW2.1, SW3.1, SW4.1, SW5.1
- net BUTTON1: now also U3.7 (GPIO5), SW1.3; no longer U3.8 (GPIO6)
- net BUTTON2: now also U3.5 (GPIO3), SW2.3; no longer U3.7 (GPIO5)
- net BUTTON3: now also SW3.3
- net BUTTON4: now also U3.8 (GPIO6), SW4.3; no longer U3.5 (GPIO3)
- net BUTTON5: now also SW5.3
- net GND: now also BT1.2 (-), J10.5 (Pin_5), J4.4 (Pin_4), J7.4 (Pin_4)
- net MISO: now also J10.3 (Pin_3)
- net MOSI: now also J10.4 (Pin_4)
- net SCL: now also J4.3 (Pin_3)
- net SCLK: now also J10.2 (Pin_2)
- net SDA: now also J4.2 (Pin_2)
- net at D3.1 (K), Q1.3 (D): now also BT1.1 (+)
- net UART0 TX: now reaches U3.27 (GPIO16)
- net UART0 TX: now also J7.3 (Pin_3)
- net UART0 RX: now reaches U3.28 (GPIO17)
- net UART0 RX: now also J7.2 (Pin_2)
- net BUTTON6: no longer names the net of U3.3 (GPIO1)
- net BUTTON7: no longer names the net of U3.2 (GPIO0)
- no-connect marks 51 -> 61
Other:
- note added: "4 cell AA"
- note added: "GPIO"
- note added: "I2C"
- note added: "SPI"
- note added: "UART"
- note removed: "5 cell AA"
- note removed: "COM UP DWN LET RHT MID SET RST"
