File: Hardware/kicad/magswitch/magswitch/magswitch.kicad_pcb (KiCad board)
At the start: 2 copper layers, 11 x 13 mm, 11 parts, among them J1 Conn_01x02, J3 Conn_01x02, Q2 AON7423, U1 SK1816G-AE3-R

Commit message: magswitch work
Parts:
- removed Q2: AON7423, .pretty:DFN-8_L3.0-W3.0-P0.65-BL
- added Q1: AON7508, .pretty:PQFN-8_L3.0-W3.0-P0.65-LS3.2-BL, F.Cu at (108.6, 120.6)
- moved R3 4.80 mm to (106.2, 117.8), turned to -90 degrees
- moved D1 3.47 mm to (108.2, 118.2), turned to 180 degrees
- moved U1 0.13 mm to (102.1, 117.9)
- moved R1 0.06 mm to (104.9, 117.7)
- turned D3 to 180 degrees
Connections:
- J1 pad 1: /SWITCH -> +BATT
- J1 pad 2: GND -> /SWITCH
Routing:
- net /SENSE OUT: track 6.63 -> 10.6 mm, vias 0 -> 2
- net +BATT: track 0.00 -> 3.90 mm
- net GND: track 4.99 -> 3.01 mm
- net Net-(D1-A): track 2.81 -> 1.58 mm
- net /SWITCH: track 0.00 -> 1.10 mm
- added copper zone on B.Cu, net +BATT
- added copper zone on F.Cu, net GND
- removed copper zone on F.Cu, net (none)
- removed copper zone on F.Cu, net +BATT
- removed copper zone on B.Cu, net GND

Commit message: post order omcmit
Parts:
- moved R3 0.48 mm to (106.6, 118.0)
- moved D1 0.43 mm to (108.6, 118.2)
Changed lines of the file:
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@@
 	(footprint "Resistor_SMD:R_0402_1005Metric"
 		(layer "F.Cu")
-		(at 106.172 117.8306 -90)
+		(at 106.6292 117.983 -90)
 		(descr "Resistor SMD 0402 (1005 Metric), square (rectangular) end terminal, IPC_7351 nominal, (Body size source: IPC-SM-782 page 72, https://www.pcb-3d.com/wordpress/wp-content/uploads/ipc-sm-782a_amendment_1_and_2.pdf), generated with kicad-footprint-generator")
 		(tags "resistor")
@@
 	(footprint "LED_SMD:LED_0603_1608Metric"
 		(layer "F.Cu")
-		(at 108.156206 118.235397 180)
+		(at 108.585 118.235397 180)
 		(descr "LED SMD 0603 (1608 Metric), square (rectangular) end terminal, IPC_7351 nominal, (Body size source: http://www.tortai-tech.com/upload/download/2011102023233369053.pdf), generated with kicad-footprint-generator")
 		(tags "LED")
@@
 	)
 	(segment
-		(start 106.172 118.3406)
-		(end 106.172 119.4054)
+		(start 107.1372 119.001)
+		(end 107.1372 119.579)
 		(width 0.5)
 		(layer "F.Cu")
@@
 	)
 	(segment
-		(start 106.172 119.4054)
-		(end 106.1974 119.4308)
+		(start 106.6292 118.493)
+		(end 107.1372 119.001)
 		(width 0.5)
 		(layer "F.Cu")
@@
 	)
 	(via
-		(at 101.3968 116.233)
+		(at 101.2952 115.8494)
 		(size 0.6)
 		(drill 0.3)
@@
 	)
 	(segment
-		(start 102.4128 117.249)
-		(end 101.3968 116.233)
+		(start 102.4128 116.967)
+		(end 102.4128 117.983)
 		(width 0.5)
 		(layer "B.Cu")
@@
 	)
 	(segment
-		(start 102.4128 117.983)
-		(end 102.4128 117.249)
+		(start 101.2952 115.8494)
+		(end 102.4128 116.967)
 		(width 0.5)
 		(layer "B.Cu")
@@
 	)
 	(segment
+		(start 103.4796 119.9256)
+		(end 104.9274 118.4778)
+		(width 0.2)
+		(layer "F.Cu")
+		(net 4)
+	)
+	(segment
+		(start 101.915 118.933)
+		(end 100.976 118.933)
+		(width 0.2)
+		(layer "F.Cu")
+		(net 4)
+	)
+	(segment
 		(start 107.1118 122.047)
 		(end 107.1118 121.5644)
@@
 	)
 	(segment
-		(start 103.4796 119.9256)
-		(end 104.9274 118.4778)
-		(width 0.2)
-		(layer "F.Cu")
-		(net 4)
-	)
-	(segment
 		(start 107.1118 121.5644)
 		(end 107.1372 121.539)
-		(width 0.2)
-		(layer "F.Cu")
-		(net 4)
-	)
-	(segment
-		(start 101.915 118.933)
-		(end 100.976 118.933)
 		(width 0.2)
 		(layer "F.Cu")
@@
 	)
 	(segment
-		(start 106.453908 117.3206)
-		(end 106.172 117.3206)
+		(start 107.035102 117.473)
+		(end 106.6292 117.473)
 		(width 0.5)
 		(layer "F.Cu")
@@
 	)
 	(segment
-		(start 107.368705 118.235397)
-		(end 106.453908 117.3206)
+		(start 107.797499 118.235397)
+		(end 107.035102 117.473)
 		(width 0.5)
 		(layer "F.Cu")
@@
 		(hatch edge 0.5)
 		(priority 3)
+		(connect_pads yes
+			(clearance 0.2)
+		)
+		(min_thickness 0.2)
+		(filled_areas_thickness no)
+		(fill yes
+			(thermal_gap 0.5)
+			(thermal_bridge_width 0.5)
+			(island_removal_mode 1)
+			(island_area_min 10)
+		)
+		(polygon
+			(pts
+				(xy 119.083555 130.742579) (xy 120.607555 107.247579) (xy 92.464355 107.323779) (xy 94.496355 131.580779)
+			)
+		)
+	)
+	(zone
+		(net 1)
+		(net_name "/SWITCH")
+		(layer "F.Cu")
+		(hatch edge 0.5)
+		(priority 5)
 		(connect_pads yes
 			(clearance 0.25)
@@
 		(polygon
 			(pts
-				(xy 119.083555 130.742579) (xy 120.607555 107.247579) (xy 92.464355 107.323779) (xy 94.496355 131.580779)
-			)
-		)
-	)
-	(zone
-		(net 1)
-		(net_name "/SWITCH")
-		(layer "F.Cu")
-		(hatch edge 0.5)
-		(priority 5)
-		(connect_pads yes
-			(clearance 0.25)
-		)
-		(min_thickness 0.25)
-		(filled_areas_thickness no)
-		(fill yes
-			(thermal_gap 0.5)
-			(thermal_bridge_width 0.5)
-			(island_removal_mode 1)
-			(island_area_min 10)
-		)
-		(polygon
-			(pts
-				(xy 107.5182 119.3546) (xy 107.5182 122.428) (xy 108.3818 122.4534) (xy 108.3818 125.0188) (xy 104.9782 125.0188)
-				(xy 104.985246 119.336137)
-			)
-		)
+				(xy 107.5182 119.3546) (xy 107.5182 122.428) (xy 108.3818 122.4534) (xy 108.3818 125.0188) (xy 105.8164 125.0188)
+				(xy 105.823446 119.336137)
+			)
+		)
