File: Hardware/kicad/magswitch/magswitch/magswitch.kicad_sch (KiCad schematic)
At the start: 11 parts, among them J1 Conn_01x02, J3 Conn_01x02, Q2 AON7423, U1 SK1816G-AE3-R

Commit message: magswitch work
Parts:
- removed Q2: AON7423, .pretty:DFN-8_L3.0-W3.0-P0.65-BL, symbol .kicad_sym:AON7423
- added Q1: AON7508, :PQFN-8_L3.0-W3.0-P0.65-LS3.2-BL, symbol .kicad_sym:AON7508
Connections:
- net +BATT: now also J1.1 (Pin_1)
- net GND: now also Q1.5 (D), Q1.6 (D), Q1.7 (D), Q1.8 (D); no longer J1.2 (Pin_2)
- net SENSE OUT: now also Q1.4 (G)
- net SWITCH: now also J1.2 (Pin_2), Q1.1 (S), Q1.2 (S), Q1.3 (S); no longer J1.1 (Pin_1)
Other:
- moved on the sheet: D1, R3

Commit message: post order omcmit
Connections:
- net +BATT: now also R3.2
- net GND: no longer D1.1 (K)
- net SWITCH: now also D1.1 (K); no longer R3.2
Other:
- moved on the sheet: D1, R3
Changed lines of the file:
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@@
+	(wire
+		(pts
+			(xy 110.49 100.33) (xy 110.49 102.87)
+		)
+		(stroke
+			(width 0)
+			(type default)
+		)
+	)
 	(wire
 		(pts
@@
 	(wire
 		(pts
-			(xy 105.41 100.33) (xy 113.03 100.33)
-		)
-		(stroke
-			(width 0)
-			(type default)
-		)
-	)
-	(wire
-		(pts
 			(xy 138.43 77.47) (xy 147.32 77.47)
 		)
@@
 	(wire
 		(pts
-			(xy 97.79 100.33) (xy 100.33 100.33)
+			(xy 95.25 102.87) (xy 97.79 102.87)
 		)
 		(stroke
@@
 	(wire
 		(pts
-			(xy 85.09 100.33) (xy 90.17 100.33)
-		)
-		(stroke
-			(width 0)
-			(type default)
-		)
-	)
-	(wire
-		(pts
-			(xy 85.09 101.6) (xy 85.09 100.33)
-		)
-		(stroke
-			(width 0)
-			(type default)
-		)
-	)
-	(wire
-		(pts
 			(xy 69.85 74.93) (xy 72.39 74.93)
 		)
@@
 		(pts
 			(xy 69.85 74.93) (xy 69.85 77.47)
+		)
+		(stroke
+			(width 0)
+			(type default)
+		)
+	)
+	(wire
+		(pts
+			(xy 74.93 102.87) (xy 87.63 102.87)
+		)
+		(stroke
+			(width 0)
+			(type default)
+		)
+	)
+	(wire
+		(pts
+			(xy 110.49 102.87) (xy 102.87 102.87)
 		)
 		(stroke
@@
 		)
 	)
-	(label "SENSE OUT"
-		(at 53.34 82.55 0)
+	(label "SWITCH"
+		(at 74.93 102.87 0)
 		(fields_autoplaced yes)
 		(effects
@@
 	)
 	(label "SENSE OUT"
-		(at 109.22 82.55 0)
+		(at 53.34 82.55 0)
 		(fields_autoplaced yes)
 		(effects
@@
 		)
 	)
-	(label "SWITCH"
-		(at 113.03 100.33 180)
+	(label "SENSE OUT"
+		(at 109.22 82.55 0)
 		(fields_autoplaced yes)
 		(effects
@@
 				(size 1.27 1.27)
 			)
-			(justify right bottom)
+			(justify left bottom)
 		)
 	)
@@
 	(symbol
 		(lib_id "power:GND")
-		(at 85.09 101.6 0)
-		(unit 1)
-		(exclude_from_sim no)
-		(in_bom yes)
-		(on_board yes)
-		(dnp no)
-		(fields_autoplaced yes)
-		(property "Reference" "#PWR09"
-			(at 85.09 107.95 0)
-			(effects
-				(font
-					(size 1.27 1.27)
-				)
-				(hide yes)
-			)
-		)
-		(property "Value" "GND"
-			(at 85.09 106.68 0)
-			(effects
-				(font
-					(size 1.27 1.27)
-				)
-			)
-		)
-		(property "Footprint" ""
-			(at 85.09 101.6 0)
-			(effects
-				(font
-					(size 1.27 1.27)
-				)
-				(hide yes)
-			)
-		)
-		(property "Datasheet" ""
-			(at 85.09 101.6 0)
-			(effects
-				(font
-					(size 1.27 1.27)
-				)
-				(hide yes)
-			)
-		)
-		(property "Description" "Power symbol creates a global label with name \"GND\" , ground"
-			(at 85.09 101.6 0)
-			(effects
-				(font
-					(size 1.27 1.27)
-				)
-				(hide yes)
-			)
-		)
-		(pin "1"
-		)
-		(instances
-			(project "magswitch"
-				(path "/d949207c-dce7-4463-8f36-829b938688ba"
-					(reference "#PWR09")
-					(unit 1)
-				)
-			)
-		)
-	)
-	(symbol
-		(lib_id "power:GND")
 		(at 152.4 67.31 0)
 		(unit 1)
@@
 	)
 	(symbol
+		(lib_id "power:+BATT")
+		(at 110.49 100.33 0)
+		(unit 1)
+		(exclude_from_sim no)
+		(in_bom yes)
+		(on_board yes)
+		(dnp no)
+		(fields_autoplaced yes)
+		(property "Reference" "#PWR06"
+			(at 110.49 104.14 0)
+			(effects
+				(font
+					(size 1.27 1.27)
+				)
+				(hide yes)
+			)
+		)
+		(property "Value" "+BATT"
+			(at 110.49 95.25 0)
+			(effects
+				(font
+					(size 1.27 1.27)
+				)
+			)
+		)
+		(property "Footprint" ""
+			(at 110.49 100.33 0)
+			(effects
+				(font
+					(size 1.27 1.27)
+				)
+				(hide yes)
+			)
+		)
+		(property "Datasheet" ""
+			(at 110.49 100.33 0)
+			(effects
+				(font
+					(size 1.27 1.27)
+				)
+				(hide yes)
+			)
+		)
+		(property "Description" "Power symbol creates a global label with name \"+BATT\""
+			(at 110.49 100.33 0)
+			(effects
+				(font
+					(size 1.27 1.27)
+				)
+				(hide yes)
+			)
+		)
+		(pin "1"
+		)
+		(instances
+			(project "magswitch"
+				(path "/d949207c-dce7-4463-8f36-829b938688ba"
+					(reference "#PWR06")
+					(unit 1)
+				)
+			)
+		)
+	)
+	(symbol
 		(lib_id "Device:C_Small")
 		(at 152.4 63.5 0)
@@
 	(symbol
 		(lib_id "Device:R_Small")
-		(at 102.87 100.33 90)
+		(at 100.33 102.87 90)
 		(unit 1)
 		(exclude_from_sim no)
@@
 		(fields_autoplaced yes)
 		(property "Reference" "R3"
-			(at 102.87 95.25 90)
+			(at 100.33 97.79 90)
 			(effects
 				(font
@@
 		)
 		(property "Value" "10k"
-			(at 102.87 97.79 90)
+			(at 100.33 100.33 90)
 			(effects
 				(font
@@
 		)
 		(property "Footprint" "Resistor_SMD:R_0402_1005Metric"
-			(at 102.87 100.33 0)
+			(at 100.33 102.87 0)
 			(effects
 				(font
@@
 		)
 		(property "Datasheet" "~"
-			(at 102.87 100.33 0)
+			(at 100.33 102.87 0)
 			(effects
 				(font
@@
 		)
 		(property "Description" "Resistor, small symbol"
-			(at 102.87 100.33 0)
+			(at 100.33 102.87 0)
 			(effects
 				(font
@@
 		)
 		(property "LCSC Part" "C25744"
-			(at 102.87 100.33 0)
+			(at 100.33 102.87 0)
 			(effects
 				(font
@@
 	(symbol
 		(lib_id "Device:LED")
-		(at 93.98 100.33 0)
+		(at 91.44 102.87 0)
 		(unit 1)
 		(exclude_from_sim no)
@@
 		(fields_autoplaced yes)
 		(property "Reference" "D1"
-			(at 92.3925 93.98 0)
+			(at 89.8525 96.52 0)
 			(effects
 				(font
@@
 		)
 		(property "Value" "LED"
-			(at 92.3925 96.52 0)
+			(at 89.8525 99.06 0)
 			(effects
 				(font
@@
 		)
 		(property "Footprint" "LED_SMD:LED_0603_1608Metric"
-			(at 93.98 100.33 0)
+			(at 91.44 102.87 0)
 			(effects
 				(font
@@
 		)
 		(property "Datasheet" "~"
-			(at 93.98 100.33 0)
+			(at 91.44 102.87 0)
 			(effects
 				(font
@@
 		)
 		(property "Description" "Light emitting diode"
-			(at 93.98 100.33 0)
+			(at 91.44 102.87 0)
 			(effects
 				(font
@@
 		)
 		(property "LCSC Part" "C72041"
-			(at 93.98 100.33 0)
-			(effects
-				(font
+			(at 91.44 102.87 0)
+			(effects
+				(font
