File: Hardware/kicad/Lyra_flight_computer/lyrav3r1/lyrav3r2/_autosave-lyrav3r2.kicad_pcb (KiCad board)
At the start: 4 copper layers, 22 x 52 mm, 110 parts, among them IC1 TESEO-LIV3F, J1 Conn_01x02, J2 Screw_Terminal_01x04, J4 Conn_01x02, J5 Conn_01x05, J6 Screw_Terminal_01x05, J7 USB_B_Micro, Q1 AO3401A, Q2 AO3400A, Q4 AO3400A, Q5 AO3400A, Q6 AO3401A, Q9 AO3400A, U1 E22-900MM22S, U2 BMI088, U3 BMP388, U4 LIS3MDLTR, U5 ADXL375BCCZ-RL7, U6 RT9013-33GB_C19268157, U7 WS7916S-6/TR, U8 RP2040, U9 W25Q128JVS, X2 SX1M12.000M10F30TNN

Commit message: woprk
Parts:
- moved U4 35.3 mm to (201.7, 88.7)
- moved C12 1.46 mm to (206.1, 92.2)
- moved C4 1.46 mm to (205.3, 93.9)
- moved U3 1.46 mm to (204.4, 92.2)
Changed lines of the file:
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@@
 	(footprint "Capacitor_SMD:C_0402_1005Metric"
 		(layer "B.Cu")
-		(at 205.5836 90.8748 90)
+		(at 206.121 92.2274 90)
 		(descr "Capacitor SMD 0402 (1005 Metric), square (rectangular) end terminal, IPC_7351 nominal, (Body size source: IPC-SM-782 page 76, https://www.pcb-3d.com/wordpress/wp-content/uploads/ipc-sm-782a_amendment_1_and_2.pdf), generated with kicad-footprint-generator")
 		(tags "capacitor")
@@
 	(footprint "easyeda2kicad:SENSORM-SMD_BMP388"
 		(layer "B.Cu")
-		(at 203.8564 90.824)
+		(at 204.3938 92.1766)
 		(property "Reference" "U3"
 			(at 0 4.87 0)
@@
 	(footprint "Capacitor_SMD:C_0402_1005Metric"
 		(layer "B.Cu")
-		(at 204.748 92.5004)
+		(at 205.2854 93.853)
 		(descr "Capacitor SMD 0402 (1005 Metric), square (rectangular) end terminal, IPC_7351 nominal, (Body size source: IPC-SM-782 page 76, https://www.pcb-3d.com/wordpress/wp-content/uploads/ipc-sm-782a_amendment_1_and_2.pdf), generated with kicad-footprint-generator")
 		(tags "capacitor")
@@
 	(footprint ".pretty:LGA-12_L2.0-W2.0-P0.50-BL"
 		(layer "B.Cu")
-		(at 236.319 81.8986 180)
+		(at 201.667 88.65 180)
 		(property "Reference" "U4"
 			(at 0 4.88 180)
