File: Hardware/kicad/Lyra_flight_computer/lyrav3r1/lyrav3r2/lyrav3r2.kicad_pcb (KiCad board)
At the start: 4 copper layers, 22 x 53 mm, 111 parts, among them IC1 TESEO-LIV3F, J1 Conn_01x02, J2 Screw_Terminal_01x04, J4 Conn_01x02, J5 Conn_01x05, J6 Screw_Terminal_01x05, J7 USB_B_Micro, Q1 AO3401A, Q2 AO3400A, Q3 AO3401A, Q4 AO3400A, Q5 AO3400A, Q9 AO3400A, U1 E22-900MM22S, U10 MXDLN16TL, U2 BMI088, U3 BMP388, U4 LIS3MDLTR, U5 ADXL375BCCZ-RL7, U6 RT9013-33GB_C19268157, U8 RP2040, U9 W25Q128JVS, X2 SX1M12.000M10F30TNN

Commit message: fabbed
Parts:
- removed R5, R6, R7, R8: 10, Resistor_SMD:R_0402_1005Metric
- moved G*** 21.4 mm to (186.9, 97.9), turned to 180 degrees
- moved C3 0.35 mm to (194.9, 109.0)
Connections:
- Q2 pad 3: Net-(Q2-D) -> /P2-
- Q4 pad 3: Net-(Q4-D) -> /P1-
- Q5 pad 3: Net-(Q5-D) -> /P3-
- Q9 pad 3: Net-(Q9-D) -> /P4-
- R20 pad 1: Net-(Q5-D) -> /P3-
- R22 pad 1: Net-(Q9-D) -> /P4-
- R24 pad 1: Net-(Q2-D) -> /P2-
- R26 pad 1: Net-(Q4-D) -> /P1-
Routing:
- net Net-(Q5-D): track 5.81 -> 0.00 mm
- net /P3-: track 2.36 -> 7.69 mm
- net Net-(Q2-D): track 5.01 -> 0.00 mm
- net /P2-: track 2.06 -> 7.04 mm
- net Net-(Q4-D): track 3.05 -> 0.00 mm
- net /P1-: track 2.08 -> 5.05 mm
- net Net-(Q9-D): track 2.86 -> 0.00 mm
- net /P4-: track 2.15 -> 4.82 mm
- net /BATT SENSE : track 16.9 -> 17.6 mm
- added copper zone on B.Cu, net (none)
- added copper zone on F.Cu, net (none)
Other:
- board text added: "3"
- board text added: "4"
- board text added: "5"
- board text added: "6"
- board text added: "7"
- board text added: "8"
- board text added: "9"
- board text added: "OOPS! NO DATA!"
- board text added: "SW- + + -B"
- board text added: "THX BB123 DKNIGHT, DELTACLIPPER ELVIN, MATT,VULPES, ULYU, SANDVOXEL"
- board text added: "The rocket knows where it is at all times. It knows this because it knows where it isn't,by subtracting where it is, from where it isn't, from where it is, whichever is"
- board text removed: "SW- + + - B"
- board text removed: "THX BB123, MATT, ELVIN, DKNIGHT, VULPES, ULYU"
- board text removed: "U R COOL"
