File: Hardware/kicad/Lyra_flight_computer/lyrav3r1/lyrav3r2/lyrav3r2.kicad_sch (KiCad schematic)
At the start: 109 parts, among them IC1 TESEO-LIV3F, J1 Conn_01x02, J2 Screw_Terminal_01x04, J4 Conn_01x02, J5 Conn_01x05, J6 Screw_Terminal_01x05, J7 USB_B_Micro, Q1 AO3401A, Q2 AO3400A, Q3 AO3401A, Q4 AO3400A, Q5 AO3400A, Q9 AO3400A, U1 E22-900MM22S, U10 MXDLN16TL, U2 BMI088, U3 BMP388, U4 LIS3MDLTR, U5 ADXL375BCCZ-RL7, U6 RT9013-33GB_C19268157, U8 RP2040, U9 W25Q128JVS, X2 SX1M12.000M10F30TNN

Commit message: fabbed
Parts:
- removed R5, R6, R7, R8: 10, Resistor_SMD:R_0402_1005Metric, symbol Device:R_Small
- R21, R23, R25, R27, R4: value 50k -> 51k
Connections:
- net P1-: now also Q4.3 (D), R26.1
- net P2-: now also Q2.3 (D), R24.1
- net P3-: now also Q5.3 (D), R20.1
- net P4-: now also Q9.3 (D), R22.1
