File: Hope/Hope/Hope.kicad_pcb (KiCad board)
At the start: 4 copper layers, 17 x 33 mm, 43 parts, among them J1 USB_B_Micro, J2 Conn_01x02, J3 Conn_01x02, J4 Screw_Terminal_01x02, J7 Conn_01x04, Q1 AO3401A, Q2 AO3401A, U1 W25Q128JVS, U2 RP2040, U3 XC6206P332MR, X1 SX1M12.000M10F30TNN

Commit message: ping pong sent for fab
Routing:
- net GND: track 48.6 -> 43.7 mm
- net /MCU/DIO3: track 12.3 -> 13.4 mm
- net /MCU/DIO2: track 13.5 -> 14.6 mm
- net /MCU/QSPI_SCLK: track 13.2 -> 12.6 mm
- net +3V3: track 33.7 -> 33.3 mm, vias 14 -> 15
Other:
- board text added: "BOOT"
- board text added: "CLK"
- board text added: "RUN"
