File: Hope/Hope/MCU.kicad_sch (KiCad schematic)
At the start: 27 parts, among them J1 USB_B_Micro, J2 Conn_01x02, J3 Conn_01x02, U1 W25Q128JVS, U2 RP2040, X1 SX1M12.000M10F30TNN

Commit message: pingpong
Parts:
- removed H1, H2: MountingHole_Pad, MountingHole:MountingHole_3.2mm_M3_DIN965_Pad, symbol Mechanical:MountingHole_Pad
- added C16: 100n, Capacitor_SMD:C_0402_1005Metric, symbol Device:C_Small
- added H3, H4: MountingHole_Pad, MountingHole:MountingHole_2.2mm_M2_DIN965_Pad, symbol Mechanical:MountingHole_Pad
- added J7: Conn_01x04, .pretty:4 pads 2.54mm spacign, symbol Connector_Generic:Conn_01x04
- added R8: 30k, Resistor_SMD:R_0402_1005Metric, symbol Device:R_Small
- added R9: 51k, Resistor_SMD:R_0402_1005Metric, symbol Device:R_Small
Connections:
- net +3V3: now also J7.1 (Pin_1)
- net BUSY: now also U2.13 (GPIO10); no longer U2.32 (GPIO21)
- net DIO1: now also U2.12 (GPIO9); no longer U2.31 (GPIO20)
- net DIO2: now also U2.3 (GPIO1); no longer U2.30 (GPIO19)
- net DIO3: now also U2.2 (GPIO0); no longer U2.29 (GPIO18)
- net GND: now also U2.57 (GND), C16.2, H3.1, H4.1, J7.4 (Pin_4), R9.2
- net MISO: now also U2.40 (GPIO28_ADC2); no longer U2.15 (GPIO12)
- net MOSI: now also U2.39 (GPIO27_ADC1); no longer U2.14 (GPIO11)
- net NSS: now also U2.37 (GPIO25); no longer U2.12 (GPIO9)
- net SCK: now also U2.38 (GPIO26_ADC0); no longer U2.13 (GPIO10)
- net TXCOEN: now also U2.14 (GPIO11); no longer U2.5 (GPIO3)
- net GPS_RX: now reaches U2.16 (GPIO13)
- net GPS_RX: now also J7.2 (Pin_2)
- net BATT SENSE : now reaches U2.41 (GPIO29_ADC3)
- net BATT SENSE : now also C16.1, R8.2, R9.1
- new net +BATT: R8.1
- new net GPS_TX: J7.3 (Pin_3), U2.15 (GPIO12)
- no-connect marks 3 -> 19
