File: Hope/Hope/Power.kicad_sch (KiCad schematic)
At the start: 10 parts, among them J4 Screw_Terminal_01x02, Q1 AO3401A, Q2 AO3401A, U3 RT9013-33GB_C19268157

Commit message: pingpong
Parts:
- removed U3: RT9013-33GB_C19268157, .pretty:SOT-23-5_L2.9-W1.6-P0.95-LS2.8-BR, symbol .kicad_sym:RT9013-33GB_C19268157
- added U3: XC6206P332MR, :SOT-23-3_L2.9-W1.6-P1.90-LS2.8-BR, symbol .kicad_sym:XC6206P332MR
Connections:
- net +3V3: now also U3.3 (Vout)
- net +BATT: now also U3.2 (Vin)
- net GND: now also U3.1 (GND)
- no-connect marks 1 -> 0
Changed lines of the file:
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@@
 	)
 	(junction
-		(at 135.89 64.77)
+		(at 132.08 64.77)
+		(diameter 0)
+		(color 0 0 0 0)
+	)
+	(junction
+		(at 149.86 78.74)
+		(diameter 0)
+		(color 0 0 0 0)
+	)
+	(junction
+		(at 133.985 97.155)
 		(diameter 0)
 		(color 0 0 0 0)
@@
 		(color 0 0 0 0)
 	)
-	(junction
-		(at 132.08 64.77)
-		(diameter 0)
-		(color 0 0 0 0)
-	)
-	(junction
-		(at 149.86 78.74)
-		(diameter 0)
-		(color 0 0 0 0)
-	)
-	(junction
-		(at 133.985 97.155)
-		(diameter 0)
-		(color 0 0 0 0)
-	)
-	(no_connect
-		(at 160.02 71.12)
-	)
 	(wire
 		(pts
@@
 	(wire
 		(pts
-			(xy 139.7 68.58) (xy 135.89 68.58)
-		)
-		(stroke
-			(width 0)
-			(type default)
-		)
-	)
-	(wire
-		(pts
 			(xy 107.315 55.88) (xy 93.98 55.88)
 		)
@@
 	(wire
 		(pts
+			(xy 132.08 64.77) (xy 137.16 64.77)
+		)
+		(stroke
+			(width 0)
+			(type default)
+		)
+	)
+	(wire
+		(pts
 			(xy 171.45 102.235) (xy 171.45 102.87)
 		)
@@
 	(wire
 		(pts
+			(xy 149.86 77.47) (xy 149.86 78.74)
+		)
+		(stroke
+			(width 0)
+			(type default)
+		)
+	)
+	(wire
+		(pts
 			(xy 97.79 92.075) (xy 97.79 90.17)
 		)
@@
 	(wire
 		(pts
-			(xy 135.89 64.77) (xy 139.7 64.77)
-		)
-		(stroke
-			(width 0)
-			(type default)
-		)
-	)
-	(wire
-		(pts
 			(xy 149.86 78.74) (xy 166.37 78.74)
 		)
@@
 	(wire
 		(pts
-			(xy 149.86 74.93) (xy 149.86 78.74)
-		)
-		(stroke
-			(width 0)
-			(type default)
-		)
-	)
-	(wire
-		(pts
 			(xy 83.82 156.21) (xy 83.82 151.13)
 		)
@@
 	(wire
 		(pts
+			(xy 162.56 64.77) (xy 166.37 64.77)
+		)
+		(stroke
+			(width 0)
+			(type default)
+		)
+	)
+	(wire
+		(pts
 			(xy 133.985 97.155) (xy 154.94 97.155)
 		)
@@
 	(wire
 		(pts
-			(xy 135.89 68.58) (xy 135.89 64.77)
-		)
-		(stroke
-			(width 0)
-			(type default)
-		)
-	)
-	(wire
-		(pts
 			(xy 127 87.63) (xy 133.985 87.63)
 		)
@@
 		(pts
 			(xy 132.08 73.66) (xy 132.08 78.74)
-		)
-		(stroke
-			(width 0)
-			(type default)
-		)
-	)
-	(wire
-		(pts
-			(xy 160.02 64.77) (xy 166.37 64.77)
-		)
-		(stroke
-			(width 0)
-			(type default)
-		)
-	)
-	(wire
-		(pts
-			(xy 132.08 64.77) (xy 135.89 64.77)
 		)
 		(stroke
@@
 	)
 	(symbol
+		(lib_id ".kicad_sym:XC6206P332MR")
+		(at 149.86 64.77 0)
+		(unit 1)
+		(exclude_from_sim no)
+		(in_bom yes)
+		(on_board yes)
+		(dnp no)
+		(fields_autoplaced yes)
+		(property "Reference" "U3"
+			(at 149.86 52.07 0)
+			(effects
+				(font
+					(size 1.27 1.27)
+				)
+			)
+		)
+		(property "Value" "XC6206P332MR"
+			(at 149.86 54.61 0)
+			(effects
+				(font
+					(size 1.27 1.27)
+				)
+			)
+		)
+		(property "Footprint" ":SOT-23-3_L2.9-W1.6-P1.90-LS2.8-BR"
+			(at 149.86 77.47 0)
+			(effects
+				(font
+					(size 1.27 1.27)
+				)
+				(hide yes)
+			)
+		)
+		(property "Datasheet" "https://lcsc.com/product-detail/Low-Dropout-Regulators-LDO_XC6206P332MR_C5446.html"
+			(at 149.86 80.01 0)
+			(effects
+				(font
+					(size 1.27 1.27)
+				)
+				(hide yes)
+			)
+		)
+		(property "Description" ""
+			(at 149.86 64.77 0)
+			(effects
+				(font
+					(size 1.27 1.27)
+				)
+				(hide yes)
+			)
+		)
+		(property "LCSC Part" "C5446"
+			(at 149.86 82.55 0)
+			(effects
+				(font
+					(size 1.27 1.27)
+				)
+				(hide yes)
+			)
+		)
+		(pin "3"
+		)
+		(pin "1"
+		)
+		(pin "2"
+		)
+		(instances
+			(project "Hope"
+				(path "/65404340-e293-4950-8719-8361f004e3c5/19f176ab-7e4d-4626-a178-223fbbd26938"
+					(reference "U3")
+					(unit 1)
+				)
+			)
+		)
+	)
+	(symbol
 		(lib_id "Device:D_Schottky")
 		(at 133.985 92.075 90)
@@
 					(unit 1)
 				)
-			)
-		)
-	)
-	(symbol
-		(lib_id ".kicad_sym:RT9013-33GB_C19268157")
-		(at 149.86 67.31 0)
-		(unit 1)
-		(exclude_from_sim no)
-		(in_bom yes)
-		(on_board yes)
-		(dnp no)
-		(fields_autoplaced yes)
-		(property "Reference" "U3"
-			(at 149.86 57.15 0)
-			(effects
-				(font
-					(size 1.27 1.27)
-				)
-			)
-		)
-		(property "Value" "RT9013-33GB_C19268157"
-			(at 149.86 59.69 0)
-			(effects
-				(font
-					(size 1.27 1.27)
-				)
-			)
-		)
-		(property "Footprint" ".pretty:SOT-23-5_L2.9-W1.6-P0.95-LS2.8-BR"
-			(at 149.86 77.47 0)
-			(effects
-				(font
-					(size 1.27 1.27)
-				)
-				(hide yes)
-			)
-		)
-		(property "Datasheet" ""
-			(at 149.86 67.31 0)
-			(effects
-				(font
-					(size 1.27 1.27)
-				)
-				(hide yes)
-			)
-		)
-		(property "Description" ""
-			(at 149.86 67.31 0)
-			(effects
-				(font
-					(size 1.27 1.27)
-				)
-				(hide yes)
-			)
-		)
-		(property "LCSC Part" "C19268157"
-			(at 149.86 80.01 0)
-			(effects
-				(font
-					(size 1.27 1.27)
-				)
-				(hide yes)
-			)
-		)
-		(pin "5"
-		)
-		(pin "1"
-		)
-		(pin "2"
-		)
-		(pin "4"
-		)
-		(pin "3"
-		)
-		(instances
-			(project "Hope"
-				(path "/65404340-e293-4950-8719-8361f004e3c5/19f176ab-7e4d-4626-a178-223fbbd26938"
-					(reference "U3")
-					(unit 1)
-				)
