File: it sure is getting hot in here/it sure is getting hot in here/it sure is getting hot in here.kicad_pcb (KiCad board)
At the start: 4 copper layers, 11.5 x 43 mm, 43 parts, among them J1 Screw_Terminal_01x02, J2 Screw_Terminal_01x02, J5 Conn_01x02, J6 Conn_01x02, Q2 AO3401A, U1 MAX31865xTP, U2 XC6206P332MR, U3 MAX31865xTP, U5 W25Q128JVS, U6 RP2040, X1 SX1M12.000M10F30TNN

Commit message: update
Parts:
- moved Q2 0.12 mm to (136.8, 104.4), turned to 90 degrees
- renumbered U3 to U1, U1 to U3
Routing:
- net /LEDINDICATION: track 3.80 -> 27.2 mm
- net +3V3: track 30.2 -> 27.7 mm
- net /SCLK: track 24.2 -> 22.2 mm
- net GND: track 45.7 -> 47.4 mm, vias 25 -> 27
- net /MOSI: track 21.1 -> 20.3 mm

Commit message: it sure is getting hot in here software
Parts:
- added C5: 100n, Capacitor_SMD:C_0603_1608Metric_Pad1.08x0.95mm_HandSolder, B.Cu at (139.9, 101.4)
- added C6: 100n, Capacitor_SMD:C_0603_1608Metric_Pad1.08x0.95mm_HandSolder, B.Cu at (143.2, 106.2)
- added R11: 5.1k, Resistor_SMD:R_0402_1005Metric, F.Cu at (145.0, 96.0)
- added R12: 5.1k, Resistor_SMD:R_0402_1005Metric, F.Cu at (144.1, 96.0)
- added U4: BMI088, easyeda2kicad:LGA-16_L4.5-W3.0-P0.50-BL, B.Cu at (140.6, 104.8)
- moved C17 0.22 mm to (144.5, 94.1)
- moved C7 0.08 mm to (137.7, 81.0)
Connections:
- U6 pad 2: unconnected-(U6-GPIO0-Pad2) -> /SDA
- U6 pad 3: unconnected-(U6-GPIO1-Pad3) -> /SCL
Routing:
- net /SDA: track 0.00 -> 44.8 mm, vias 0 -> 3
- net /SCL: track 0.00 -> 30.9 mm, vias 0 -> 2
- net +3V3: track 27.7 -> 41.6 mm, vias 16 -> 19
- net GND: track 47.4 -> 59.1 mm, vias 27 -> 30
- net /LEDINDICATION: track 27.2 -> 24.4 mm
- net /USB_D-: track 17.7 -> 18.7 mm
- net /QSPI_SD1: track 9.05 -> 8.26 mm
- removed copper zone on B.Cu, net GND
- removed copper zone on F.Cu, net GND
Other:
- board text added: "BOOT"
- board text added: "JLCJLCJLCJLC"
- board text added: "SWD"
- board text added: "for internal use only warranty void if used externally"
- board text added: "it sure is getting hot in here! designed by polaris V1.0"
- board text added: "oops wha hap"
- board text added: "thx ulyu"
