File: it sure is getting hot in here/it sure is getting hot in here/it sure is getting hot in here.kicad_sch (KiCad schematic)
At the start: 43 parts, among them J1 Screw_Terminal_01x02, J2 Screw_Terminal_01x02, J5 Conn_01x02, J6 Conn_01x02, Q2 AO3401A, U1 MAX31865xTP, U2 XC6206P332MR, U3 MAX31865xTP, U5 W25Q128JVS, U6 RP2040, X1 SX1M12.000M10F30TNN

Commit message: update
Parts:
- renumbered U3 to U1, U1 to U3
Changed lines of the file:
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@@
 		(dnp no)
 		(fields_autoplaced yes)
-		(property "Reference" "U1"
-			(at 338.1091 52.705 0)
+		(property "Reference" "U3"
+			(at 338.1091 53.34 0)
 			(effects
 				(font
@@
 		)
 		(property "Value" "MAX31865xTP"
-			(at 338.1091 55.245 0)
+			(at 338.1091 55.88 0)
 			(effects
 				(font
@@
 			(project "it sure is getting hot in here"
 				(path "/3bd0164c-2575-48ce-96af-9cdaca468833"
-					(reference "U1")
+					(reference "U3")
 					(unit 1)
 				)
@@
 		(dnp no)
 		(fields_autoplaced yes)
-		(property "Reference" "U3"
+		(property "Reference" "U1"
 			(at 338.7441 114.3 0)
 			(effects
@@
 			(project "it sure is getting hot in here"
 				(path "/3bd0164c-2575-48ce-96af-9cdaca468833"
-					(reference "U3")
-					(unit 1)
-				)
+					(reference "U1")
+					(unit 1)
+				)

Commit message: it sure is getting hot in here software
Parts:
- added C5, C6: 100n, Capacitor_SMD:C_0603_1608Metric_Pad1.08x0.95mm_HandSolder, symbol Device:C_Small
- added R11, R12: 5.1k, Resistor_SMD:R_0402_1005Metric, symbol Device:R_Small
- added U4: BMI088, easyeda2kicad:LGA-16_L4.5-W3.0-P0.50-BL, symbol BMI088:BMI088
- D1, D3: now in the parts list
Connections:
- net +3V3: now also C5.1, C6.1, R11.1, R12.1, U4.11 (VDDIO), U4.14 (CSB1), U4.3 (VDD), U4.7 (PS)
- net GND: now also C5.2, C6.2, U4.10 (SDO2), U4.15 (SDO1), U4.4 (GNDA), U4.6 (GNDIO)
- net SDA: now reaches U6.2 (GPIO0)
- net SDA: now also R11.2, U4.9 (SDA/SDI)
- net SCL: now reaches U6.3 (GPIO1)
- net SCL: now also R12.2, U4.8 (SCL/SCK)
- no-connect marks 22 -> 26
Other:
- note added: "IMU"
- note added: "POWER & CONNECTOR"
- note added: "RTD reader circuits"
- moved on the sheet: C10, C12, C13, C14, C15, C16, C17, C18, C19, C20, C21, C22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
