File: it sure is getting hot in here/it sure is getting hot in here/it sure is getting hot in here.kicad_sch (KiCad schematic)
At the start: 48 parts, among them J1 Screw_Terminal_01x02, J2 Screw_Terminal_01x02, J5 Conn_01x02, J6 Conn_01x02, Q2 AO3401A, U1 MAX31865xTP, U2 XC6206P332MR, U3 MAX31865xTP, U4 BMI088, U5 W25Q128JVS, U6 RP2040, X1 SX1M12.000M10F30TNN

Commit message: cam control
Changed lines of the file:
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@@
 	(rectangle
 		(start 253.365 179.07)
-		(end 408.305 253.365)
+		(end 407.67 253.365)
 		(stroke
 			(width 0)
@@
 	)
 	(rectangle
-		(start 283.21 13.335)
-		(end 407.67 166.37)
+		(start 283.845 12.065)
+		(end 407.035 165.735)
 		(stroke
 			(width 0)
@@
 	)
 	(rectangle
-		(start 12.7 84.455)
-		(end 208.915 284.48)
+		(start 12.065 84.455)
+		(end 208.915 285.115)
 		(stroke
 			(width 0)
