File: it sure is getting hot in here/it sure is getting ROUND in here/it sure is getting ROUND in here.kicad_sch (KiCad schematic)
At the start: 48 parts, among them J1 Screw_Terminal_01x02, J2 Screw_Terminal_01x02, J5 Conn_01x02, J6 Conn_01x02, Q2 AO3401A, U1 MAX31865xTP, U2 XC6206P332MR, U3 MAX31865xTP, U4 BMI088, U5 W25Q128JVS, U6 RP2040, X1 SX1M12.000M10F30TNN

Commit message: weorjk
Parts:
- removed C4, C9: 100n, Capacitor_SMD:C_0402_1005Metric, symbol Device:C_Small
- added C11: 100n, Capacitor_SMD:C_0402_1005Metric, symbol Device:C_Small
- added H?: MountingHole, symbol Mechanical:MountingHole
- J1, J2: footprint Connector_PinHeader_2.54mm:PinHeader_1x02_P2.54mm_Vertical -> Jumper:SolderJumper-2_P1.3mm_Open_Pad1.0x1.5mm
Connections:
- net +3V3: now also C11.1
- net GND: now also C11.2
