File: CamControl/universal ground station/universal ground station.kicad_sch (KiCad schematic)
At the start: 4 parts, among them U1 Pico, U2 E22-400MM22S

Commit message: cam control rework
Changed lines of the file:
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@@
 	(symbol
 		(lib_id ".kicad_sym:E22-400MM22S")
-		(at 161.29 71.12 0)
+		(at 176.53 52.705 0)
 		(unit 1)
 		(exclude_from_sim no)
@@
 		(fields_autoplaced yes)
 		(property "Reference" "U2"
-			(at 161.544 37.846 0)
+			(at 176.784 19.431 0)
 			(effects
 				(font
@@
 		)
 		(property "Value" "E22-400MM22S"
-			(at 160.528 41.148 0)
+			(at 175.768 22.733 0)
 			(effects
 				(font
@@
 		)
 		(property "Footprint" ":WIRELM-SMD_E22-400MM22S"
-			(at 160.528 43.688 0)
+			(at 175.768 25.273 0)
 			(effects
 				(font
@@
 		)
 		(property "Datasheet" ""
-			(at 161.29 71.12 0)
+			(at 176.53 52.705 0)
 			(effects
 				(font
@@
 		)
 		(property "Description" ""
-			(at 161.29 71.12 0)
+			(at 176.53 52.705 0)
 			(effects
 				(font
@@
 		)
 		(property "LCSC Part" "C5333984"
-			(at 160.528 46.228 0)
+			(at 175.768 27.813 0)
 			(effects
 				(font
