File: CamControl/camcontrol stm32/camcontrol stm32.kicad_pcb (KiCad board)
At the start: 4 copper layers, 25.4 x 25.4 mm, 38 parts, among them J1 Power 1, J2 USB_B_Micro, J3 Power 1, J4 Power 1, J5 Power 1, J6 Conn_01x02, J7 Power 1, Q1 AO3401A, Q3 AO3401A, U1 BGS12WN6E6327, U2 BALFHB-WL-02D3, U3 STM32WLE4CCUx, U4 XC6206P332MR, U5 TPS25970LRPWR, U6 TPS25970LRPWR

Commit message: work
Parts:
- removed C15: 100n, Capacitor_SMD:C_0402_1005Metric
- removed J2: USB_B_Micro, easyeda2kicad2:MICRO-USB-SMD_U254-051T-4BHJ25-F2S
- added AE1: Antenna_Shield, .pretty:ANT-SMD_1909763-1, F.Cu at (165.1, 122.2)
- added C17: 100n, Capacitor_SMD:C_0402_1005Metric, F.Cu at (166.5, 124.3)
- added C18: 470n, Capacitor_SMD:C_0402_1005Metric, F.Cu at (167.7, 138.6)
- added D2: LED, LED_SMD:LED_0603_1608Metric, B.Cu at (167.5, 138.5)
- added H1: MountingHole_Pad, MountingHole:MountingHole_2.2mm_M2_DIN965_Pad, F.Cu at (172.1, 143.0)
- added H2: MountingHole_Pad, MountingHole:MountingHole_2.2mm_M2_DIN965_Pad, F.Cu at (161.3, 122.0)
- added J8: DNP, Connector_PinHeader_2.54mm:PinHeader_1x05_P2.54mm_Vertical, B.Cu at (161.3, 143.0)
- added R23: 15k, Resistor_SMD:R_0402_1005Metric, F.Cu at (172.3, 130.5)
- added R24: 51k, Resistor_SMD:R_0402_1005Metric, F.Cu at (173.3, 130.5)
- added R3: 20m, Resistor_SMD:R_0402_1005Metric, F.Cu at (171.2, 125.1)
- added R4: 33k, Resistor_SMD:R_0402_1005Metric, F.Cu at (166.7, 129.0)
- added R5: 20m, Resistor_SMD:R_0402_1005Metric, F.Cu at (160.8, 139.6)
- added R7: 1k, Resistor_SMD:R_0402_1005Metric, F.Cu at (159.7, 128.9)
- added R8: 15k, Resistor_SMD:R_0402_1005Metric, F.Cu at (173.0, 139.8)
- added R9: 51k, Resistor_SMD:R_0402_1005Metric, F.Cu at (174.0, 139.8)
- added U7: INA2180, Package_SON:WSON-8-1EP_2x2mm_P0.5mm_EP0.9x1.6mm, F.Cu at (172.2, 133.4)
- added Y1: 32MHz, Crystal:Crystal_SMD_2016-4Pin_2.0x1.6mm, F.Cu at (160.3, 131.7)
- C2, C3: footprint Capacitor_SMD:C_0402_1005Metric -> Capacitor_SMD:C_0201_0603Metric
- J1, J3, J4, J7: footprint Connector_Molex:Molex_PicoBlade_53048-0210_1x02_P1.25mm_Horizontal -> Connector_Molex:Molex_PicoBlade_53261-0271_1x02-1MP_P1.25mm_Horizontal
- J5: value Power 1 -> Conn_01x06; footprint Connector_Molex:Molex_PicoBlade_53048-0210_1x02_P1.25mm_Horizontal -> Connector_PinHeader_1.27mm:PinHeader_1x06_P1.27mm_Vertical; moved to B.Cu
- J6: moved to B.Cu
- L1: footprint Inductor_SMD:L_0201_0603Metric -> Inductor_SMD:L_0402_1005Metric
- moved C22 69.5 mm to (161.4, 129.7), turned to 180 degrees
- moved J6 68.5 mm to (166.3, 134.4), turned to 90 degrees
- moved C11 67.3 mm to (161.0, 134.1), turned to -90 degrees
- moved C8 67.3 mm to (162.8, 138.3), turned to 180 degrees
- moved C9 64.5 mm to (165.3, 138.8), turned to -90 degrees
- moved C7 64.4 mm to (160.7, 128.3), turned to -90 degrees
- moved U6 63.6 mm to (171.5, 127.0)
- moved C4 63.4 mm to (161.7, 128.3), turned to -90 degrees
- moved C10 63.1 mm to (166.3, 138.8), turned to -90 degrees
- moved C14 63.0 mm to (169.6, 138.3)
- moved L1 62.4 mm to (162.6, 128.3), turned to 90 degrees
- moved C2 60.8 mm to (164.4, 125.5), turned to 180 degrees
- moved C13 60.8 mm to (170.8, 130.6), turned to 90 degrees
- moved C3 60.7 mm to (164.4, 128.7), turned to -90 degrees
- moved R2 60.3 mm to (173.4, 127.2), turned to -90 degrees
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Connections:
- J3 pad 1: /PWR B -> GND
- J3 pad 2: GND -> /PWR B
- J5 pad 1: /CAM RX -> /CAM1 RX
- J5 pad 2: /CAM TX -> /CAM1 TX
- J7 pad 1: /PWR A -> GND
- J7 pad 2: GND -> /PWR A
- U1 pad 2: unconnected-(U1-GND-Pad2) -> GND
- U1 pad 4: unconnected-(U1-VDD-Pad4) -> +3V3
- U1 pad 5: unconnected-(U1-RFIN-Pad5) -> Net-(AE1-A)
- U1 pad 6: unconnected-(U1-CTRL-Pad6) -> /RF CTRL
- U3 pad 10: unconnected-(U3-PA3-Pad10) -> /CAM1 TX
- U3 pad 12: unconnected-(U3-PA4-Pad12) -> /BATT SENSE A
- U3 pad 13: unconnected-(U3-PA5-Pad13) -> /PWRB EN
- U3 pad 14: unconnected-(U3-PA6-Pad14) -> /BATT SENSE B
- U3 pad 19: unconnected-(U3-PH3-Pad19) -> /BOOTSEL
- U3 pad 2: unconnected-(U3-PB4-Pad2) -> /PRWA EN
- U3 pad 26: unconnected-(U3-OSC_IN-Pad26) -> /OSC_IN
- U3 pad 27: unconnected-(U3-OSC_OUT-Pad27) -> /OSC_OUT
- U3 pad 29: +3V3 -> /VFBSMPS
- U3 pad 30: unconnected-(U3-PB0-Pad30) -> /LED INDICATION
- U3 pad 34: unconnected-(U3-PA11-Pad34) -> /CURRENT SENSE B
- U3 pad 38: unconnected-(U3-PC13-Pad38) -> /RF CTRL
- U3 pad 4: unconnected-(U3-PB6-Pad4) -> /CAM2 RX
- U3 pad 45: unconnected-(U3-VFBSMPS-Pad45) -> /VFBSMPS
- U3 pad 5: unconnected-(U3-PB7-Pad5) -> /CAM2 TX
- U3 pad 7: unconnected-(U3-PA0-Pad7) -> /CURRENT SENSE A
- U3 pad 9: unconnected-(U3-PA2-Pad9) -> /CAM1 RX
- U5 pad 1: /PRW1 EN -> /PRWA EN
- U5 pad 6: /PWR A -> /PWR A SENS
- U6 pad 1: /PWR2 EN -> /PWRB EN
- U6 pad 6: /PWR A -> /PWR B SENS
Routing:
- net /RF CTRL: track 0.00 -> 32.4 mm, vias 0 -> 2
- net /CURRENT SENSE B: track 0.00 -> 28.7 mm, vias 0 -> 2
- net GND: track 0.00 -> 28.1 mm, vias 0 -> 12
- net /CAM1 TX: track 0.00 -> 24.6 mm, vias 0 -> 1
- net /CAM1 RX: track 0.00 -> 23.9 mm, vias 0 -> 1
- net +3V3: track 0.00 -> 21.7 mm, vias 0 -> 7
- net /PWR B: track 0.00 -> 20.7 mm, vias 0 -> 2
- net +12VA: track 0.00 -> 18.3 mm, vias 0 -> 2
- net /PWR A SENS: track 0.00 -> 17.3 mm
- net /PWR B SENS: track 0.00 -> 15.7 mm, vias 0 -> 2
- net /PWRB EN: track 0.00 -> 12.1 mm, vias 0 -> 2
- net +12V: track 0.00 -> 11.4 mm, vias 0 -> 1
- net /CAM2 TX: track 0.00 -> 9.90 mm, vias 0 -> 1
- net /CAM2 RX: track 0.00 -> 8.98 mm, vias 0 -> 1
- net /BATT SENSE B: track 0.00 -> 6.39 mm
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- removed copper zone on In2.Cu, net GND
Other:
- board size 25.4 x 25.4 mm -> 15.9 x 25.4 mm

Commit message: final version?
Parts:
- removed D4: D_Schottky, Diode_SMD:D_SOD-323F
- removed J8: DNP, Connector_PinHeader_2.54mm:PinHeader_1x05_P2.54mm_Vertical
- removed Q3: AO3401A, Package_TO_SOT_SMD:SOT-23
- added D3: D_Zener, Diode_SMD:D_SOD-323F, F.Cu at (170.3, 124.3)
- added J2: Conn_01x04, Connector_PinHeader_2.54mm:PinHeader_1x04_P2.54mm_Vertical, B.Cu at (173.4, 143.6)
- added R10: 51k, Resistor_SMD:R_0402_1005Metric, F.Cu at (172.8, 124.0)
- added REF**: BreakLine_5h_D0.5mm_P0.85mm, Panelization:BreakLine_5h_D0.5mm_P0.85mm, F.Cu at (161.1, 119.5)
- added REF**: BreakLine_5h_D0.5mm_P0.85mm, Panelization:BreakLine_5h_D0.5mm_P0.85mm, F.Cu at (172.6, 145.6)
- H1, H2: value MountingHole_Pad -> MountingHole; footprint MountingHole:MountingHole_2.2mm_M2_DIN965_Pad -> MountingHole:MountingHole_2.2mm_M2_DIN965; moved to B.Cu
- J1, J3, J4, J7: footprint Connector_Molex:Molex_PicoBlade_53261-0271_1x02-1MP_P1.25mm_Horizontal -> Connector_Molex:Molex_PicoBlade_53048-0210_1x02_P1.25mm_Horizontal
- U4: value XC6206P332MR -> DS8242; footprint Package_TO_SOT_SMD:SOT-23-3 -> .pretty:SOT-23-3_L2.9-W1.6-P1.90-LS2.8-BR
- moved H2 27.7 mm to (172.6, 147.3)
- moved H1 27.4 mm to (161.1, 117.9)
- moved R1 17.9 mm to (160.4, 144.0), turned to 0 degrees
- moved R6 13.3 mm to (161.5, 140.7), turned to 90 degrees
- moved R9 12.5 mm to (161.6, 138.1), turned to 180 degrees
- moved J3 12.0 mm to (160.1, 127.1)
- moved R8 11.7 mm to (161.6, 137.1), turned to 0 degrees
- moved C12 11.5 mm to (162.0, 122.7)
- moved J4 11.4 mm to (160.2, 134.5)
- moved U6 10.3 mm to (161.5, 124.8)
- moved R2 10.3 mm to (163.4, 124.7)
- moved R3 10.0 mm to (161.4, 127.2), turned to -90 degrees
- moved D2 9.97 mm to (160.6, 131.2), turned to 0 degrees
- moved U5 9.80 mm to (163.4, 141.0), turned to 180 degrees
- moved D1 9.52 mm to (161.0, 144.0), turned to 0 degrees
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Connections:
- Q1 pad 1: GND -> Net-(D3-A)
- Q1 pad 3: Net-(D4-K) -> Net-(JP1-C)
- U3 pad 12: /BATT SENSE A -> /BATT SENSE B
- U3 pad 14: /BATT SENSE B -> unconnected-(U3-PA6-Pad14)
- U3 pad 30: /LED INDICATION -> unconnected-(U3-PB0-Pad30)
- U3 pad 34: /CURRENT SENSE B -> unconnected-(U3-PA11-Pad34)
- U3 pad 35: unconnected-(U3-PA12-Pad35) -> /LED INDICATION
- U3 pad 36: unconnected-(U3-PA13-Pad36) -> /BATT SENSE A
- U3 pad 8: unconnected-(U3-PA1-Pad8) -> /CURRENT SENSE B
Routing:
- net /CURRENT SENSE B: track 28.7 -> 3.56 mm, vias 2 -> 0
- net /PWR B SENS: track 15.7 -> 34.7 mm
- net /PWR A: track 5.76 -> 22.8 mm, vias 2 -> 3
- net +12V: track 11.4 -> 22.1 mm, vias 1 -> 2
- net /PRWA EN: track 2.07 -> 12.1 mm
- net /CAM1 RX: track 23.9 -> 14.3 mm
- net /PWR B: track 20.7 -> 29.6 mm, vias 2 -> 1
- net +12VA: track 18.3 -> 26.5 mm, vias 2 -> 1
- net /CAM1 TX: track 24.6 -> 17.0 mm
- net /LED INDICATION: track 0.00 -> 6.96 mm, vias 0 -> 1
- net /VFBSMPS: track 4.95 -> 11.5 mm, vias 0 -> 2
- net /RF CTRL: track 32.4 -> 26.1 mm
- net /PWR A SENS: track 17.3 -> 23.5 mm, vias 0 -> 2
- net /PWRB EN: track 12.1 -> 17.7 mm
- net Net-(D4-K): track 5.58 -> 0.00 mm
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- added copper zone on F.Cu, net GND
Other:
- board size 15.9 x 25.4 mm -> 15.9 x 33.8 mm
- board text added: "- +"
- board text added: "A IN"
- board text added: "A OUT"
- board text added: "B A"
- board text added: "B IN"
- board text added: "B OUT"
- board text added: "GND TX RX GND TX RX"
- board text added: "THE THING AMAJIG"
