File: CamControl/camcontrol stm32/camcontrol stm32.kicad_sch (KiCad schematic)
At the start: 53 parts, among them J1 Power 1, J2 Conn_01x04, J3 Power 1, J4 Power 1, J5 Conn_01x06, J6 Conn_01x02, J7 Power 1, Q1 AO3401A, U1 BGS12P2L6, U2 BALFHB-WL-02D3, U3 STM32WLE4CCUx, U4 DS8242, U5 TPS25970LRPWR, U6 TPS25970LRPWR, U7 INA2180, Y1 32MHz

Commit message: fixed dumb issue
Connections:
- net +3V3: now also U1.4 (VDD)
Changed lines of the file:
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@@
 	(wire
 		(pts
-			(xy 123.825 205.74) (xy 131.445 205.74)
+			(xy 121.92 205.74) (xy 131.445 205.74)
 		)
 		(stroke
@@
 	(wire
 		(pts
+			(xy 38.735 184.15) (xy 38.735 187.325)
+		)
+		(stroke
+			(width 0)
+			(type default)
+		)
+	)
+	(wire
+		(pts
 			(xy 154.305 241.3) (xy 155.575 241.3)
 		)
@@
 	)
 	(label "BOOTSEL"
-		(at 123.825 205.74 0)
+		(at 121.92 205.74 0)
 		(effects
 			(font
@@
 	)
 	(symbol
+		(lib_id "power:+3V3")
+		(at 38.735 184.15 0)
+		(unit 1)
+		(exclude_from_sim no)
+		(in_bom yes)
+		(on_board yes)
+		(dnp no)
+		(fields_autoplaced yes)
+		(property "Reference" "#PWR029"
+			(at 38.735 187.96 0)
+			(effects
+				(font
+					(size 1.27 1.27)
+				)
+				(hide yes)
+			)
+		)
+		(property "Value" "+3V3"
+			(at 38.735 179.705 0)
+			(effects
+				(font
+					(size 1.27 1.27)
+				)
+			)
+		)
+		(property "Footprint" ""
+			(at 38.735 184.15 0)
+			(effects
+				(font
+					(size 1.27 1.27)
+				)
+				(hide yes)
+			)
+		)
+		(property "Datasheet" ""
+			(at 38.735 184.15 0)
+			(effects
+				(font
+					(size 1.27 1.27)
+				)
+				(hide yes)
+			)
+		)
+		(property "Description" "Power symbol creates a global label with name \"+3V3\""
+			(at 38.735 184.15 0)
+			(effects
+				(font
+					(size 1.27 1.27)
+				)
+				(hide yes)
+			)
+		)
+		(pin "1"
+		)
+		(instances
+			(project "camcontrol stm32"
+				(path "/299d0a04-aa0f-4714-a339-a062da4333a5"
+					(reference "#PWR029")
+					(unit 1)
+				)
+			)
+		)
+	)
+	(symbol
 		(lib_id "Device:D_Zener")
 		(at 346.075 225.425 270)
@@
 		(dnp no)
 		(property "Reference" "AE1"
-			(at 23.495 177.1649 0)
+			(at 22.86 173.355 0)
 			(effects
 				(font
@@
 		)
 		(property "Value" "Antenna_Shield"
-			(at 23.495 179.7049 0)
+			(at 22.86 175.895 0)
 			(effects
 				(font
