File: CamControl/camcontrol stm32/camcontrol stm32.kicad_sch (KiCad schematic)
At the start: 53 parts, among them J1 Power 1, J2 Conn_01x04, J3 Power 1, J4 Power 1, J5 Conn_01x06, J6 Conn_01x02, J7 Power 1, Q1 AO3401A, U1 BGS12P2L6, U2 BALFHB-WL-02D3, U3 STM32WLE4CCUx, U4 DS8242, U5 TPS25970LRPWR, U6 TPS25970LRPWR, U7 INA2180, Y1 32MHz

Commit message: trying to get hope code working again
Parts:
- removed C15: 100n, Capacitor_SMD:C_0402_1005Metric, symbol Device:C_Small
Connections:
- net +12V: now also R24.1; no longer R23.1
- net +12VA: now also R9.1; no longer R8.1
- net +3V3: now also J6.1 (Pin_1)
- net BATT SENSE A: now also R8.1, R9.2; no longer R8.2, R9.1
- net BATT SENSE B: now also R23.1, R24.2; no longer R23.2, R24.1
- net GND: now also R23.2, R8.2; no longer J6.1 (Pin_1), R24.2, R9.2
Other:
- moved on the sheet: R23, R24, R8, R9
