File: Metrumizer/metrumizer/metrumizer.kicad_sch (KiCad schematic)
At the start: 95 parts, among them J1 Screw_Terminal_01x02, J2 USB_B_Micro, J3 Conn_01x04, J4 Conn_01x06, Q1 AO3401A, Q2 AO3401A, Q3 Si7232DN, U1 ATSAMD21G17A-M, U10 LM293, U2 CC1200, U3 W25Q128JVS, U4 ADXL375BCCZ-RL7, U5 MS5607-02BA, U6 MAX-M10S, U7 MCP130-315, U8 XC6206P332MR, Y1 X322516MLB4SI, Y2 Crystal_GND24

Commit message: new pyro, looking at new RF. still no baord
Parts:
- removed J1: Screw_Terminal_01x02, TerminalBlock_Phoenix:TerminalBlock_Phoenix_MPT-0,5-2-2.54_1x02_P2.54mm_Horizontal, symbol Connector:Screw_Terminal_01x02
- removed J4: Conn_01x06, symbol Connector_Generic:Conn_01x06
- removed Q3: Si7232DN, Package_DirectFET:DirectFET_SA, symbol Transistor_FET:IRF6802SD
- removed R21: 100k, Resistor_SMD:R_0402_1005Metric, symbol Device:R_Small
- removed R22: 27k, Resistor_SMD:R_0402_1005Metric, symbol Device:R_Small
- removed U10: LM293, .pretty:MINISO-8_L3.0-W3.0-P0.65-LS4.9-BL, symbol Comparator:LM393
- added C37: 1.8n, Capacitor_SMD:C_0402_1005Metric, symbol Device:C_Small
- added H1, H2, H3, H4: MountingHole, MountingHole:MountingHole_3.2mm_M3, symbol Mechanical:MountingHole
- added J1, J4: Conn_01x03, footprints:CONN3_2059-303&slash_998-403_WAG, symbol Connector_Generic:Conn_01x03
- added R23: 5.6k, Resistor_SMD:R_0402_1005Metric, symbol Device:R_Small
- added R24: 10k, Resistor_SMD:R_0402_1005Metric, symbol Device:R_Small
- added R25: 1k, Resistor_SMD:R_0402_1005Metric, symbol Device:R_Small
- added U10: 74LVC2G14, symbol 74xGxx:74LVC2G14
- added U9: TPS2H160BQPWPRQ1, .pretty:HTSSOP-16_L5.0-W4.4-P0.65-LS6.4-BL-EP-A, symbol .kicad_sym:TPS2H160BQPWPRQ1
- AE1: footprint (none) -> .pretty:ANT-SMD_1909763-1; LCSC Part (none) -> C392444
- C11, C9: footprint (none) -> Capacitor_SMD:C_0402_1005Metric; LCSC Part (none) -> C1547
- C15, C19, C35: footprint (none) -> Capacitor_SMD:C_0402_1005Metric; LCSC Part (none) -> C15195
- C16, C17: footprint (none) -> Capacitor_SMD:C_0402_1005Metric; LCSC Part (none) -> C1554
- C18, C20, C21, C22, C24, C25, C26, C29: footprint (none) -> Capacitor_SMD:C_0603_1608Metric; LCSC Part (none) -> C1622
- C23: footprint (none) -> Capacitor_SMD:C_0402_1005Metric; LCSC Part (none) -> C16772
- C27, C28, C30: footprint (none) -> Capacitor_SMD:C_0402_1005Metric; LCSC Part (none) -> C60220
- C31: footprint (none) -> Capacitor_SMD:C_0402_1005Metric; LCSC Part (none) -> C1563
- C32: footprint (none) -> Capacitor_SMD:C_0402_1005Metric; LCSC Part (none) -> C1559
- C33: footprint (none) -> Capacitor_SMD:C_0402_1005Metric; LCSC Part (none) -> C41744
- C34: footprint (none) -> Capacitor_SMD:C_0603_1608Metric; LCSC Part (none) -> C39148
- C36: footprint (none) -> Capacitor_SMD:C_0402_1005Metric; LCSC Part (none) -> C1546
- JP1: footprint (none) -> Jumper:SolderJumper-2_P1.3mm_Bridged_RoundedPad1.0x1.5mm
- L1, L3, L4: footprint (none) -> Inductor_SMD:L_0402_1005Metric; LCSC Part (none) -> C18830; Part # (none) -> LQG15HS27NJ02D
- L2, L9: footprint (none) -> Inductor_SMD:L_0402_1005Metric; LCSC Part (none) -> C395071; Part # (none) -> LQG15HS56NJ02D
- L5, L6: footprint (none) -> Inductor_SMD:L_0402_1005Metric; LCSC Part (none) -> C27143; Part # (none) -> LQG15HS15NJ02D
- L7: footprint (none) -> Inductor_SMD:L_0402_1005Metric; LCSC Part (none) -> C3032783; Part # (none) -> MLG1005S43NJTD25
- L8: footprint (none) -> Inductor_SMD:L_0402_1005Metric; Part # (none) -> LQG15HS22NG02D
- R11, R13: footprint (none) -> Resistor_SMD:R_0402_1005Metric; LCSC Part (none) -> C25744
- R15: value 1k -> 100k
- R16: value 3.3k -> 27k; LCSC Part C11702 -> (none)
- R17: value 3.3k -> 100k
- R18: value 1k -> 27k; LCSC Part C11702 -> (none)
- R2, R3: footprint (none) -> Resistor_SMD:R_0402_1005Metric; LCSC Part (none) -> C25105
- R20: value 27k -> 100k
- R7, R8: footprint (none) -> Resistor_SMD:R_0402_1005Metric; LCSC Part (none) -> C25796
- U1: LCSC Part (none) -> C614532
- U2: LCSC Part (none) -> C122881
- U3: LCSC Part (none) -> C97521
- U5: LCSC Part (none) -> C97627
- U7: LCSC Part (none) -> C625194
- Y1: footprint (none) -> Crystal:Crystal_SMD_3225-4Pin_3.2x2.5mm; LCSC Part (none) -> C5444547
- Y2: value Crystal_GND24 -> YF4040M00033T8188097; footprint (none) -> Crystal:Crystal_SMD_3225-4Pin_3.2x2.5mm; LCSC Part (none) -> C2831465
Connections:
- net +3V3: no longer JP1.2 (B)
- net +BATT: now also R19.1, R20.1, R23.1, U10.5 (VCC), U9.13 (VS), U9.14 (VS)
- net BATT POSTSW: now also J4.5 (Pin_3), J4.6 (Pin_3)
- net GND: now also R16.1, R18.1, Y2.1, Y2.3, J1.3 (Pin_2), J1.4 (Pin_2), J4.1 (Pin_1), J4.2 (Pin_1), J4.3 (Pin_2), J4.4 (Pin_2), R24.2, R25.1, U10.2 (GND), U9.17 (EP), U9.8 (GND), U9.9 (THER); no longer R16.2, R17.2, R20.1, Y2.2, Y2.4
- net fet_a: now also J1.1 (Pin_1), J1.2 (Pin_1), U10.3, U9.15 (OUT1), U9.16 (OUT1); no longer R20.2, U1.15 (PA10)
- net fire_a: now also U9.2 (IN2); no longer R15.1, R16.1
- net fire_b: now also U9.1 (IN1); no longer R17.1, R18.1
- net sense_b: now also R17.2, R18.2
- net v_batt: now also R23.2, R24.1
- net xosc Q1: now also Y2.2; no longer Y2.1
- net xosc Q2: now also Y2.4; no longer Y2.3
- net sense_a: now reaches R15.2
- net sense_a: now also R16.2, U1.15 (PA10)
- net at U2.23 (LPF0): now also C37.2
- net at U2.24 (LPF1): now also C37.1
- net VCC_RF: now reaches U6.14 (VCC_RF)
- net VCC_RF: now also JP1.2 (B)
- new net: R15.1, U10.4
- new net: R17.1, U10.6
- new net: R25.2, U9.7 (CL)
- new net fet_b: J1.5 (Pin_3), J1.6 (Pin_3), R20.2, U10.1, U9.11 (OUT2), U9.12 (OUT2)
- no-connect marks 16 -> 20
Other:
- note added: "DEBUG"
- note added: "IO"
- moved on the sheet: Y2

Commit message: dan f10, n511 module, board layout
Parts:
- removed AE1: IPEX, .pretty:ANT-SMD_1909763-1, symbol Device:Antenna_Shield
- removed C15, C19, C35: 10n, Capacitor_SMD:C_0402_1005Metric, symbol Device:C_Small
- removed C16, C17: 20p, Capacitor_SMD:C_0402_1005Metric, symbol Device:C_Small
- removed C18, C20, C21, C22, C24, C25, C26, C29: 47n, Capacitor_SMD:C_0603_1608Metric, symbol Device:C_Small
- removed C23: 0.22u, Capacitor_SMD:C_0402_1005Metric, symbol Device:C_Small
- removed C27, C28, C30: 5.1p, Capacitor_SMD:C_0402_1005Metric, symbol Device:C_Small
- removed C31: 39p, Capacitor_SMD:C_0402_1005Metric, symbol Device:C_Small
- removed C32: 2.2p, Capacitor_SMD:C_0402_1005Metric, symbol Device:C_Small
- removed C33: 6.2p, Capacitor_SMD:C_0402_1005Metric, symbol Device:C_Small
- removed C34: 56p, Capacitor_SMD:C_0603_1608Metric, symbol Device:C_Small
- removed C36: 100p, Capacitor_SMD:C_0402_1005Metric, symbol Device:C_Small
- removed C37: 1.8n, Capacitor_SMD:C_0402_1005Metric, symbol Device:C_Small
- removed D5: LED, LED_SMD:LED_0805_2012Metric, symbol Device:LED
- removed FL1: B39162B8813P810, Filter:Filter_1109-5_1.1x0.9mm, symbol Filter:B39162B8813P810
- removed JP1: jumper, Jumper:SolderJumper-2_P1.3mm_Bridged_RoundedPad1.0x1.5mm, symbol Jumper:SolderJumper_2_Open
- removed L1, L3, L4: 27n, Inductor_SMD:L_0402_1005Metric, symbol Device:L_Small
- removed L5, L6: 15n, Inductor_SMD:L_0402_1005Metric, symbol Device:L_Small
- removed L7: 43n, Inductor_SMD:L_0402_1005Metric, symbol Device:L_Small
- removed L8: 22n, Inductor_SMD:L_0402_1005Metric, symbol Device:L_Small
- removed L9: 56n, Inductor_SMD:L_0402_1005Metric, symbol Device:L_Small
- removed R10: 10, Resistor_SMD:R_0402_1005Metric, symbol Device:R_Small
- removed R11, R13: 10k, Resistor_SMD:R_0402_1005Metric, symbol Device:R_Small
- removed R12: 8k06, symbol Device:R_Small
- removed R14: 9k09, symbol Device:R_Small
- removed R6: 1k, Resistor_SMD:R_0402_1005Metric, symbol Device:R_Small
- removed R7: 56k, Resistor_SMD:R_0402_1005Metric, symbol Device:R_Small
- removed R9: 18, symbol Device:R_Small
- removed U2: CC1200, Package_DFN_QFN:QFN-32-1EP_5x5mm_P0.5mm_EP3.45x3.45mm, symbol RF:CC1200
- removed U6: MAX-M10S, RF_GPS:ublox_MAX, symbol RF_GPS:MAX-M10S
- removed Y2: YF4040M00033T8188097, Crystal:Crystal_SMD_3225-4Pin_3.2x2.5mm, symbol Device:Crystal_GND24
- added AE2: SMA, .pretty:CONN-SMD_KH-SMA-KE8-G, symbol Device:Antenna_Shield
- added IC1: DAN-F10N-00B, KiCad:DANF10N00B, symbol DAN-F10N-00B:DAN-F10N-00B
- added JP2, JP3: SolderJumper_3_Open, Jumper:SolderJumper-3_P1.3mm_Open_RoundedPad1.0x1.5mm, symbol Jumper:SolderJumper_3_Open
- added U11: N511_433, .pretty:N511 433, symbol .kicad_sym:N511_433
- AE3: value SMA -> IPEX; footprint .pretty:CONN-SMD_KH-SMA-KE8-G -> .pretty:ANT-SMD_1909763-1; LCSC Part C530661 -> C392444
- L2: value 56n -> 27n; LCSC Part C395071 -> C18830; Part # LQG15HS56NJ02D -> LQG15HS27NJ02D
- R16, R18: LCSC Part (none) -> C25771
- R8: value 56k -> 10; LCSC Part C25796 -> C11702
- U10: footprint (none) -> Package_TO_SOT_SMD:SOT-363_SC-70-6; LCSC Part (none) -> C19829575
Connections:
- net LNA_N is gone; now on an unnamed net: L2.1
- net LNA_P is gone; now on an unnamed net: L2.2
- net +3V3: now also IC1.52 (VCC_1), IC1.53 (VCC_2), JP2.1 (A), JP3.1 (A), U11.13 (VCC)
- net GND: now also AE2.2 (Shield), IC1.1 (GND_1), IC1.100 (GND_80), IC1.13 (GND_9), IC1.14 (GND_10), IC1.15 (GND_11), IC1.19 (GND_12), IC1.2 (GND_2), IC1.21 (GND_13), IC1.22 (GND_14), IC1.23 (GND_15), IC1.26 (GND_16), IC1.27 (GND_17), IC1.28 (GND_18), IC1.29 (GND_19), IC1.3 (GND_3), IC1.30 (GND_20), IC1.33 (GND_21), IC1.35 (GND_22), IC1.37 (GND_23), IC1.38 (GND_24), IC1.4 (GND_4), IC1.40 (GND_25), IC1.41 (GND_26), IC1.42 (GND_27), IC1.43 (GND_28), IC1.44 (GND_29), IC1.47 (GND_30), IC1.48 (GND_31), IC1.49 (GND_32), IC1.5 (GND_5), IC1.50 (GND_33), IC1.51 (GND_34), IC1.54 (GND_35), IC1.56 (GND_36), IC1.57 (GND_37), IC1.58 (GND_38), IC1.59 (GND_39), IC1.6 (GND_6), IC1.60 (GND_40), IC1.61 (GND_41), IC1.62 (GND_42), IC1.63 (GND_43), IC1.64 (GND_44), IC1.65 (GND_45), IC1.66 (GND_46), IC1.67 (GND_47), IC1.68 (GND_48), IC1.69 (GND_49), IC1.7 (GND_7), IC1.70 (GND_50), IC1.71 (GND_51), IC1.72 (GND_52), IC1.73 (GND_53), IC1.74 (GND_54), IC1.75 (GND_55), IC1.76 (GND_56), IC1.77 (GND_57), IC1.78 (GND_58), IC1.79 (GND_59), IC1.8 (GND_8), IC1.80 (GND_60), IC1.81 (GND_61), IC1.82 (GND_62), IC1.83 (GND_63), IC1.84 (GND_64), IC1.85 (GND_65), IC1.86 (GND_66), IC1.87 (GND_67), IC1.88 (GND_68), IC1.89 (GND_69), IC1.90 (GND_70), IC1.91 (GND_71), IC1.92 (GND_72), IC1.93 (GND_73), IC1.94 (GND_74), IC1.95 (GND_75), IC1.96 (GND_76), IC1.97 (GND_77), IC1.98 (GND_78), IC1.99 (GND_79), JP2.3 (B), JP3.3 (B), U11.14 (GND), U11.2 (GND), U11.3 (GND); no longer R8.2
- net VCC_RF: now also R8.2, IC1.31 (VCC_RF)
- net cs_radio: now also U11.12 (NSS)
- net fet_a: now also U10.1; no longer U10.3
- net fet_b: now also U10.3; no longer U10.1
- net miso5: now also U11.10 (MISO)
- net mosi5: now also U11.8 (MOSI)
- net radio_int: now also U11.7 (GPIO2)
- net radio_marc_int: now also U11.4 (GPIO3)
- net reset_n: now also IC1.16 (RESET_N), U11.5 (RST)
- net rx1: now also IC1.10 (TXD)
- net sck5: now also U11.9 (SCK)
- net tx1: now also IC1.9 (RXD)
- net at U10.4: now also R17.1; no longer R15.1
- net at AE3.1 (A): now also IC1.34 (EXT_RF_IN)
- net at U10.6: now also R15.1; no longer R17.1
- new net: JP2.2 (C), U11.6 (VTC)
- new net: AE2.1 (A), U11.1 (RF)
- new net ANT_CTRL: IC1.32 (ANT_CTRL), JP3.2 (C)
- no-connect marks 20 -> 26
Other:
- note removed: "1 EA for VDD & AVDD exp. AVDD_XOSC"
- note removed: "GPS"
- moved on the sheet: U10A, U10B

Commit message: weorjk
Parts:
- removed AE3: IPEX, .pretty:ANT-SMD_1909763-1, symbol Device:Antenna_Shield
- removed H3, H4: MountingHole, MountingHole:MountingHole_3.2mm_M3, symbol Mechanical:MountingHole
- removed IC1: DAN-F10N-00B, KiCad:DANF10N00B, symbol DAN-F10N-00B:DAN-F10N-00B
- removed J3: Conn_01x04, .pretty:4 pads 2.54mm spacign, symbol Connector_Generic:Conn_01x04
- removed JP3: SolderJumper_3_Open, Jumper:SolderJumper-3_P1.3mm_Open_RoundedPad1.0x1.5mm, symbol Jumper:SolderJumper_3_Open
- removed L2: 27n, Inductor_SMD:L_0402_1005Metric, symbol Device:L_Small
- removed R8: 10, Resistor_SMD:R_0402_1005Metric, symbol Device:R_Small
- added AE1: IPEX, .pretty:ANT-SMD_1909763-1, symbol Device:Antenna_Shield
- added D5: LED, LED_SMD:LED_0805_2012Metric, symbol Device:LED
- added J3, J5: Conn_01x02, Jumper:SolderJumper-2_P1.3mm_Open_Pad1.0x1.5mm, symbol Connector_Generic:Conn_01x02
- added L1: 27n, Inductor_SMD:L_0402_1005Metric, symbol Device:L_Small
- added R10: 10, Resistor_SMD:R_0402_1005Metric, symbol Device:R_Small
- added R6: 1k, Resistor_SMD:R_0402_1005Metric, symbol Device:R_Small
- added R7: 56k, Resistor_SMD:R_0402_1005Metric, symbol Device:R_Small
- added U6: MAX-M10S, RF_GPS:ublox_MAX, symbol RF_GPS:MAX-M10S
Connections:
- net +3V3: now also U6.7 (VCC_IO), U6.8 (VCC)
- net +BATT: now also R7.2
- net GND: now also AE1.2 (Shield), J3.2 (Pin_2), R6.1, U6.1 (GND), U6.10 (GND), U6.12 (GND)
- net VCC_RF: now also R10.2, U6.14 (VCC_RF)
- net reset_n: now also J5.1 (Pin_1), U6.9 (~{RESET})
- net rx1: now also U6.3 (RXD)
- net swclk: now also J3.1 (Pin_1)
- net swdio: now also J5.2 (Pin_2)
- net tx1: now also U6.2 (TXD)
- new net: D5.1 (K), R6.2
- new net: R7.1, U6.6 (V_BCKP)
- new net: L1.1, R10.1
- new net: AE1.1 (A), L1.2, U6.11 (RF_IN)
- new net: D5.2 (A), U6.4 (TIMEPULSE)
- no-connect marks 26 -> 20
Other:
- note added: "GPS"

Commit message: cam control
Parts:
- removed Q2: AO3401A, Package_TO_SOT_SMD:SOT-23, symbol Transistor_FET:AO3401A
- added C15: 100n, Capacitor_SMD:C_0402_1005Metric, symbol Device:C_Small
- added C16: 1n, Capacitor_SMD:C_0402_1005Metric, symbol Device:C_Small
- added C17: 10n, Capacitor_SMD:C_0402_1005Metric, symbol Device:C_Small
- added Q3, Q4: AO3401A, Package_TO_SOT_SMD:SOT-23, symbol Transistor_FET:AO3401A
- added R8, R9: 1k, Resistor_SMD:R_0402_1005Metric, symbol Device:R_Small
- added U2: HX6571, :SOT-23-3_L2.9-W1.6-P1.90-LS2.8-BR, symbol .kicad_sym:HX6571
Connections:
- net +3V3: now also C15.1; no longer U3.4 (GND)
- net +BATT: now also C17.1, Q3.2 (S), R8.2, U2.2 (Vin)
- net GND: now also U3.4 (GND), C15.2, C16.2, C17.2, Q4.1 (G), U2.1 (GND)
- net at D2.1 (K), Q1.2 (S): now also Q4.3 (D)
- new net: Q3.1 (G), R9.2
- new net: Q3.3 (D), Q4.2 (S)
- new net MAG LATCH: C16.1, R8.1, R9.1, U2.3 (Vout)
Other:
- moved on the sheet: C1, C2, C3, D1, D2, Q1, R1, R23, R24, U8

Commit message: things
Parts:
- removed R19, R20: 100k, Resistor_SMD:R_0402_1005Metric, symbol Device:R_Small
- removed R25: 1k, Resistor_SMD:R_0402_1005Metric, symbol Device:R_Small
- removed U10: 74LVC2G14, Package_TO_SOT_SMD:SOT-363_SC-70-6, symbol 74xGxx:74LVC2G14
- removed U9: TPS2H160BQPWPRQ1, .pretty:HTSSOP-16_L5.0-W4.4-P0.65-LS6.4-BL-EP-A, symbol .kicad_sym:TPS2H160BQPWPRQ1
- added C18: 1u, Capacitor_SMD:C_0402_1005Metric, symbol Device:C_Small
- added Q2, Q5: AO3400A, Package_TO_SOT_SMD:SOT-23, symbol Transistor_FET:AO3400A
- added R11: 510, Resistor_SMD:R_0402_1005Metric, symbol Device:R_Small
- added U9: TPS25970LRPWR, easyeda2kicad2:QFN-10-2x2-hotrod, symbol easyeda2kicad2:TPS25970LRPWR
Connections:
- net +BATT: now also C18.1, U9.5 (IN)
- net GND: now also C18.2, Q2.2 (S), Q5.2 (S), R11.2, U9.2 (OLVO), U9.8 (GND); no longer J1.3 (Pin_2), J1.4 (Pin_2), J4.1 (Pin_1), J4.2 (Pin_1)
- net fet_a: now also R15.1, Q2.3 (D)
- net fet_b: now also R17.1, Q5.3 (D)
- net fire_a: now also Q2.1 (G), Q5.1 (G)
- net BATT POSTSW renamed BATT PRESW
- new net: R11.1, U9.9 (ILM)
- new net PWRB EN: U9.1 (EN/UVLO)
- new net PYRO PWR: J1.3 (Pin_2), J1.4 (Pin_2), J4.1 (Pin_1), J4.2 (Pin_1), U9.6 (OUT)
- no-connect marks 20 -> 19
Other:
- moved on the sheet: AE2, JP2, R15, R16, R17, R18, U11
