File: Hardware/kicad/Lyra_flight_computer/lyra r1/lyra r1/lyra r1.kicad_sch (KiCad schematic)
At the start: 82 parts, among them J1 USB_B_Micro, J10 BOOT 0 HEADER, J11 Screw_Terminal_01x04, J12 Screw_Terminal_01x04, J2 UART Breakout, J3 Screw_Terminal_01x04, J4 I2C Breakout, J5 Screw_Terminal_01x04, J6 Conn_02x03_Top_Bottom, J7 Conn_02x03_Top_Bottom, J8 SPI Breakout, J9 MEM2067-02-180-00-A, Q1 AO3401A, Q2 Q_NMOS_GSD, Q3 Q_NMOS_GSD, SW1 SW_SPST, SW2 SW_Push_DPDT, U1 LM317_SOT-223, U2 LM317_SOT-223, U3 USBLC6-2SC6, U4 BMI088, U5 BMP390L, U6 W25Q32JVSS, U7 STM32F405RGTx, X1 ECS-2520MV-xxx-xx

Commit message: autosaves
Other:
- moved on the sheet: J10, R19
